Commit message: Finished joy control

File: i3e-d3_description/urdf/wheel.urdf.xacro (robot description, xacro)
@@ -1,4 +1,6 @@
 <?xml version="1.0"?>
 <robot xmlns:xacro="http://www.ros.org/wiki/xacro" name="i3e-d3_wheel">
+    <xacro:property name="husky_wheel_length" value="0.1143" />
+    <xacro:property name="husky_wheel_radius" value="0.1651" />
     <xacro:macro name="i3e-d3_wheel" params="prefix *joint_pose">
         <link name="${prefix}_wheel_link">
@@ -15,5 +17,6 @@
                 <origin xyz="0.0 0.0 0.0" rpy="0.0 0.0 0.0"/>
                 <geometry>
-                    <mesh filename="package://i3e-d3_description/meshes/wheel_130x60.stl"/>
+                    <mesh filename="package://i3e-d3_description/meshes/wheel_husky.stl"
+                          scale="${wheel_radius/husky_wheel_radius} ${wheel_length/husky_wheel_length} ${wheel_radius/husky_wheel_radius}"/>
                 </geometry>
             </visual>
