Commit message: Just a backup commit

File: i3e-d3_description/urdf/decorations.urdf.xacro (robot description, xacro)
@@ -19,5 +19,5 @@
         </link>
         <joint name="display_joint" type="fixed">
-            <origin xyz="0.15 0.0 0.028" rpy="0.0 ${28.74*PI/180} 0.0"/>
+            <origin xyz="0.16 0.0 0.019" rpy="0.0 ${40*PI/180} 0.0"/>
             <parent link="base_link"/>
             <child link="display_link"/>

File: i3e-d3_description/urdf/i3e-d3.urdf.xacro (robot description, xacro)
@@ -78,9 +78,9 @@
         <inertial>
             <origin xyz="0.0 0.0 0.0" rpy="0 0 0"/>
-            <mass value="1.086"/>
+            <mass value="3"/>
             <inertia
-              ixx="7.72416e-3" ixy="0.0" ixz="1.75758e-4"
-              iyy="1.39907e-2" iyz="0.0"
-              izz="1.92855e-2"/>
+              ixx="2.15524e-2" ixy="0.0" ixz="5.5686e-4"
+              iyy="3.76598e-2" iyz="0.0"
+              izz="5.25852e-2"/>
         </inertial>
     </link>
@@ -106,8 +106,8 @@
     <!-- Sensors -->
     <xacro:i3e-d3_lidar>
-        <origin xyz="0.029 0.0 ${base_z_size/2 + 0.025}" rpy="0.0 0.0 0.0"/>
+        <origin xyz="0.0469 0.0 ${base_z_size/2 + 0.025}" rpy="0.0 0.0 0.0"/>
     </xacro:i3e-d3_lidar>
     <xacro:i3e-d3_camera>
-        <origin xyz="-0.026 0.0 ${base_z_size/2 + camera_box_size + 0.025}" rpy="0.0 0.0 0.0"/>
+        <origin xyz="-0.005 0.0 ${base_z_size/2 + camera_box_size + 0.025}" rpy="0.0 0.0 0.0"/>
     </xacro:i3e-d3_camera>
     <gazebo reference="base_link"><material>Gazebo/Yellow</material></gazebo>

Commit message: update map launch files

File: i3e-d3_description/urdf/decorations.urdf.xacro (robot description, xacro)
@@ -6,5 +6,5 @@
                 <origin xyz="0.0 0.0 0.0" rpy="0.0 0.0 0.0"/>
                 <geometry>
-                    <box size="0.05386 0.09604 0.005"/>
+                    <box size="0.106 0.174 0.005"/>
                 </geometry>
             </visual>

File: i3e-d3_description/urdf/i3e-d3_open_manipulator.urdf.xacro (robot description, xacro)
@@ -10,5 +10,5 @@
     <parent link="base_link"/>
     <child link="link1"/>
-    <origin xyz="-0.095 0.0 -0.03" rpy="0.0 0.0 0.0"/>
+    <origin xyz="0.0 -0.2 0.25" rpy="0.0 ${PI} ${PI}"/>
   </joint>
 </robot>
