Commit message: add servo transmitions in urdf

File: i3e-d3_description/urdf/head.urdf.xacro (robot description, xacro)
@@ -2,4 +2,17 @@
 <robot name="i3e-d3_head" xmlns:xacro="http://www.ros.org/wiki/xacro">
   <xacro:property name="base_height" value="0.342"/>
+  <!-- Transmission macro -->
+  <xacro:macro name="SimpleTransmission" params="joint n">
+    <transmission name="tran_${n}">
+      <type>transmission_interface/SimpleTransmission</type>
+      <joint name="${joint}">
+        <hardwareInterface>hardware_interface/PositionJointInterface</hardwareInterface>
+      </joint>
+      <actuator name="servo_${n}">
+        <hardwareInterface>hardware_interface/PositionJointInterface</hardwareInterface>
+        <mechanicalReduction>1</mechanicalReduction>
+      </actuator>
+    </transmission>
+  </xacro:macro>
   <link name="motor_neck_link">
       <visual>
@@ -51,9 +64,12 @@
       </inertial>
   </link>
-  <joint name="neck_joint" type="fixed">
+  <joint name="neck_joint" type="revolute">
       <parent link="motor_neck_link"/>
       <child link="neck_link"/>
+      <axis xyz="0 0 1"/>
+      <limit lower="-1.5707" upper="1.5707" effort="1.0" velocity="2.0"/>
       <origin xyz="0.0 0.0 0.038" rpy="0.0 0.0 0.0"/>
   </joint>
+  <xacro:SimpleTransmission n="neck" joint="neck_joint" />
   <link name="motor_head_link">
       <visual>
@@ -78,9 +94,13 @@
       </inertial>
   </link>
-  <joint name="motor_head_joint" type="fixed">
-      <origin xyz="0.0 -0.02 0.065" rpy="0.0 ${-PI/2} 0.0"/>
-      <parent link="neck_link"/>
-      <child link="motor_head_link"/>
+  <joint name="motor_head_joint" type="revolute">
+    <origin xyz="0.0 -0.02 0.065" rpy="0.0 ${-PI/2} 0.0"/>
+    <parent link="neck_link"/>
+    <child link="motor_head_link"/>
+    <axis xyz="0 0 1"/>
+    <limit lower="-0.2618" upper="0.7854" effort="1.0" velocity="2.0"/>
+    <origin xyz="0.0 0.0 0.038" rpy="0.0 0.0 0.0"/>
   </joint>
+  <xacro:SimpleTransmission n="head" joint="motor_head_joint" />
   <link name="head_link">
       <visual>

Commit message: add head and neck joint control

File: i3e-d3_description/urdf/head.urdf.xacro (robot description, xacro)
@@ -30,5 +30,5 @@
       <inertial>
           <origin xyz="0.0 0.0 0.0" rpy="0.0 0.0 0.0"/>
-              <mass value="0.069"/>
+              <mass value="0.001"/>
               <inertia
                   ixx="1e-6" ixy="0.0" ixz="0.0"
@@ -57,5 +57,5 @@
       <inertial>
           <origin xyz="0.0 0.0 0.0" rpy="0.0 0.0 0.0"/>
-              <mass value="0.05"/>
+              <mass value="0.001"/>
               <inertia
                   ixx="1e-6" ixy="0.0" ixz="0.0"
@@ -68,5 +68,5 @@
       <child link="neck_link"/>
       <axis xyz="0 0 1"/>
-      <limit lower="-1.5707" upper="1.5707" effort="1.0" velocity="2.0"/>
+      <limit lower="-1.5707" upper="1.5707" effort="0.8" velocity="0.2"/>
       <origin xyz="0.0 0.0 0.038" rpy="0.0 0.0 0.0"/>
   </joint>
@@ -87,5 +87,5 @@
       <inertial>
           <origin xyz="0.0 0.0 0.0" rpy="0.0 0.0 0.0"/>
-              <mass value="0.069"/>
+              <mass value="0.001"/>
               <inertia
                   ixx="1e-6" ixy="0.0" ixz="0.0"
@@ -99,5 +99,5 @@
     <child link="motor_head_link"/>
     <axis xyz="0 0 1"/>
-    <limit lower="-0.2618" upper="0.7854" effort="1.0" velocity="2.0"/>
+    <limit lower="-0.2618" upper="0.7854" effort="0.8" velocity="0.2"/>
     <origin xyz="0.0 0.0 0.038" rpy="0.0 0.0 0.0"/>
   </joint>
@@ -118,5 +118,5 @@
       <inertial>
           <origin xyz="0.0 0.0 0.0" rpy="0.0 0.0 0.0"/>
-              <mass value="0.05"/>
+              <mass value="0.001"/>
               <inertia
                   ixx="1e-6" ixy="0.0" ixz="0.0"
@@ -145,5 +145,5 @@
       <inertial>
           <origin xyz="0.0 0.0 0.0" rpy="0.0 0.0 0.0"/>
-              <mass value="0.05"/>
+              <mass value="0.001"/>
               <inertia
                   ixx="1e-6" ixy="0.0" ixz="0.0"

Commit message: caster urf inprog

File: i3e-d3_description/urdf/head.urdf.xacro (robot description, xacro)
@@ -93,5 +93,5 @@
         </inertial>
     </link>
-    <joint name="motor_head_joint" type="revolute">
+    <joint name="head_joint" type="revolute">
         <origin xyz="0.0 -0.02 0.065" rpy="0.0 ${-PI/2} 0.0"/>
         <parent link="neck_link"/>
@@ -100,5 +100,5 @@
         <limit lower="-0.2618" upper="0.7854" effort="0.8" velocity="0.5"/>
     </joint>
-    <xacro:TransmissionServo n="head" joint="motor_head_joint" />
+    <xacro:TransmissionServo n="head" joint="head_joint" />
     <link name="head_link">
         <visual>
@@ -123,5 +123,5 @@
         </inertial>
     </link>
-    <joint name="head_joint" type="fixed">
+    <joint name="motor_head_joint" type="fixed">
         <origin xyz="0.0 -0.04 0.0" rpy="0.0 ${PI/2} 0.0"/>
         <child link="head_link"/>

File: i3e-d3_description/urdf/i3e-d3.urdf.xacro (robot description, xacro)
@@ -69,8 +69,8 @@
     </xacro:i3e-d3_wheel>
     <xacro:i3e-d3_caster prefix="front">
-        <origin xyz="0.11 0.0 ${wheel_z_offset - wheel_radius + 0.0351}" rpy="0.0 0.0 0.0"/>
+        <!--origin xyz="0.11 0.0 ${wheel_z_offset - wheel_radius + 0.0351}" rpy="0.0 0.0 0.0"/-->
     </xacro:i3e-d3_caster>
     <xacro:i3e-d3_caster prefix="back">
-        <origin xyz="-0.11 0.0 ${wheel_z_offset - wheel_radius + 0.0351}" rpy="0.0 0.0 0.0"/>
+        <!--origin xyz="-0.11 0.0 ${wheel_z_offset - wheel_radius + 0.0351}" rpy="0.0 0.0 0.0"/-->
     </xacro:i3e-d3_caster>
     <!-- Sensors -->

File: i3e-d3_description/urdf/wheel.urdf.xacro (robot description, xacro)
@@ -53,29 +53,116 @@
         </transmission>
     </xacro:macro>
-    <xacro:macro name="i3e-d3_caster" params="prefix *joint_pose">
-        <link name="${prefix}_caster_link">
+    <!--xacro:macro name="i3e-d3_caster" params="prefix *joint_pose"-->
+    <xacro:macro name="i3e-d3_caster" params="prefix">
+        <link name="${prefix}_caster_wheel">
             <visual>
-                <origin xyz="0.0 0.0 0.0" rpy="0.0 0.0 0.0"/>
                 <geometry>
-                    <sphere radius="0.035"/>
+                    <sphere radius="0.01"/>
                 </geometry>
+                <material name="black">
+                    <color rgba="0.0 0.0 0.0 1"/>
+                </material>
             </visual>
             <collision>
-                <origin xyz="-0.0 0.0 0.0" rpy="0.0 0.0 0.0"/>
                 <geometry>
-                    <sphere radius="0.035"/>
+                    <sphere radius="0.01"/>
                 </geometry>
             </collision>
+            <inertial>
+                <origin xyz="0.0 0.0 0.0" rpy="0 0 0"/>
+                <mass value="0.01"/>
+                <inertia ixx="4e-7" ixy="0.0" ixz="0.0" iyy="4e-7" iyz="0.0" izz="4e-7"/>
+            </inertial>
         </link>
-        <gazebo reference="${prefix}_caster">
-            <material>Gazebo/DarkGrey</material>
-            <mu1 value="0.0"/>
-            <mu2 value="0.0"/>
-        </gazebo>
-        <joint name="${prefix}_caster" type="fixed">
-            <xacro:insert_block name="joint_pose"/>
+        <link name="${prefix}_caster_support">
+            <visual>
+                <geometry>
+                    <cylinder radius="0.011" length="0.025"/>
+                </geometry>
+                <material name="gray">
+                    <color rgba="0.7 0.7 0.7 1"/>
+                </material>
+            </visual>
+            <collision>
+                <geometry>
+                    <cylinder radius="0.011" length="0.025"/>
+                </geometry>
+            </collision>
+            <inertial>
+                <origin xyz="0.0 0.0 0.0" rpy="0 0 0"/>
+                <mass value="0.01"/>
+                <inertia ixx="8.2333e-7" ixy="0.0" ixz="0.0" iyy="8.2333e-7" iyz="0.0" izz="6.05e-7"/>
+            </inertial>
+        </link>
+        <link name="${prefix}_caster_right">
+            <visual>
+                <geometry>
+                    <box size="0.026 0.003 0.01"/>
+                </geometry>
+                <material name="gray">
+                    <color rgba="0.7 0.7 0.7 1"/>
+                </material>
+            </visual>
+            <collision>
+                <geometry>
+                    <box size="0.026 0.003 0.01"/>
+                </geometry>
+            </collision>
+            <inertial>
+                <origin xyz="0.0 0.0 0.0" rpy="0 0 0"/>
+                <mass value="0.01"/>
+                <inertia ixx="9.0833e-8" ixy="0.0" ixz="0.0" iyy="6.4667e-7" iyz="0.0" izz="5.7083e-7"/>
+            </inertial>
+        </link>
+        <link name="${prefix}_caster_left">
+            <visual>
+                <geometry>
+                    <box size="0.026 0.003 0.01"/>
+                </geometry>
+                <material name="gray">
+                    <color rgba="0.7 0.7 0.7 1"/>
+                </material>
+            </visual>
+            <collision>
+                <geometry>
+                    <box size="0.026 0.003 0.01"/>
+                </geometry>
+            </collision>
+            <inertial>
+                <origin xyz="0.0 0.0 0.0" rpy="0 0 0"/>
+                <mass value="0.01"/>
+                <inertia ixx="9.0833e-8" ixy="0.0" ixz="0.0" iyy="6.4667e-7" iyz="0.0" izz="5.7083e-7"/>
+            </inertial>
+        </link>
+        <joint name="${prefix}_caster_support_joint" type="continuous">
+            <origin xyz="-0.049 0.0 -0.0125" rpy="0 0 0"/>
             <parent link="base_link"/>
-            <child link="${prefix}_caster_link"/>
-            <axis xyz="0 1 0" rpy="0.0 0.0 0.0"/>
+            <child link="${prefix}_caster_support"/>
+            <axis xyz="0 0 1"/>
+        </joint>
+        <joint name="${prefix}_caster_right_joint" type="fixed">
+            <origin xyz="-0.013 0.0115 -0.0125" rpy="0 0 0"/>
+            <parent link="${prefix}_caster_support"/>
+            <child link="${prefix}_caster_right"/>
+            <axis xyz="0 0 1"/>
+        </joint>
+        <joint name="${prefix}_caster_left_joint" type="fixed">
+            <origin xyz="-0.013 -0.0115 -0.0125" rpy="0 0 0"/>
+            <parent link="${prefix}_caster_support"/>
+            <child link="${prefix}_caster_left"/>
+            <axis xyz="0 0 1"/>
+        </joint>
+        <joint name="${prefix}_caster_wheel_right_joint" type="continuous">
+            <origin xyz="-0.013 -0.0115 0.0" rpy="1.5707 0 0"/>
+            <parent link="${prefix}_caster_right"/>
+            <child link="${prefix}_caster_wheel"/>
+            <axis xyz="0 0 1"/>
+        </joint>
+        <joint name="${prefix}_caster_wheel_left_joint" type="continuous">
+            <origin xyz="-0.013 0.0115 0.0" rpy="1.5707 0 0"/>
+            <parent link="${prefix}_caster_left"/>
+            <child link="${prefix}_caster_wheel"/>
+            <axis xyz="0 0 1"/>
+            <mimic joint="${prefix}_caster_wheel_right_joint"/>
         </joint>
     </xacro:macro>
