Commit message: First verry simple URDF

File: i3e-d3_description/urdf/i3e-d3.urdf.xacro (robot description, xacro)
@@ -3,5 +3,5 @@
     <arg name="robot_namespace" default="/"/>
     <xacro:property name="PI" value="3.14159"/>
-    <!-- Included URDF/XACROS Files -->
+    <!-- Included URDF/XACRO Files -->
     <xacro:include filename="$(find i3e-d3_description)/urdf/wheel.urdf.xacro"/>
     <!-- Base size -->
@@ -12,4 +12,9 @@
     <xacro:property name="wheel_length" value="0.06"/>
     <xacro:property name="wheel_radius" value="0.065"/>
+    <!-- Wheel Mounting Positions -->
+    <!-- Need to adjust offsets -->
+    <xacro:property name="wheel_x_offset" value="0.155"/>
+    <xacro:property name="wheel_y_offset" value="${wheel_length/2 + 0.13}"/>
+    <xacro:property name="wheel_z_offset" value="0.0"/>
     <!-- Base link is the center of the robot -->
     <link name="base_link">
@@ -24,11 +29,46 @@
         </visual>
         <collision>
+            <!-- Need to adjust collision origin -->
             <origin xyz="0.0 0.0 0.0" rpy="0.0 0.0 0.0"/>
             <geometry>
-                <box size="0.0 0.0 0.0"/>
+                <box size="${base_x_size} ${base_y_size} ${base_z_size}"/>
             </geometry>
         </collision>
     </link>
+    <!-- Base footprint link is on the ground under the robot-->
+    <link name="base_footprint"/>
+    <joint name="base_footprint_joint" type="fixed">
+        <origin xyz="0.0 ${wheel_vertical_offset - wheel_radius} " rpy="0.0 0.0 0.0"/>
+        <parent link="base_link"/>
+        <child link="base_footprint_link"/>
+    </joint>
+    <!-- Base inertial link -->
+    <link name="inertial_link">
+        <inertial>
+            <!-- Need to adjust all inertia matrix -->
+            <origin xyz="0.0 0.0 0.0" rpy="0.0 0.0 0.0"/>
+            <mass value="3.0"/>
+            <inertia ixx="0.6" ixy="-0.023" ixz="-0.12" iyy="1.73" iyz="-0.0015" izz="2.02"/>
+        </inertial>
+    </link>
+    <joint name="inertial_joint" type="fixed">
+        <parent link="base_link"/>
+        <child link="inertial_link"/>
+        <origin xyz="0.0 0.0 0.0" rpy="0.0 0.0 0.0"/>
+    </joint>
     <!-- I3E-D3 wheel macros -->
+    <xacro:i3e-d3_wheel prefix="front_left">
+        <origin xyz="${wheel_x_offset} ${wheel_y_offset} ${wheel_z_offset}" rpy="0.0 0.0 0.0"/>
+    </xacro:i3e-d3_wheel>
+    <xacro:i3e-d3_wheel prefix="front_right">
+        <origin xyz="${wheel_x_offset} ${-wheel_y_offset} ${wheel_z_offset}" rpy="0.0 0.0 0.0"/>
+    </xacro:i3e-d3_wheel>
+    <xacro:i3e-d3_wheel prefix="rear_left">
+        <origin xyz="${-wheel_x_offset} ${wheel_y_offset} ${wheel_z_offset}" rpy="0.0 0.0 0.0"/>
+    </xacro:i3e-d3_wheel>
+    <xacro:i3e-d3_wheel prefix="rear_right">
+        <origin xyz="${-wheel_x_offset} ${-wheel_y_offset} ${wheel_z_offset}" rpy="0.0 0.0 0.0"/>
+    </xacro:i3e-d3_wheel>
+    <!-- Gazebo ROS Control Plugin -->
     <gazebo>
         <plugin name="gazebo_ros_control" filename="libgazebo_ros_control.so">

File: i3e-d3_description/urdf/wheel.urdf.xacro (robot description, xacro)
@@ -4,4 +4,5 @@
         <link name="${prefix}_wheel_link">
             <inertial>
+                <!-- Need to adjust inertia matrix -->
                 <origin xyz="0.0 0.0 0.0" rpy="0.0 0.0 0.0"/>
                 <mass value="0.16"/>

Commit message: Model spawned in a empty world

File: i3e-d3_description/urdf/i3e-d3.urdf.xacro (robot description, xacro)
@@ -14,7 +14,7 @@
     <!-- Wheel Mounting Positions -->
     <!-- Need to adjust offsets -->
-    <xacro:property name="wheel_x_offset" value="0.155"/>
+    <xacro:property name="wheel_x_offset" value="0.11"/>
     <xacro:property name="wheel_y_offset" value="${wheel_length/2 + 0.13}"/>
-    <xacro:property name="wheel_z_offset" value="0.0"/>
+    <xacro:property name="wheel_z_offset" value="-0.03"/>
     <!-- Base link is the center of the robot -->
     <link name="base_link">
@@ -24,5 +24,5 @@
                 <box size="${base_x_size} ${base_y_size} ${base_z_size}"/>
             </geometry>
-            <material>
+            <material name="blue">
                 <color rgba="0.0 0.0 1.0 1.0"/>
             </material>
@@ -39,7 +39,7 @@
     <link name="base_footprint"/>
     <joint name="base_footprint_joint" type="fixed">
-        <origin xyz="0.0 ${wheel_vertical_offset - wheel_radius} " rpy="0.0 0.0 0.0"/>
+        <origin xyz="0.0 0.0 ${wheel_z_offset - wheel_radius}" rpy="0.0 0.0 0.0"/>
         <parent link="base_link"/>
-        <child link="base_footprint_link"/>
+        <child link="base_footprint"/>
     </joint>
     <!-- Base inertial link -->

File: i3e-d3_description/urdf/wheel.urdf.xacro (robot description, xacro)
@@ -5,19 +5,19 @@
             <inertial>
                 <!-- Need to adjust inertia matrix -->
-                <origin xyz="0.0 0.0 0.0" rpy="0.0 0.0 0.0"/>
+                <origin xyz="0.0 0.0 0.0"/>
                 <mass value="0.16"/>
                 <inertia  ixx="0.02467" ixy="0" ixz="0" iyy="0.04411" iyz="0" izz="0.02467" />
             </inertial>
             <visual>
-                <origin xyz="0.0 0.0 0.0" rpy="0.0 0.0 0.0"/>
+                <origin xyz="0.0 0.0 0.0" rpy="${PI/2} 0.0 0.0"/>
                 <geometry>
                     <cylinder radius="${wheel_radius}" length="${wheel_length}"/>
                 </geometry>
-                <material>
+                <material name="green">
                     <color rgba="0.0 1.0 0.0 1.0"/>
                 </material>
             </visual>
             <collision>
-                <origin xyz="${PI/2} 0.0 0.0" rpy="0.0 0.0 0.0"/>
+                <origin xyz="0.0 0.0 0.0" rpy="${PI/2} 0.0 0.0"/>
                 <geometry>
                     <cylinder radius="${wheel_radius}" length="${wheel_length}"/>
@@ -37,5 +37,5 @@
         <parent link="base_link"/>
         <child link="${prefix}_wheel_link"/>
-        <axis xyz="0 1 0"/>
+        <axis xyz="0 1 0" rpy="0.0 0.0 0.0"/>
     </joint>
     <transmission name="${prefix}_wheel_trans" type="SimpleTransmission">

Commit message: created i3e-d3_tests pkg

File: i3e-d3_description/urdf/i3e-d3.urdf.xacro (robot description, xacro)
@@ -10,6 +10,6 @@
     <xacro:property name="base_z_size" value="0.085"/>
     <!-- Wheel Dimensions -->
-    <xacro:property name="wheel_length" value="0.06"/>
-    <xacro:property name="wheel_radius" value="0.065"/>
+    <xacro:property name="wheel_length" value="0.035"/>
+    <xacro:property name="wheel_radius" value="0.04"/>
     <!-- Wheel Mounting Positions -->
     <!-- Need to adjust offsets -->

Commit message: Implemeting joy control. Not working yet

File: i3e-d3_description/urdf/i3e-d3.urdf.xacro (robot description, xacro)
@@ -48,6 +48,6 @@
             <!-- Need to adjust all inertia matrix -->
             <origin xyz="0.0 0.0 0.0" rpy="0.0 0.0 0.0"/>
-            <mass value="3.0"/>
-            <inertia ixx="0.6" ixy="-0.023" ixz="-0.12" iyy="1.73" iyz="-0.0015" izz="2.02"/>
+            <mass value="7.824"/>
+            <inertia ixx="0.04546" ixy="0.0" ixz="0.0" iyy="0.08458" iyz="0.0" izz="0.1206"/>
         </inertial>
     </link>

File: i3e-d3_description/urdf/wheel.urdf.xacro (robot description, xacro)
@@ -27,9 +27,9 @@
     <!-- Need to adjust gazebo properties -->
     <gazebo reference="{prefix}_wheel_link">
-        <mu1 value="1.0"/>
-        <mu2 value="1.0"/>
-        <kp value="1.0"/>
-        <kd value="1.0"/>
-        <fdir1 value="1 0 0"/>
+        <mu1 value="10.0"/>
+        <mu2 value="10.0"/>
+        <kp value="10.0"/>
+        <kd value="10.0"/>
+        <fdir1 value="10 0 0"/>
     </gazebo>
     <joint name="${prefix}_wheel" type="continuous">

Commit message: Joy control workin, but need to aprimore

File: i3e-d3_description/urdf/i3e-d3.urdf.xacro (robot description, xacro)
@@ -46,8 +46,12 @@
     <link name="inertial_link">
         <inertial>
+            <!-- Center of mass -->
+            <origin xyz="0.012  0.002 0.067" rpy="0 0 0"/>
+            <mass value="16.523"/>
             <!-- Need to adjust all inertia matrix -->
-            <origin xyz="0.0 0.0 0.0" rpy="0.0 0.0 0.0"/>
-            <mass value="7.824"/>
-            <inertia ixx="0.04546" ixy="0.0" ixz="0.0" iyy="0.08458" iyz="0.0" izz="0.1206"/>
+            <inertia
+              ixx="0.3136" ixy="-0.0008" ixz="0.0164"
+              iyy="0.3922" iyz="-0.0009"
+              izz="0.4485"/>
         </inertial>
     </link>
@@ -70,4 +74,7 @@
         <origin xyz="${-wheel_x_offset} ${-wheel_y_offset} ${wheel_z_offset}" rpy="0.0 0.0 0.0"/>
     </xacro:i3e-d3_wheel>
+    <gazebo reference="base_link">
+        <material>Gazebo/Yellow</material>
+    </gazebo>
     <!-- Gazebo ROS Control Plugin -->
     <gazebo>

File: i3e-d3_description/urdf/wheel.urdf.xacro (robot description, xacro)
@@ -7,5 +7,8 @@
                 <origin xyz="0.0 0.0 0.0"/>
                 <mass value="0.16"/>
-                <inertia  ixx="0.02467" ixy="0" ixz="0" iyy="0.04411" iyz="0" izz="0.02467" />
+                <inertia
+                  ixx="0.0013" ixy="0" ixz="0"
+                  iyy="0.0024" iyz="0"
+                  izz="0.0013"/>
             </inertial>
             <visual>
@@ -27,8 +30,9 @@
     <!-- Need to adjust gazebo properties -->
     <gazebo reference="${prefix}_wheel_link">
-        <mu1 value="1.0"/>
-        <mu2 value="1.0"/>
+        <material>Gazebo/DarkGrey</material>
+        <mu1 value="0.5"/>
+        <mu2 value="0.5"/>
         <kp value="10000000.0" />
-        <kd value="1.0" />
+        <kd value="1" />
         <fdir1 value="1 0 0"/>
     </gazebo>

Commit message: adding lidar

File: i3e-d3_description/urdf/i3e-d3.urdf.xacro (robot description, xacro)
@@ -5,4 +5,5 @@
     <!-- Included URDF/XACRO Files -->
     <xacro:include filename="$(find i3e-d3_description)/urdf/wheel.urdf.xacro"/>
+    <xacro:include filename="$(find i3e-d3_description)/urdf/accessories.urdf.xacro"/>
     <!-- Base size -->
     <xacro:property name="base_x_size" value="0.35"/>
@@ -74,7 +75,9 @@
         <origin xyz="${-wheel_x_offset} ${-wheel_y_offset} ${wheel_z_offset}" rpy="0.0 0.0 0.0"/>
     </xacro:i3e-d3_wheel>
-    <gazebo reference="base_link">
-        <material>Gazebo/Yellow</material>
-    </gazebo>
+    <!-- Sensors -->
+    <xacro:i3e-d3_lidar>
+        <origin xyz="0.047 0.0 ${base_z_size/2 + lidar_length/2}" rpy="0.0 0.0 0.0"/>
+    </xacro:i3e-d3_lidar>
+    <gazebo reference="base_link"><material>Gazebo/Yellow</material></gazebo>
     <!-- Gazebo ROS Control Plugin -->
     <gazebo>

File: i3e-d3_description/urdf/wheel.urdf.xacro (robot description, xacro)
@@ -17,7 +17,4 @@
                     <cylinder radius="${wheel_radius}" length="${wheel_length}"/>
                 </geometry>
-                <material name="green">
-                    <color rgba="0.0 1.0 0.0 1.0"/>
-                </material>
             </visual>
             <collision>
@@ -28,28 +25,28 @@
             </collision>
         </link>
-    <!-- Need to adjust gazebo properties -->
-    <gazebo reference="${prefix}_wheel_link">
-        <material>Gazebo/DarkGrey</material>
-        <mu1 value="0.5"/>
-        <mu2 value="0.5"/>
-        <kp value="10000000.0" />
-        <kd value="1" />
-        <fdir1 value="1 0 0"/>
-    </gazebo>
-    <joint name="${prefix}_wheel" type="continuous">
-        <xacro:insert_block name="joint_pose"/>
-        <parent link="base_link"/>
-        <child link="${prefix}_wheel_link"/>
-        <axis xyz="0 1 0" rpy="0.0 0.0 0.0"/>
-    </joint>
-    <transmission name="${prefix}_wheel_trans" type="SimpleTransmission">
-        <type>transmission_interface/SimpleTransmission</type>
-        <actuator name="${prefix}_wheel_motor">
-            <mechanicalReduction>1</mechanicalReduction>
-        </actuator>
-        <joint name="${prefix}_wheel">
-            <hardwareInterface>hardware_interface/VelocityJointInterface</hardwareInterface>
+        <!-- Need to adjust gazebo properties -->
+        <gazebo reference="${prefix}_wheel_link">
+            <material>Gazebo/DarkGrey</material>
+            <mu1 value="0.5"/>
+            <mu2 value="0.5"/>
+            <kp value="10000000.0" />
+            <kd value="1" />
+            <fdir1 value="1 0 0"/>
+        </gazebo>
+        <joint name="${prefix}_wheel" type="continuous">
+            <xacro:insert_block name="joint_pose"/>
+            <parent link="base_link"/>
+            <child link="${prefix}_wheel_link"/>
+            <axis xyz="0 1 0" rpy="0.0 0.0 0.0"/>
         </joint>
-    </transmission>
+        <transmission name="${prefix}_wheel_trans" type="SimpleTransmission">
+            <type>transmission_interface/SimpleTransmission</type>
+            <actuator name="${prefix}_wheel_motor">
+                <mechanicalReduction>1</mechanicalReduction>
+            </actuator>
+            <joint name="${prefix}_wheel">
+                <hardwareInterface>hardware_interface/VelocityJointInterface</hardwareInterface>
+            </joint>
+        </transmission>
     </xacro:macro>
 </robot>

Commit message: new urdf inprog

File: i3e-d3_description/urdf/i3e-d3.urdf.xacro (robot description, xacro)
@@ -7,18 +7,21 @@
     <xacro:include filename="$(find i3e-d3_description)/urdf/accessories.urdf.xacro"/>
     <xacro:include filename="$(find i3e-d3_description)/urdf/decorations.urdf.xacro"/>
-    <!-- Base and support sizes -->
-    <xacro:property name="support_x_size" value="0.31"/>
-    <xacro:property name="support_depth" value="0.009"/>
-    <xacro:property name="base_x_size" value="0.35"/>
-    <xacro:property name="base_y_size" value="0.22"/>
-    <xacro:property name="base_z_size" value="0.085"/>
+    <!-- Base, head and neck sizes -->
+    <xacro:property name="base_x_size" value="0.30"/>
+    <xacro:property name="base_y_size" value="0.30"/>
+    <xacro:property name="base_z_size" value="0.50"/>
+    <xacro:property name="head_x_size" value="0.20"/>
+    <xacro:property name="head_y_size" value="0.20"/>
+    <xacro:property name="head_z_size" value="0.215"/>
+    <xacro:property name="neck_x_size" value="0.08"/>
+    <xacro:property name="neck_y_size" value="0.08"/>
+    <xacro:property name="neck_z_size" value="0.07"/>
     <!-- Wheel Dimensions -->
     <xacro:property name="wheel_length" value="0.06"/>
     <xacro:property name="wheel_radius" value="0.065"/>
     <!-- Wheel Mounting Positions -->
-    <xacro:property name="wheel_xf_offset" value="0.09068514"/>
-    <xacro:property name="wheel_xr_offset" value="0.08931486"/>
+    <xacro:property name="wheel_x_offset" value="-0.05"/>
     <xacro:property name="wheel_y_offset" value="${wheel_length/2 + base_y_size/2 + 0.005}"/>
-    <xacro:property name="wheel_z_offset" value="-0.02805562"/>
+    <xacro:property name="wheel_z_offset" value="-0.25"/>
     <!-- Base link is the center of the robot -->
     <link name="base_link">
@@ -26,5 +29,5 @@
             <origin xyz="0.0 0.0 0.0" rpy="0.0 0.0 0.0"/>
             <geometry>
-                <mesh filename="package://i3e-d3_description/meshes/chassis.stl"/>
+                <mesh filename="package://i3e-d3_description/meshes/body.stl"/>
             </geometry>
             <material name="blue">
@@ -46,32 +49,4 @@
         <child link="base_footprint"/>
     </joint>
-    <!-- Base support link -->
-    <link name="support_link">
-        <inertial>
-            <origin xyz="0.0 0.0 0.0" rpy="0.0 0.0 0.0"/>
-            <mass value="0.4358"/>
-            <inertia
-                ixx="1.7607e-3" ixy="0.0" ixz="0.0"
-                iyy="3.4930e-3" iyz="0.0"
-                izz="5.2477e-3"/>
-        </inertial>
-        <visual>
-            <origin xyz="0.0 0.0 0.0" rpy="0.0 0.0 0.0"/>
-            <geometry>
-                <box size="${support_x_size} ${base_y_size} ${support_depth}"/>
-            </geometry>
-        </visual>
-        <collision>
-            <origin xyz="0.0 0.0 0.0" rpy="0.0 0.0 0.0"/>
-            <geometry>
-                <box size="${support_x_size} ${base_y_size} ${support_depth}"/>
-            </geometry>
-        </collision>
-    </link>
-    <joint name="support_joint" type="fixed">
-        <origin xyz="-0.008 0.0 ${-base_z_size/2}" rpy="0.0 0.0 0.0"/>
-        <parent link="base_link"/>
-        <child link="support_link"/>
-    </joint>
     <!-- Base inertial link -->
     <link name="inertial_link">
@@ -90,17 +65,85 @@
         <origin xyz="0.0 0.0 0.0" rpy="0.0 0.0 0.0"/>
     </joint>
-    <xacro:i3e-d3_decorate/>
+    <link name="neck">
+        <visual>
+            <origin xyz="0.0 0.0 0.0" rpy="0.0 0.0 0.0"/>
+            <geometry>
+                <box size="${neck_x_size} ${neck_y_size} ${neck_z_size}"/>
+            </geometry>
+            <material name="blue">
+                <color rgba="0.0 0.0 1.0 1.0"/>
+            </material>
+        </visual>
+        <collision>
+            <origin xyz="0.0 0.0 0.0" rpy="0.0 0.0 0.0"/>
+            <geometry>
+                <box size="${neck_x_size} ${neck_y_size} ${neck_z_size}"/>
+            </geometry>
+        </collision>
+        <inertial>
+            <origin xyz="0.0 0.0 0.0" rpy="0.0 0.0 0.0"/>
+            <mass value="0.0"/>
+            <inertia ixx="1e-6" ixy="0.0" ixz="0.0" iyy="1e-6" iyz="0.0" izz="1e-6"/>
+        </inertial>
+    </link>
+    <joint name="neck_joint" type="fixed">
+        <parent link="base_link"/>
+        <child link="neck"/>
+        <origin xyz="-0.077 0.0 ${neck_z_size/2 + 0.262}" rpy="0.0 0.0 0.0"/>
+    </joint>
+    <link name="head">
+        <visual>
+            <origin xyz="0.0 0.0 0.0" rpy="0.0 0.0 0.0"/>
+            <geometry>
+                <mesh filename="package://i3e-d3_description/meshes/head.stl"/>
+            </geometry>
+            <material name="blue">
+                <color rgba="0.0 0.0 1.0 1.0"/>
+            </material>
+        </visual>
+        <collision>
+            <origin xyz="0.0 0.0 0.0" rpy="0.0 0.0 0.0"/>
+            <geometry>
+                <box size="${head_x_size} ${head_y_size} ${head_z_size}"/>
+            </geometry>
+        </collision>
+        <inertial>
+            <origin xyz="0.0 0.0 0.0" rpy="0.0 0.0 0.0"/>
+            <mass value="0.0"/>
+            <inertia ixx="1e-6" ixy="0.0" ixz="0.0" iyy="1e-6" iyz="0.0" izz="1e-6"/>
+        </inertial>
+    </link>
+    <joint name="head_joint" type="fixed">
+        <parent link="base_link"/>
+        <child link="head"/>
+        <origin xyz="-0.077 0.0 ${neck_z_size + 0.262 + 0.096}" rpy="0.0 0.0 0.0"/>
+    </joint>
+    <!-- I3E-D3 caster -->
+    <link name="caster">
+        <visual>
+            <origin xyz="0.0 0.0 0.0" rpy="0.0 0.0 0.0"/>
+            <geometry>
+                <box size="0.05 0.05 0.05"/>
+            </geometry>
+        </visual>
+        <collision>
+            <origin xyz="0.0 0.0 0.0" rpy="0.0 0.0 0.0"/>
+            <geometry>
+                <box size="0.05 0.05 0.05"/>
+            </geometry>
+        </collision>
+    </link>
+    <joint name="caster_fixed" type="fixed">
+        <parent link="base_link"/>
+        <child link="caster"/>
+        <origin xyz="0.1 0.0 ${wheel_z_offset - wheel_radius/2}" rpy="0.0 0.0 0.0"/>
+    </joint>
+    <!--xacro:i3e-d3_decorate/-->
     <!-- I3E-D3 wheel macros -->
-    <xacro:i3e-d3_wheel prefix="front_left">
-        <origin xyz="${wheel_xf_offset} ${wheel_y_offset} ${wheel_z_offset}" rpy="0.0 0.0 0.0"/>
+    <xacro:i3e-d3_wheel prefix="left">
+        <origin xyz="${wheel_x_offset} ${wheel_y_offset} ${wheel_z_offset}" rpy="0.0 0.0 0.0"/>
     </xacro:i3e-d3_wheel>
-    <xacro:i3e-d3_wheel prefix="front_right">
-        <origin xyz="${wheel_xf_offset} ${-wheel_y_offset} ${wheel_z_offset}" rpy="0.0 0.0 0.0"/>
-    </xacro:i3e-d3_wheel>
-    <xacro:i3e-d3_wheel prefix="rear_left">
-        <origin xyz="${-wheel_xr_offset} ${wheel_y_offset} ${wheel_z_offset}" rpy="0.0 0.0 0.0"/>
-    </xacro:i3e-d3_wheel>
-    <xacro:i3e-d3_wheel prefix="rear_right">
-        <origin xyz="${-wheel_xr_offset} ${-wheel_y_offset} ${wheel_z_offset}" rpy="0.0 0.0 0.0"/>
+    <xacro:i3e-d3_wheel prefix="right">
+        <origin xyz="${wheel_x_offset} ${-wheel_y_offset} ${wheel_z_offset}" rpy="0.0 0.0 0.0"/>
     </xacro:i3e-d3_wheel>
     <!-- Sensors -->
@@ -112,5 +155,4 @@
     </xacro:i3e-d3_camera>
     <gazebo reference="base_link"><material>Gazebo/Yellow</material></gazebo>
-    <gazebo reference="support_link"><material>Gazebo/DarkYellow</material></gazebo>
     <!-- Gazebo ROS Control Plugin -->
     <gazebo>
