Commit message: i3e-d3_manipulation pkg created

File: i3e-d3_description/urdf/i3e-d3.urdf.xacro (robot description, xacro)
@@ -8,5 +8,5 @@
     <xacro:include filename="$(find i3e-d3_description)/urdf/decorations.urdf.xacro"/>
     <!-- Base, head and neck sizes -->
-    <xacro:property name="base_x_size" value="0.30"/>
+    <xacro:property name="base_x_size" value="0.35"/>
     <xacro:property name="base_y_size" value="0.30"/>
     <xacro:property name="base_z_size" value="0.50"/>
@@ -31,6 +31,6 @@
             <origin xyz="0.0 0.0 0.0" rpy="0.0 0.0 0.0"/>
             <geometry>
-                <mesh filename="package://i3e-d3_description/meshes/body.stl"/>
-                <!--cylinder radius="${base_x_size/2}" length="${base_z_size}"/-->
+                <!--mesh filename="package://i3e-d3_description/meshes/body.stl"/-->
+                <cylinder radius="${base_x_size/2}" length="${base_z_size}"/>
             </geometry>
             <material name="blue">
@@ -169,9 +169,16 @@
     </gazebo>
     <!-- Gazebo ROS Control Plugin -->
-    <gazebo>
+    <!--gazebo>
         <plugin name="gazebo_ros_control" filename="libgazebo_ros_control.so">
             <robotNamespace>$(arg robot_namespace)</robotNamespace>
             <legacyModeNS>true</legacyModeNS>
         </plugin>
-    </gazebo>
+    </gazebo-->
+  <gazebo>
+    <plugin name="gazebo_ros_control" filename="libgazebo_ros_control.so">
+      <controlPeriod>0.001</controlPeriod>
+      <robotSimType>gazebo_ros_control/DefaultRobotHWSim</robotSimType>
+      <legacyModeNS>true</legacyModeNS>
+    </plugin>
+  </gazebo>
 </robot>

File: i3e-d3_manipulation/urdf/open_manipulator.gazebo.xacro (robot description, xacro)
@@ -13,4 +13,6 @@
     </gazebo>
   </xacro:macro>
+  <!-- World -->
+  <gazebo reference="world"/>
   <!-- Link1 -->
   <RefLink ref="link1"/>
@@ -33,11 +35,4 @@
   <!-- ros_control plugin -->
   <gazebo>
-    <plugin name="gazebo_ros_control" filename="libgazebo_ros_control.so">
-      <controlPeriod>0.001</controlPeriod>
-      <robotSimType>gazebo_ros_control/DefaultRobotHWSim</robotSimType>
-      <legacyModeNS>true</legacyModeNS>
-    </plugin>
-  </gazebo>
-  <gazebo>
     <!-- loading plugin: mimic joints works in gazebo now -->
     <plugin name="gazebo_gripper_ros_control" filename="libroboticsgroup_gazebo_mimic_joint_plugin.so">
@@ -46,5 +41,4 @@
       <multiplier>1.0</multiplier>
       <offset>0.0</offset>
-      <hasPID>/gazebo_ros_control/pid_gains/gripper_sub</hasPID>
     </plugin>
   </gazebo>

File: i3e-d3_manipulation/urdf/open_manipulator.transmission.xacro (robot description, xacro)
@@ -9,5 +9,4 @@
       </joint>
       <actuator name="motor${n}">
-        <hardwareInterface>hardware_interface/PositionJointInterface</hardwareInterface>
         <mechanicalReduction>1</mechanicalReduction>
       </actuator>
@@ -22,5 +21,4 @@
       </joint>
       <actuator name="motor${n}">
-        <hardwareInterface>hardware_interface/EffortJointInterface</hardwareInterface>
         <mechanicalReduction>1</mechanicalReduction>
       </actuator>

File: i3e-d3_manipulation/urdf/open_manipulator.urdf.xacro (robot description, xacro)
@@ -1,8 +1,5 @@
 <?xml version="1.0"?>
+<!-- Open_Manipulator Chain -->
 <robot xmlns:xacro="http://ros.org/wiki/xacro">
-  <!-- Include OpenManipulator Gazebo Parameter -->
-  <xacro:include filename="$(find turtlebot3_manipulation_description)/urdf/open_manipulator_x.gazebo.xacro"/>
-  <!-- Include OpenManipulator Transmission -->
-  <xacro:include filename="$(find turtlebot3_manipulation_description)/urdf/open_manipulator_x.transmission.xacro"/>
   <!-- Link 1 -->
   <link name="link1">
@@ -10,15 +7,15 @@
       <origin xyz="0 0 0" rpy="0 0 0"/>
       <geometry>
-        <mesh filename="package://turtlebot3_manipulation_description/meshes/chain_link1.stl" scale="0.001 0.001 0.001"/>
-      </geometry>
-      <material name="grey"/>
-    </visual>
-    <collision>
-      <origin xyz="0 0 0" rpy="0 0 0"/>
-      <geometry>
-        <mesh filename="package://turtlebot3_manipulation_description/meshes/chain_link1.stl" scale="0.001 0.001 0.001"/>
-      </geometry>
-    </collision>
-     <inertial>
+        <mesh filename="package://open_manipulator_description/meshes/chain_link1.stl" scale="0.001 0.001 0.001"/>
+      </geometry>
+      <material name="grey"/>
+    </visual>
+    <collision>
+      <origin xyz="0 0 0" rpy="0 0 0"/>
+      <geometry>
+        <mesh filename="package://open_manipulator_description/meshes/chain_link1.stl" scale="0.001 0.001 0.001"/>
+      </geometry>
+    </collision>
+    <inertial>
       <origin xyz="3.0876154e-04 0.0000000e+00 -1.2176461e-04" />
       <mass value="7.9119962e-02" />
@@ -39,17 +36,17 @@
   <link name="link2">
     <visual>
-      <origin xyz="0 0 0.018" rpy="0 0 0"/>
-      <geometry>
-        <mesh filename="package://turtlebot3_manipulation_description/meshes/chain_link2.stl" scale="0.001 0.001 0.001"/>
-      </geometry>
-      <material name="grey"/>
-    </visual>
-    <collision>
-      <origin xyz="0 0 0.018" rpy="0 0 0"/>
-      <geometry>
-        <mesh filename="package://turtlebot3_manipulation_description/meshes/chain_link2.stl" scale="0.001 0.001 0.001"/>
-      </geometry>
-    </collision>
-     <inertial>
+      <origin xyz="0 0 0.019" rpy="0 0 0"/>
+      <geometry>
+        <mesh filename="package://open_manipulator_description/meshes/chain_link2.stl" scale="0.001 0.001 0.001"/>
+      </geometry>
+      <material name="grey"/>
+    </visual>
+    <collision>
+      <origin xyz="0 0 0.019" rpy="0 0 0"/>
+      <geometry>
+        <mesh filename="package://open_manipulator_description/meshes/chain_link2.stl" scale="0.001 0.001 0.001"/>
+      </geometry>
+    </collision>
+    <inertial>
       <origin xyz="-3.0184870e-04 5.4043684e-04 ${0.018 + 2.9433464e-02}" />
       <mass value="9.8406837e-02" />
@@ -63,5 +60,5 @@
     <parent link="link2"/>
     <child link="link3"/>
-    <origin xyz="0.0 0.0 0.058" rpy="0 0 0"/>
+    <origin xyz="0.0 0.0 0.0595" rpy="0 0 0"/>
     <axis xyz="0 1 0"/>
     <limit velocity="4.8" effort="1" lower="${-pi*0.57}" upper="${pi*0.5}" />
@@ -72,15 +69,15 @@
       <origin xyz="0 0 0" rpy="0 0 0"/>
       <geometry>
-        <mesh filename="package://turtlebot3_manipulation_description/meshes/chain_link3.stl" scale="0.001 0.001 0.001"/>
-      </geometry>
-      <material name="grey"/>
-    </visual>
-    <collision>
-      <origin xyz="0 0 0" rpy="0 0 0"/>
-      <geometry>
-        <mesh filename="package://turtlebot3_manipulation_description/meshes/chain_link3.stl" scale="0.001 0.001 0.001"/>
-      </geometry>
-    </collision>
-     <inertial>
+        <mesh filename="package://open_manipulator_description/meshes/chain_link3.stl" scale="0.001 0.001 0.001"/>
+      </geometry>
+      <material name="grey"/>
+    </visual>
+    <collision>
+      <origin xyz="0 0 0" rpy="0 0 0"/>
+      <geometry>
+        <mesh filename="package://open_manipulator_description/meshes/chain_link3.stl" scale="0.001 0.001 0.001"/>
+      </geometry>
+    </collision>
+    <inertial>
       <origin xyz="1.0308393e-02 3.7743363e-04 1.0170197e-01" />
       <mass value="1.3850917e-01" />
@@ -103,15 +100,15 @@
       <origin xyz="0 0 0" rpy="0 0 0"/>
       <geometry>
-        <mesh filename="package://turtlebot3_manipulation_description/meshes/chain_link4.stl" scale="0.001 0.001 0.001"/>
-      </geometry>
-      <material name="grey"/>
-    </visual>
-    <collision>
-      <origin xyz="0 0 0" rpy="0 0 0"/>
-      <geometry>
-        <mesh filename="package://turtlebot3_manipulation_description/meshes/chain_link4.stl" scale="0.001 0.001 0.001"/>
-      </geometry>
-    </collision>
-     <inertial>
+        <mesh filename="package://open_manipulator_description/meshes/chain_link4.stl" scale="0.001 0.001 0.001"/>
+      </geometry>
+      <material name="grey"/>
+    </visual>
+    <collision>
+      <origin xyz="0 0 0" rpy="0 0 0"/>
+      <geometry>
+        <mesh filename="package://open_manipulator_description/meshes/chain_link4.stl" scale="0.001 0.001 0.001"/>
+      </geometry>
+    </collision>
+    <inertial>
       <origin xyz="9.0909590e-02 3.8929816e-04 2.2413279e-04" />
       <mass value="1.3274562e-01" />
@@ -134,47 +131,20 @@
       <origin xyz="0 0 0" rpy="0 0 0"/>
       <geometry>
-        <mesh filename="package://turtlebot3_manipulation_description/meshes/chain_link5.stl" scale="0.001 0.001 0.001"/>
-      </geometry>
-      <material name="grey"/>
-    </visual>
-    <collision>
-      <origin xyz="0 0 0" rpy="0 0 0"/>
-      <geometry>
-        <mesh filename="package://turtlebot3_manipulation_description/meshes/chain_link5.stl" scale="0.001 0.001 0.001"/>
+        <mesh filename="package://open_manipulator_description/meshes/chain_link5.stl" scale="0.001 0.001 0.001"/>
+      </geometry>
+      <material name="grey"/>
+    </visual>
+    <collision>
+      <origin xyz="0 0 0" rpy="0 0 0"/>
+      <geometry>
+        <mesh filename="package://open_manipulator_description/meshes/chain_link5.stl" scale="0.001 0.001 0.001"/>
       </geometry>
     </collision>
     <inertial>
       <origin xyz="4.4206755e-02 3.6839985e-07 8.9142216e-03" />
-      <!-- <mass value="1.4327573e-01" />
+      <mass value="1.4327573e-01" />
       <inertia ixx="8.0870749e-05" ixy="0.0" ixz="-1.0157896e-06"
                iyy="7.5980465e-05" iyz="0.0"
-               izz="9.3127351e-05" /> -->
-      <mass value="1.0e-03" />
-      <inertia ixx="1.0e-03" ixy="0.0" ixz="0.0"
-               iyy="1.0e-03" iyz="0.0"
-               izz="1.0e-03" />
-    </inertial>
-  </link>
-  <!--  Gripper link -->
-  <link name="gripper_link">
-    <visual>
-      <origin xyz="0.0 0.0 0" rpy="0 0 0"/>
-      <geometry>
-        <mesh filename="package://turtlebot3_manipulation_description/meshes/chain_link_grip_l.stl" scale="0.001 0.001 0.001"/>
-      </geometry>
-      <material name="grey"/>
-    </visual>
-    <collision>
-      <origin xyz="0.0 0.0 0" rpy="0 0 0"/>
-      <geometry>
-        <mesh filename="package://turtlebot3_manipulation_description/meshes/chain_link_grip_l.stl" scale="0.001 0.001 0.001"/>
-      </geometry>
-    </collision>
-    <inertial>
-      <origin xyz="0 0 0" />
-      <mass value="1.0e-03" />
-      <inertia ixx="1.0e-03" ixy="0.0" ixz="0.0"
-               iyy="1.0e-03" iyz="0.0"
-               izz="1.0e-03" />
+               izz="9.3127351e-05" />
     </inertial>
   </link>
@@ -187,17 +157,17 @@
     <limit velocity="4.8" effort="1" lower="-0.010" upper="0.019" />
   </joint>
-  <!--  Gripper link sub -->
-  <link name="gripper_link_sub">
-    <visual>
-      <origin xyz="0.0 -0.0 0" rpy="0 0 0"/>
-      <geometry>
-        <mesh filename="package://turtlebot3_manipulation_description/meshes/chain_link_grip_r.stl" scale="0.001 0.001 0.001"/>
-      </geometry>
-      <material name="grey"/>
-    </visual>
-    <collision>
-      <origin xyz="0.0 -0.0 0" rpy="0 0 0"/>
-      <geometry>
-        <mesh filename="package://turtlebot3_manipulation_description/meshes/chain_link_grip_r.stl" scale="0.001 0.001 0.001"/>
+  <!--  Gripper link -->
+  <link name="gripper_link">
+    <visual>
+      <origin xyz="0.0 0.0 0" rpy="0 0 0"/>
+      <geometry>
+        <mesh filename="package://open_manipulator_description/meshes/chain_link_grip_l.stl" scale="0.001 0.001 0.001"/>
+      </geometry>
+      <material name="grey"/>
+    </visual>
+    <collision>
+      <origin xyz="0.0 0.0 0" rpy="0 0 0"/>
+      <geometry>
+        <mesh filename="package://open_manipulator_description/meshes/chain_link_grip_l.stl" scale="0.001 0.001 0.001"/>
       </geometry>
     </collision>
@@ -219,4 +189,27 @@
     <mimic joint="gripper" multiplier="1"/>
   </joint>
+  <!--  Gripper link sub -->
+  <link name="gripper_link_sub">
+    <visual>
+      <origin xyz="0.0 -0.0 0" rpy="0 0 0"/>
+      <geometry>
+        <mesh filename="package://open_manipulator_description/meshes/chain_link_grip_r.stl" scale="0.001 0.001 0.001"/>
+      </geometry>
+      <material name="grey"/>
+    </visual>
+    <collision>
+      <origin xyz="0.0 -0.0 0" rpy="0 0 0"/>
+      <geometry>
+        <mesh filename="package://open_manipulator_description/meshes/chain_link_grip_r.stl" scale="0.001 0.001 0.001"/>
+      </geometry>
+    </collision>
+    <inertial>
+      <origin xyz="0 0 0" />
+      <mass value="1.0e-03" />
+      <inertia ixx="1.0e-03" ixy="0.0" ixz="0.0"
+               iyy="1.0e-03" iyz="0.0"
+               izz="1.0e-03" />
+    </inertial>
+  </link>
   <!-- end effector joint -->
   <joint name="end_effector_joint" type="fixed">

Commit message: add description.launch

File: i3e-d3_description/urdf/i3e-d3.urdf.xacro (robot description, xacro)
@@ -1,5 +1,5 @@
 <?xml version="1.0"?>
 <robot name="i3e-d3" xmlns:xacro="http://www.ros.org/wiki/xacro">
-    <arg name="robot_namespace" default="i3e_d3"/>
+    <xacro:arg name="robot_namespace" default="i3e_d3"/>
     <xacro:property name="PI" value="3.14159"/>
     <!-- Included URDF/XACRO Files -->
@@ -31,6 +31,6 @@
             <origin xyz="0.0 0.0 0.0" rpy="0.0 0.0 0.0"/>
             <geometry>
-                <!--mesh filename="package://i3e-d3_description/meshes/body.stl"/-->
-                <cylinder radius="${base_x_size/2}" length="${base_z_size}"/>
+                <mesh filename="package://i3e-d3_description/meshes/body.stl"/>
+                <!--cylinder radius="${base_x_size/2}" length="${base_z_size}"/-->
             </geometry>
             <material name="blue">

Commit message: Update i3e-d3.urdf.xacro

File: i3e-d3_description/urdf/i3e-d3.urdf.xacro (robot description, xacro)
@@ -8,7 +8,6 @@
     <xacro:include filename="$(find i3e-d3_description)/urdf/decorations.urdf.xacro"/>
     <!-- Base, head and neck sizes -->
-    <xacro:property name="base_x_size" value="0.35"/>
-    <xacro:property name="base_y_size" value="0.30"/>
-    <xacro:property name="base_z_size" value="0.50"/>
+    <xacro:property name="base_diameter" value="0.315"/>
+    <xacro:property name="base_height" value="0.34"/>
     <xacro:property name="head_x_size" value="0.20"/>
     <xacro:property name="head_y_size" value="0.20"/>
@@ -17,6 +16,6 @@
     <xacro:property name="neck_y_size" value="0.08"/>
     <xacro:property name="neck_z_size" value="0.07"/>
-    <xacro:property name="cog_x" value="-0.013"/>
-    <xacro:property name="cog_z" value="-0.23825904"/>
+    <!--xacro:property name="cog_x" value="-0.013"/-->
+    <!--xacro:property name="cog_z" value="-0.23825904"/-->
     <!-- Wheel Dimensions -->
     <xacro:property name="wheel_length" value="0.0762"/>
@@ -24,6 +23,6 @@
     <!-- Wheel Mounting Positions -->
     <xacro:property name="wheel_x_offset" value="-0.075"/>
-    <xacro:property name="wheel_y_offset" value="${wheel_length/2 + base_y_size/2 + 0.005}"/>
-    <xacro:property name="wheel_z_offset" value="${cog_z + 0.05}"/>
+    <xacro:property name="wheel_y_offset" value="${wheel_length/2 + base_diameter/2 + 0.005}"/>
+    <xacro:property name="wheel_z_offset" value="${-base_height/2 + 0.05}"/>
     <!-- Base link is the center of the robot -->
     <link name="base_link">
@@ -31,6 +30,6 @@
             <origin xyz="0.0 0.0 0.0" rpy="0.0 0.0 0.0"/>
             <geometry>
-                <mesh filename="package://i3e-d3_description/meshes/body.stl"/>
-                <!--cylinder radius="${base_x_size/2}" length="${base_z_size}"/-->
+                <!--mesh filename="package://i3e-d3_description/meshes/body.stl"/-->
+                <cylinder radius="${base_diameter/2}" length="${base_height}"/>
             </geometry>
             <material name="blue">
@@ -41,5 +40,5 @@
             <origin xyz="0.0 0.0 0.0" rpy="0.0 0.0 0.0"/>
             <geometry>
-                <box size="${base_x_size} ${base_y_size} ${base_z_size}"/>
+                <cylinder radius="${base_diameter/2}" length="${base_height}"/>
             </geometry>
         </collision>
@@ -93,5 +92,5 @@
         <parent link="base_link"/>
         <child link="neck"/>
-        <origin xyz="-0.077 0.0 ${neck_z_size/2 + 0.262}" rpy="0.0 0.0 0.0"/>
+        <origin xyz="-0.04 0.0 ${neck_z_size/2 + base_height/2}" rpy="0.0 0.0 0.0"/>
     </joint>
     <link name="head">
@@ -120,5 +119,5 @@
         <parent link="base_link"/>
         <child link="head"/>
-        <origin xyz="-0.077 0.0 ${neck_z_size + 0.262 + 0.096}" rpy="0.0 0.0 0.0"/>
+        <origin xyz="-0.04 0.0 ${neck_z_size + base_height/2 + 0.096}" rpy="0.0 0.0 0.0"/>
     </joint>
     <!-- I3E-D3 caster -->
@@ -152,8 +151,8 @@
     <!-- Sensors -->
     <xacro:i3e-d3_lidar>
-        <origin xyz="0.008 0.0 ${base_z_size + cog_z + 0.025}" rpy="0.0 0.0 0.0"/>
+        <origin xyz="0.045 0.0 ${base_height/2 + 0.025}" rpy="0.0 0.0 0.0"/>
     </xacro:i3e-d3_lidar>
     <xacro:i3e-d3_camera>
-        <origin xyz="0.03 0.0 ${base_z_size + cog_z + neck_z_size + 0.04}" rpy="0.0 0.0 0.0"/>
+        <origin xyz="0.067 0.0 ${base_height/2 + neck_z_size + 0.04}" rpy="0.0 0.0 0.0"/>
     </xacro:i3e-d3_camera>
     <xacro:i3e-d3_imu>

Commit message: urdf inprog

File: i3e-d3_description/urdf/i3e-d3.urdf.xacro (robot description, xacro)
@@ -2,5 +2,5 @@
 <robot name="i3e-d3" xmlns:xacro="http://www.ros.org/wiki/xacro">
     <xacro:arg name="robot_namespace" default="i3e_d3"/>
-    <xacro:arg name="use_open_manipulator" default="true"/>
+    <xacro:arg name="use_open_manipulator" default="false"/>
     <xacro:property name="PI" value="3.14159"/>
     <!-- Included URDF/XACRO Files -->
@@ -9,7 +9,6 @@
     <xacro:include filename="$(find i3e-d3_description)/urdf/decorations.urdf.xacro"/>
     <!-- Base, head and neck sizes -->
-    <xacro:property name="base_x_size" value="0.35"/>
-    <xacro:property name="base_y_size" value="0.30"/>
-    <xacro:property name="base_z_size" value="0.50"/>
+    <xacro:property name="base_radius" value="0.155"/>
+    <xacro:property name="base_height" value="0.342"/>
     <xacro:property name="head_x_size" value="0.20"/>
     <xacro:property name="head_y_size" value="0.20"/>
@@ -18,12 +17,15 @@
     <xacro:property name="neck_y_size" value="0.08"/>
     <xacro:property name="neck_z_size" value="0.07"/>
-    <xacro:property name="cog_x" value="-0.013"/>
-    <xacro:property name="cog_z" value="-0.23825904"/>
+    <!--xacro:property name="cog_x" value="-0.013"/>
+    <xacro:property name="cog_z" value="-0.23825904"/-->
+    <xacro:property name="cog_x" value="0"/>
+    <xacro:property name="cog_z" value="${-base_height/2}"/>
+    <xacro:property name="base_weight" value="0.515"/>
     <!-- Wheel Dimensions -->
     <xacro:property name="wheel_length" value="0.0762"/>
-    <xacro:property name="wheel_radius" value="0.127"/>
+    <xacro:property name="wheel_radius" value="0.088"/>
     <!-- Wheel Mounting Positions -->
-    <xacro:property name="wheel_x_offset" value="-0.075"/>
-    <xacro:property name="wheel_y_offset" value="${wheel_length/2 + base_y_size/2 + 0.005}"/>
+    <xacro:property name="wheel_x_offset" value="0"/>
+    <xacro:property name="wheel_y_offset" value="${wheel_length/2 + base_radius + 0.005}"/>
     <xacro:property name="wheel_z_offset" value="${cog_z + 0.05}"/>
     <!-- Base link is the center of the robot -->
@@ -32,6 +34,5 @@
             <origin xyz="0.0 0.0 0.0" rpy="0.0 0.0 0.0"/>
             <geometry>
-                <mesh filename="package://i3e-d3_description/meshes/body.stl"/>
-                <!--cylinder radius="${base_x_size/2}" length="${base_z_size}"/-->
+                <cylinder radius="${base_radius}" length="${base_height}"/>
             </geometry>
             <material name="blue">
@@ -42,5 +43,5 @@
             <origin xyz="0.0 0.0 0.0" rpy="0.0 0.0 0.0"/>
             <geometry>
-                <box size="${base_x_size} ${base_y_size} ${base_z_size}"/>
+                <cylinder radius="${base_radius}" length="${base_height}"/>
             </geometry>
         </collision>
@@ -123,24 +124,4 @@
         <origin xyz="-0.077 0.0 ${neck_z_size + 0.262 + 0.096}" rpy="0.0 0.0 0.0"/>
     </joint>
-    <!-- I3E-D3 caster -->
-    <link name="caster">
-        <visual>
-            <origin xyz="0.0 0.0 0.0" rpy="0.0 0.0 0.0"/>
-            <geometry>
-                <sphere radius="0.035"/>
-            </geometry>
-        </visual>
-        <collision>
-            <origin xyz="0.0 0.0 0.0" rpy="0.0 0.0 0.0"/>
-            <geometry>
-                <box size="0.07 0.07 0.07"/>
-            </geometry>
-        </collision>
-    </link>
-    <joint name="caster_fixed" type="fixed">
-        <parent link="base_link"/>
-        <child link="caster"/>
-        <origin xyz="0.1 0.0 ${wheel_z_offset - wheel_radius + 0.035}" rpy="0.0 0.0 0.0"/>
-    </joint>
     <xacro:i3e-d3_decorate/>
     <!-- I3E-D3 wheel macros -->
@@ -151,10 +132,16 @@
         <origin xyz="${wheel_x_offset} ${-wheel_y_offset} ${wheel_z_offset}" rpy="0.0 0.0 0.0"/>
     </xacro:i3e-d3_wheel>
+    <xacro:i3e-d3_caster prefix="front">
+        <origin xyz="0.11 0.0 ${wheel_z_offset - wheel_radius + 0.0351}" rpy="0.0 0.0 0.0"/>
+    </xacro:i3e-d3_caster>
+    <xacro:i3e-d3_caster prefix="back">
+        <origin xyz="-0.11 0.0 ${wheel_z_offset - wheel_radius + 0.0351}" rpy="0.0 0.0 0.0"/>
+    </xacro:i3e-d3_caster>
     <!-- Sensors -->
     <xacro:i3e-d3_lidar>
-        <origin xyz="0.008 0.0 ${base_z_size + cog_z + 0.025}" rpy="0.0 0.0 0.0"/>
+        <origin xyz="${base_radius/2} 0.0 ${base_height + cog_z + 0.025}" rpy="0.0 0.0 0.0"/>
     </xacro:i3e-d3_lidar>
     <xacro:i3e-d3_camera>
-        <origin xyz="0.03 0.0 ${base_z_size + cog_z + neck_z_size + 0.04}" rpy="0.0 0.0 0.0"/>
+        <origin xyz="0.03 0.0 ${base_height + cog_z + neck_z_size + 0.04}" rpy="0.0 0.0 0.0"/>
     </xacro:i3e-d3_camera>
     <xacro:i3e-d3_imu>

File: i3e-d3_description/urdf/wheel.urdf.xacro (robot description, xacro)
@@ -53,3 +53,30 @@
         </transmission>
     </xacro:macro>
+    <xacro:macro name="i3e-d3_caster" params="prefix *joint_pose">
+        <link name="${prefix}_caster_link">
+            <visual>
+                <origin xyz="0.0 0.0 0.0" rpy="0.0 0.0 0.0"/>
+                <geometry>
+                    <sphere radius="0.035"/>
+                </geometry>
+            </visual>
+            <collision>
+                <origin xyz="0.0 0.0 0.0" rpy="0.0 0.0 0.0"/>
+                <geometry>
+                    <box size="0.07 0.07 0.07"/>
+                </geometry>
+            </collision>
+        </link>
+        <gazebo reference="${prefix}_caster">
+            <material>Gazebo/DarkGrey</material>
+            <mu1 value="0.0"/>
+            <mu2 value="0.0"/>
+        </gazebo>
+        <joint name="${prefix}_caster" type="fixed">
+            <xacro:insert_block name="joint_pose"/>
+            <parent link="base_link"/>
+            <child link="${prefix}_caster_link"/>
+            <axis xyz="0 1 0" rpy="0.0 0.0 0.0"/>
+        </joint>
+    </xacro:macro>
 </robot>
