Commit message: Update i3e-d3.urdf.xacro

File: i3e-d3_description/urdf/i3e-d3.urdf.xacro (robot description, xacro)
@@ -11,14 +11,4 @@
     <xacro:property name="base_radius" value="0.155"/>
     <xacro:property name="base_height" value="0.342"/>
-    <xacro:property name="head_x_size" value="0.20"/>
-    <xacro:property name="head_y_size" value="0.20"/>
-    <xacro:property name="head_z_size" value="0.215"/>
-    <xacro:property name="neck_x_size" value="0.08"/>
-    <xacro:property name="neck_y_size" value="0.08"/>
-    <xacro:property name="neck_z_size" value="0.07"/>
-    <!--xacro:property name="cog_x" value="-0.013"/>
-    <xacro:property name="cog_z" value="-0.23825904"/-->
-    <xacro:property name="cog_x" value="0"/>
-    <xacro:property name="cog_z" value="${-base_height/2}"/>
     <xacro:property name="base_weight" value="0.515"/>
     <!-- Wheel Dimensions -->
@@ -28,5 +18,5 @@
     <xacro:property name="wheel_x_offset" value="0"/>
     <xacro:property name="wheel_y_offset" value="${wheel_length/2 + base_radius + 0.005}"/>
-    <xacro:property name="wheel_z_offset" value="${cog_z + 0.05}"/>
+    <xacro:property name="wheel_z_offset" value="${-base_height/2 + 0.05}"/>
     <!-- Base link is the center of the robot -->
     <link name="base_link">
@@ -70,59 +60,5 @@
         <origin xyz="0.0 0.0 0.0" rpy="0.0 0.0 0.0"/>
     </joint>
-    <link name="neck">
-        <visual>
-            <origin xyz="0.0 0.0 0.0" rpy="0.0 0.0 0.0"/>
-            <geometry>
-                <box size="${neck_x_size} ${neck_y_size} ${neck_z_size}"/>
-            </geometry>
-            <material name="blue">
-                <color rgba="0.0 0.0 1.0 1.0"/>
-            </material>
-        </visual>
-        <collision>
-            <origin xyz="0.0 0.0 0.0" rpy="0.0 0.0 0.0"/>
-            <geometry>
-                <box size="${neck_x_size} ${neck_y_size} ${neck_z_size}"/>
-            </geometry>
-        </collision>
-        <inertial>
-            <origin xyz="0.0 0.0 0.0" rpy="0.0 0.0 0.0"/>
-            <mass value="0.0"/>
-            <inertia ixx="1e-6" ixy="0.0" ixz="0.0" iyy="1e-6" iyz="0.0" izz="1e-6"/>
-        </inertial>
-    </link>
-    <joint name="neck_joint" type="fixed">
-        <parent link="base_link"/>
-        <child link="neck"/>
-        <origin xyz="-0.077 0.0 ${neck_z_size/2 + 0.262}" rpy="0.0 0.0 0.0"/>
-    </joint>
-    <link name="head">
-        <visual>
-            <origin xyz="0.0 0.0 0.0" rpy="0.0 0.0 0.0"/>
-            <geometry>
-                <mesh filename="package://i3e-d3_description/meshes/head.stl"/>
-            </geometry>
-            <material name="blue">
-                <color rgba="0.0 0.0 1.0 1.0"/>
-            </material>
-        </visual>
-        <collision>
-            <origin xyz="0.0 0.0 0.0" rpy="0.0 0.0 0.0"/>
-            <geometry>
-                <box size="${head_x_size} ${head_y_size} ${head_z_size}"/>
-            </geometry>
-        </collision>
-        <inertial>
-            <origin xyz="0.0 0.0 0.0" rpy="0.0 0.0 0.0"/>
-            <mass value="0.0"/>
-            <inertia ixx="1e-6" ixy="0.0" ixz="0.0" iyy="1e-6" iyz="0.0" izz="1e-6"/>
-        </inertial>
-    </link>
-    <joint name="head_joint" type="fixed">
-        <parent link="base_link"/>
-        <child link="head"/>
-        <origin xyz="-0.077 0.0 ${neck_z_size + 0.262 + 0.096}" rpy="0.0 0.0 0.0"/>
-    </joint>
-    <xacro:i3e-d3_decorate/>
+    <!--xacro:i3e-d3_decorate/-->
     <!-- I3E-D3 wheel macros -->
     <xacro:i3e-d3_wheel prefix="left">
@@ -140,20 +76,19 @@
     <!-- Sensors -->
     <xacro:i3e-d3_lidar>
-        <origin xyz="${base_radius/2} 0.0 ${base_height + cog_z + 0.025}" rpy="0.0 0.0 0.0"/>
+        <origin xyz="${base_radius/2} 0.0 ${base_height/2 + 0.025}" rpy="0.0 0.0 0.0"/>
     </xacro:i3e-d3_lidar>
+    <!--
     <xacro:i3e-d3_camera>
-        <origin xyz="0.03 0.0 ${base_height + cog_z + neck_z_size + 0.04}" rpy="0.0 0.0 0.0"/>
+        <origin xyz="0.03 0.0 ${base_height/2 + neck_z_size + 0.04}" rpy="0.0 0.0 0.0"/>
     </xacro:i3e-d3_camera>
+    -->
     <xacro:i3e-d3_imu>
         <origin xyz="0.0 0.0 0.0" rpy="0.0 0.0 0.0"/>
     </xacro:i3e-d3_imu>
     <gazebo reference="base_link"><material>Gazebo/Yellow</material></gazebo>
+    <!--
     <gazebo reference="neck"><material>Gazebo/DarkGrey</material></gazebo>
     <gazebo reference="head"><material>Gazebo/Yellow</material></gazebo>
-    <gazebo reference="caster">
-        <material>Gazebo/DarkGrey</material>
-        <mu1 value="0.0"/>
-        <mu2 value="0.0"/>
-    </gazebo>
+    -->
     <!-- Gazebo ROS Control Plugin -->
     <!--gazebo>

Commit message: new caster. done

File: i3e-d3_description/urdf/i3e-d3.urdf.xacro (robot description, xacro)
@@ -69,8 +69,8 @@
     </xacro:i3e-d3_wheel>
     <xacro:i3e-d3_caster prefix="front">
-        <!--origin xyz="0.11 0.0 ${wheel_z_offset - wheel_radius + 0.0351}" rpy="0.0 0.0 0.0"/-->
+        <origin xyz="${2*base_radius/3} 0.0 ${-base_height/2}" rpy="0.0 0.0 0.0"/>
     </xacro:i3e-d3_caster>
     <xacro:i3e-d3_caster prefix="back">
-        <!--origin xyz="-0.11 0.0 ${wheel_z_offset - wheel_radius + 0.0351}" rpy="0.0 0.0 0.0"/-->
+        <origin xyz="${-2*base_radius/3} 0.0 ${-base_height/2}" rpy="0.0 0.0 0.0"/>
     </xacro:i3e-d3_caster>
     <!-- Sensors -->

File: i3e-d3_description/urdf/wheel.urdf.xacro (robot description, xacro)
@@ -53,116 +53,87 @@
         </transmission>
     </xacro:macro>
-    <!--xacro:macro name="i3e-d3_caster" params="prefix *joint_pose"-->
-    <xacro:macro name="i3e-d3_caster" params="prefix">
-        <link name="${prefix}_caster_wheel">
+    <xacro:macro name="i3e-d3_caster" params="prefix *joint_pose">
+        <link name="${prefix}_caster_base">
+            <inertial>
+                <origin xyz="0.0 0.0 0.0" rpy="0.0 0.0 0.0"/>
+                <mass value="0.005"/>
+                <inertia ixx="1e-6" ixy="0.0" ixz="0.0" iyy="1e-6" iyz="0.0" izz="1e-6"/>
+            </inertial>
             <visual>
+                <origin xyz="0.0 0.0 0.0" rpy="0.0 0.0 0.0"/>
                 <geometry>
-                    <sphere radius="0.01"/>
+                    <box size="0.05 0.05 0.005"/>
                 </geometry>
-                <material name="black">
-                    <color rgba="0.0 0.0 0.0 1"/>
-                </material>
             </visual>
             <collision>
+                <origin xyz="0.0 0.0 0.0" rpy="0.0 0.0 0.0"/>
                 <geometry>
-                    <sphere radius="0.01"/>
+                    <box size="0.05 0.05 0.005"/>
                 </geometry>
             </collision>
+        </link>
+        <link name="${prefix}_caster_wheel_support">
+            <xacro:property name="caster_wheel_support_box">
+                <geometry>
+                    <box size="0.025 0.0045 0.02"/>
+                </geometry>
+            </xacro:property>
             <inertial>
-                <origin xyz="0.0 0.0 0.0" rpy="0 0 0"/>
-                <mass value="0.01"/>
-                <inertia ixx="4e-7" ixy="0.0" ixz="0.0" iyy="4e-7" iyz="0.0" izz="4e-7"/>
+                <origin xyz="0.0 0.0 0.0" rpy="0.0 0.0 0.0"/>
+                <mass value="0.02"/>
+                <inertia ixx="1e-6" ixy="0.0" ixz="0.0" iyy="1e-6" iyz="0.0" izz="1e-6"/>
             </inertial>
-        </link>
-        <link name="${prefix}_caster_support">
             <visual>
-                <geometry>
-                    <cylinder radius="0.011" length="0.025"/>
-                </geometry>
-                <material name="gray">
-                    <color rgba="0.7 0.7 0.7 1"/>
-                </material>
+                <origin xyz="0.0 0.016 0.0" rpy="0.0 0.0 0.0"/>
+                <xacro:insert_block name="caster_wheel_support_box"/>
+            </visual>
+            <visual>
+                <origin xyz="0.0 -0.016 0.0" rpy="0.0 0.0 0.0"/>
+                <xacro:insert_block name="caster_wheel_support_box"/>
             </visual>
             <collision>
+                <origin xyz="0.0 0.016 0.0" rpy="0.0 0.0 0.0"/>
+                <xacro:insert_block name="caster_wheel_support_box"/>
+            </collision>
+            <collision>
+                <origin xyz="0.0 -0.016 0.0" rpy="0.0 0.0 0.0"/>
+                <xacro:insert_block name="caster_wheel_support_box"/>
+            </collision>
+        </link>
+        <link name="${prefix}_caster_wheel">
+            <inertial>
+                <origin xyz="0.0 0.0 0.0" rpy="0.0 0.0 0.0"/>
+                <mass value="0.01"/>
+                <inertia ixx="1e-6" ixy="0.0" ixz="0.0" iyy="1e-6" iyz="0.0" izz="1e-6"/>
+            </inertial>
+            <visual>
+                <origin xyz="0.0 0.0 0.0" rpy="0.0 0.0 0.0"/>
                 <geometry>
-                    <cylinder radius="0.011" length="0.025"/>
+                    <sphere radius="0.014"/>
+                </geometry>
+            </visual>
+            <collision>
+                <origin xyz="0.0 0.0 0.0" rpy="0.0 0.0 0.0"/>
+                <geometry>
+                    <sphere radius="0.014"/>
                 </geometry>
             </collision>
-            <inertial>
-                <origin xyz="0.0 0.0 0.0" rpy="0 0 0"/>
-                <mass value="0.01"/>
-                <inertia ixx="8.2333e-7" ixy="0.0" ixz="0.0" iyy="8.2333e-7" iyz="0.0" izz="6.05e-7"/>
-            </inertial>
         </link>
-        <link name="${prefix}_caster_right">
-            <visual>
-                <geometry>
-                    <box size="0.026 0.003 0.01"/>
-                </geometry>
-                <material name="gray">
-                    <color rgba="0.7 0.7 0.7 1"/>
-                </material>
-            </visual>
-            <collision>
-                <geometry>
-                    <box size="0.026 0.003 0.01"/>
-                </geometry>
-            </collision>
-            <inertial>
-                <origin xyz="0.0 0.0 0.0" rpy="0 0 0"/>
-                <mass value="0.01"/>
-                <inertia ixx="9.0833e-8" ixy="0.0" ixz="0.0" iyy="6.4667e-7" iyz="0.0" izz="5.7083e-7"/>
-            </inertial>
-        </link>
-        <link name="${prefix}_caster_left">
-            <visual>
-                <geometry>
-                    <box size="0.026 0.003 0.01"/>
-                </geometry>
-                <material name="gray">
-                    <color rgba="0.7 0.7 0.7 1"/>
-                </material>
-            </visual>
-            <collision>
-                <geometry>
-                    <box size="0.026 0.003 0.01"/>
-                </geometry>
-            </collision>
-            <inertial>
-                <origin xyz="0.0 0.0 0.0" rpy="0 0 0"/>
-                <mass value="0.01"/>
-                <inertia ixx="9.0833e-8" ixy="0.0" ixz="0.0" iyy="6.4667e-7" iyz="0.0" izz="5.7083e-7"/>
-            </inertial>
-        </link>
-        <joint name="${prefix}_caster_support_joint" type="continuous">
-            <origin xyz="-0.049 0.0 -0.0125" rpy="0 0 0"/>
+        <joint name="${prefix}_caster_base_joint" type="fixed">
             <parent link="base_link"/>
-            <child link="${prefix}_caster_support"/>
+            <child link="${prefix}_caster_base"/>
+            <xacro:insert_block name="joint_pose"/>
+        </joint>
+        <joint name="${prefix}_caster_wheel_support_joint" type="continuous">
+            <parent link="${prefix}_caster_base"/>
+            <child link="${prefix}_caster_wheel_support"/>
             <axis xyz="0 0 1"/>
+            <origin xyz="0 0 -0.0125" rpy="0 0 0"/>
         </joint>
-        <joint name="${prefix}_caster_right_joint" type="fixed">
-            <origin xyz="-0.013 0.0115 -0.0125" rpy="0 0 0"/>
-            <parent link="${prefix}_caster_support"/>
-            <child link="${prefix}_caster_right"/>
-            <axis xyz="0 0 1"/>
-        </joint>
-        <joint name="${prefix}_caster_left_joint" type="fixed">
-            <origin xyz="-0.013 -0.0115 -0.0125" rpy="0 0 0"/>
-            <parent link="${prefix}_caster_support"/>
-            <child link="${prefix}_caster_left"/>
-            <axis xyz="0 0 1"/>
-        </joint>
-        <joint name="${prefix}_caster_wheel_right_joint" type="continuous">
-            <origin xyz="-0.013 -0.0115 0.0" rpy="1.5707 0 0"/>
-            <parent link="${prefix}_caster_right"/>
+        <joint name="${prefix}_wheel_joint" type="continuous">
+            <parent link="${prefix}_caster_wheel_support"/>
             <child link="${prefix}_caster_wheel"/>
-            <axis xyz="0 0 1"/>
-        </joint>
-        <joint name="${prefix}_caster_wheel_left_joint" type="continuous">
-            <origin xyz="-0.013 0.0115 0.0" rpy="1.5707 0 0"/>
-            <parent link="${prefix}_caster_left"/>
-            <child link="${prefix}_caster_wheel"/>
-            <axis xyz="0 0 1"/>
-            <mimic joint="${prefix}_caster_wheel_right_joint"/>
+            <axis xyz="0 1 0"/>
+            <origin xyz="0 0 -0.011" rpy="0 0 0"/>
         </joint>
     </xacro:macro>

Commit message: Update casters

File: i3e-d3_description/urdf/i3e-d3.urdf.xacro (robot description, xacro)
@@ -6,4 +6,5 @@
     <!-- Included URDF/XACRO Files -->
     <xacro:include filename="$(find i3e-d3_description)/urdf/wheel.urdf.xacro"/>
+    <xacro:include filename="$(find i3e-d3_description)/urdf/caster.urdf.xacro"/>
     <xacro:include filename="$(find i3e-d3_description)/urdf/accessories.urdf.xacro"/>
     <xacro:include filename="$(find i3e-d3_description)/urdf/head.urdf.xacro"/>
@@ -69,10 +70,28 @@
     </xacro:i3e-d3_wheel>
     <!-- I3E-D3 caster macros -->
-    <xacro:i3e-d3_caster prefix="front">
-        <origin xyz="${2*base_radius/3} 0.0 ${-base_height/2}" rpy="0.0 0.0 0.0"/>
-    </xacro:i3e-d3_caster>
-    <xacro:i3e-d3_caster prefix="back">
-        <origin xyz="${-2*base_radius/3} 0.0 ${-base_height/2}" rpy="0.0 0.0 0.0"/>
-    </xacro:i3e-d3_caster>
+    <xacro:i3e-d3_caster prefix="front_caster"
+						 radius="0.025"
+						 x="${2*base_radius/3}"
+						 y="0.0"
+						 z="${-base_height/2 + 0.01}"
+						 roll="0.0"
+						 pitch="0.0"
+						 yaw="0.0"
+						 axis_x="0.577350269"
+						 axis_y="0.577350269"
+						 axis_z="0.577350269"
+						 parent_link="base_link" />
+    <xacro:i3e-d3_caster prefix="rear_caster"
+						 radius="0.025"
+						 x="${-2*base_radius/3}"
+						 y="0.0"
+						 z="${-base_height/2 + 0.01}"
+						 roll="0.0"
+						 pitch="0.0"
+						 yaw="0.0"
+						 axis_x="0.577350269"
+						 axis_y="0.577350269"
+						 axis_z="0.577350269"
+						 parent_link="base_link" />
     <!-- Sensors -->
     <xacro:i3e-d3_camera>

File: i3e-d3_description/urdf/wheel.urdf.xacro (robot description, xacro)
@@ -53,88 +53,3 @@
         </transmission>
     </xacro:macro>
-    <xacro:macro name="i3e-d3_caster" params="prefix *joint_pose">
-        <link name="${prefix}_caster_base">
-            <inertial>
-                <origin xyz="0.0 0.0 0.0" rpy="0.0 0.0 0.0"/>
-                <mass value="0.005"/>
-                <inertia ixx="1e-6" ixy="0.0" ixz="0.0" iyy="1e-6" iyz="0.0" izz="1e-6"/>
-            </inertial>
-            <visual>
-                <origin xyz="0.0 0.0 0.0" rpy="0.0 0.0 0.0"/>
-                <geometry>
-                    <box size="0.05 0.05 0.005"/>
-                </geometry>
-            </visual>
-            <collision>
-                <origin xyz="0.0 0.0 0.0" rpy="0.0 0.0 0.0"/>
-                <geometry>
-                    <box size="0.05 0.05 0.005"/>
-                </geometry>
-            </collision>
-        </link>
-        <link name="${prefix}_caster_wheel_support">
-            <xacro:property name="caster_wheel_support_box">
-                <geometry>
-                    <box size="0.025 0.0045 0.02"/>
-                </geometry>
-            </xacro:property>
-            <inertial>
-                <origin xyz="0.0 0.0 0.0" rpy="0.0 0.0 0.0"/>
-                <mass value="0.02"/>
-                <inertia ixx="1e-6" ixy="0.0" ixz="0.0" iyy="1e-6" iyz="0.0" izz="1e-6"/>
-            </inertial>
-            <visual>
-                <origin xyz="0.0 0.016 0.0" rpy="0.0 0.0 0.0"/>
-                <xacro:insert_block name="caster_wheel_support_box"/>
-            </visual>
-            <visual>
-                <origin xyz="0.0 -0.016 0.0" rpy="0.0 0.0 0.0"/>
-                <xacro:insert_block name="caster_wheel_support_box"/>
-            </visual>
-            <collision>
-                <origin xyz="0.0 0.016 0.0" rpy="0.0 0.0 0.0"/>
-                <xacro:insert_block name="caster_wheel_support_box"/>
-            </collision>
-            <collision>
-                <origin xyz="0.0 -0.016 0.0" rpy="0.0 0.0 0.0"/>
-                <xacro:insert_block name="caster_wheel_support_box"/>
-            </collision>
-        </link>
-        <link name="${prefix}_caster_wheel">
-            <inertial>
-                <origin xyz="0.0 0.0 0.0" rpy="0.0 0.0 0.0"/>
-                <mass value="0.01"/>
-                <inertia ixx="1e-6" ixy="0.0" ixz="0.0" iyy="1e-6" iyz="0.0" izz="1e-6"/>
-            </inertial>
-            <visual>
-                <origin xyz="0.0 0.0 0.0" rpy="0.0 0.0 0.0"/>
-                <geometry>
-                    <sphere radius="0.014"/>
-                </geometry>
-            </visual>
-            <collision>
-                <origin xyz="0.0 0.0 0.0" rpy="0.0 0.0 0.0"/>
-                <geometry>
-                    <sphere radius="0.014"/>
-                </geometry>
-            </collision>
-        </link>
-        <joint name="${prefix}_caster_base_joint" type="fixed">
-            <parent link="base_link"/>
-            <child link="${prefix}_caster_base"/>
-            <xacro:insert_block name="joint_pose"/>
-        </joint>
-        <joint name="${prefix}_caster_wheel_support_joint" type="continuous">
-            <parent link="${prefix}_caster_base"/>
-            <child link="${prefix}_caster_wheel_support"/>
-            <axis xyz="0 0 1"/>
-            <origin xyz="0 0 -0.0125" rpy="0 0 0"/>
-        </joint>
-        <joint name="${prefix}_wheel_joint" type="continuous">
-            <parent link="${prefix}_caster_wheel_support"/>
-            <child link="${prefix}_caster_wheel"/>
-            <axis xyz="0 1 0"/>
-            <origin xyz="0 0 -0.011" rpy="0 0 0"/>
-        </joint>
-    </xacro:macro>
 </robot>
