Commit message: Added camera and Lidar

File: i3e-d3_description/urdf/accessories.urdf.xacro (robot description, xacro)
@@ -3,4 +3,6 @@
     <xacro:property name="lidar_radius" value="0.055"/>
     <xacro:property name="lidar_length" value="0.05"/>
+    <xacro:property name="camera_box_size" value="0.035"/>
+    <arg name="robot_namespace" default="/"/>
     <!-- 3irobotix LIDAR -->
     <xacro:macro name="i3e-d3_lidar" params="*joint_pose">
@@ -17,10 +19,4 @@
                 </geometry>
             </visual>
-            <collision>
-                <origin xyz="0.0 0.0 0.0" rpy="0.0 0.0 0.0"/>
-                <geometry>
-                    <cylinder radius="0.1" length="0.05"/>
-                </geometry>
-            </collision>
         </link>
         <joint name="lidar_joint" type="fixed">
@@ -29,12 +25,10 @@
             <xacro:insert_block name="joint_pose"/>
         </joint>
-        <gazebo reference="3irobotix_lidar">
-            <material>Gazebo/Black</material>
-        </gazebo>
+        <gazebo reference="3irobotix_lidar"><material>Gazebo/Black</material></gazebo>
          <!-- Laser Plugin -->
         <gazebo reference="3irobotix_lidar">
-            <sensor type="gpu_ray" name="head_hokuyo_sensor">
+            <sensor type="ray" name="lidar_sensor">
               <pose>0 0 0 0 0 0</pose>
-              <visualize>false</visualize>
+              <visualize>true</visualize>
               <update_rate>40</update_rate>
               <ray>
@@ -43,11 +37,11 @@
                     <samples>720</samples>
                     <resolution>1</resolution>
-                    <min_angle>-1.570796</min_angle>
-                    <max_angle>1.570796</max_angle>
+                    <min_angle>-2.35619</min_angle>
+                    <max_angle>2.35619</max_angle>
                   </horizontal>
                 </scan>
                 <range>
                   <min>0.10</min>
-                  <max>30.0</max>
+                  <max>4.0</max>
                   <resolution>0.01</resolution>
                 </range>
@@ -62,6 +56,7 @@
                 </noise>
               </ray>
-              <plugin name="gazebo_ros_head_hokuyo_controller" filename="libgazebo_ros_gpu_laser.so">
-                <topicName>/i3e-d3/laser/scan</topicName>
+              <plugin name="gazebo_ros_head_hokuyo_controller" filename="libgazebo_ros_laser.so">
+                <robotNamespace>$(arg robot_namespace)</robotNamespace>
+                <topicName>/i3e_d3/laser/scan</topicName>
                 <frameName>3irobotix_lidar</frameName>
               </plugin>
@@ -69,3 +64,72 @@
         </gazebo>
     </xacro:macro>
+    <!-- Camera -->
+    <xacro:macro name="i3e-d3_camera" params="*joint_pose">
+        <link name="camera_link">
+            <inertial>
+                <origin xyz="0.0 0.0 0.0" rpy="0.0 0.0 0.0"/>
+                <mass value="0.05"/>
+                <inertia ixx="1e-6" ixy="0.0" ixz="0.0" iyy="1e-6" iyz="0.0" izz="1e-6"/>
+            </inertial>
+            <visual>
+                <origin xyz="0.0 0.0 0.0" rpy="0.0 0.0 0.0"/>
+                <geometry>
+                    <box size="${camera_box_size} ${camera_box_size} ${camera_box_size}"/>
+                </geometry>
+            </visual>
+            <collision>
+                <origin xyz="0.0 0.0 0.0" rpy="0.0 0.0 0.0"/>
+                <geometry>
+                    <box size="${camera_box_size} ${camera_box_size} ${camera_box_size}"/>
+                </geometry>
+            </collision>
+        </link>
+        <joint name="camera_joint" type="fixed">
+            <parent link="base_link"/>
+            <child link="camera_link"/>
+            <xacro:insert_block name="joint_pose"/>
+        </joint>
+        <gazebo reference="camera_link"><material>Gazebo/Red</material></gazebo>
+        <!-- Camera Plugin -->
+        <gazebo reference="camera_link">
+          <sensor type="camera" name="camera">
+            <update_rate>30.0</update_rate>
+            <camera name="head">
+              <horizontal_fov>1.3962634</horizontal_fov>
+              <image>
+                <width>800</width>
+                <height>800</height>
+                <format>R8G8B8</format>
+              </image>
+              <clip>
+                <near>0.02</near>
+                <far>300</far>
+              </clip>
+              <noise>
+                <type>gaussian</type>
+                <!-- Noise is sampled independently per pixel on each frame.
+                     That pixel's noise value is added to each of its color
+                     channels, which at that point lie in the range [0,1]. -->
+                <mean>0.0</mean>
+                <stddev>0.007</stddev>
+              </noise>
+            </camera>
+            <plugin name="camera_controller" filename="libgazebo_ros_camera.so">
+              <robotNamespace>$(arg robot_namespace)</robotNamespace>
+              <alwaysOn>true</alwaysOn>
+              <updateRate>0.0</updateRate>
+              <cameraName>i3e_d3/camera1</cameraName>
+              <imageTopicName>image_raw</imageTopicName>
+              <cameraInfoTopicName>camera_info</cameraInfoTopicName>
+              <frameName>camera_link</frameName>
+              <hackBaseline>0.07</hackBaseline>
+              <distortionK1>0.0</distortionK1>
+              <distortionK2>0.0</distortionK2>
+              <distortionK3>0.0</distortionK3>
+              <distortionT1>0.0</distortionT1>
+              <distortionT2>0.0</distortionT2>
+            </plugin>
+          </sensor>
+        </gazebo>
+    </xacro:macro>
 </robot>

File: i3e-d3_description/urdf/i3e-d3.urdf.xacro (robot description, xacro)
@@ -79,4 +79,7 @@
         <origin xyz="0.047 0.0 ${base_z_size/2 + lidar_length/2}" rpy="0.0 0.0 0.0"/>
     </xacro:i3e-d3_lidar>
+    <xacro:i3e-d3_camera>
+        <origin xyz="0.047 0.0 ${base_z_size/2 + lidar_length + camera_box_size/2}" rpy="0.0 0.0 0.0"/>
+    </xacro:i3e-d3_camera>
     <gazebo reference="base_link"><material>Gazebo/Yellow</material></gazebo>
     <!-- Gazebo ROS Control Plugin -->

Commit message: Updated URDF

File: i3e-d3_description/urdf/accessories.urdf.xacro (robot description, xacro)
@@ -1,7 +1,5 @@
 <?xml version="1.0"?>
 <robot xmlns:xacro="http://www.ros.org/wiki/xacro" name="i3e-d3_accessories">
-    <xacro:property name="lidar_radius" value="0.055"/>
-    <xacro:property name="lidar_length" value="0.05"/>
-    <xacro:property name="camera_box_size" value="0.035"/>
+    <xacro:property name="camera_box_size" value="0.02"/>
     <arg name="robot_namespace" default="/"/>
     <!-- 3irobotix LIDAR -->
@@ -16,5 +14,5 @@
                 <origin xyz="0.0 0.0 0.0" rpy="0.0 0.0 0.0"/>
                 <geometry>
-                    <cylinder radius="${lidar_radius}" length="${lidar_length}"/>
+                    <mesh filename="package://i3e-d3_description/meshes/lidar.stl"/>
                 </geometry>
             </visual>

File: i3e-d3_description/urdf/decorations.urdf.xacro (robot description, xacro)
@@ -1,4 +1,27 @@
 <?xml version="1.0"?>
 <robot xmlns:xacro="http://www.ros.org/wiki/xacro" name="i3e-d3_decorations">
-    <!-- To Do-->
+    <xacro:macro name="i3e-d3_decorate">
+        <link name="display_link">
+            <visual>
+                <origin xyz="0.0 0.0 0.0" rpy="0.0 0.0 0.0"/>
+                <geometry>
+                    <box size="0.05386 0.09604 0.005"/>
+                </geometry>
+            </visual>
+            <inertial>
+                <origin xyz="0.0 0.0 0.0" rpy="0.0 0.0 0.0"/>
+                <mass value="0.141"/>
+                <inertia
+                    ixx="1e-6" ixy="0.0" ixz="0.0"
+                    iyy="1e-6" iyz="0.0"
+                    izz="1e-6"/>
+            </inertial>
+        </link>
+        <joint name="display_joint" type="fixed">
+            <origin xyz="0.15 0.0 0.028" rpy="0.0 ${28.74*PI/180} 0.0"/>
+            <parent link="base_link"/>
+            <child link="display_link"/>
+        </joint>
+        <gazebo reference="display_link"><material>Gazebo/White</material></gazebo>
+    </xacro:macro>
 </robot>

File: i3e-d3_description/urdf/i3e-d3.urdf.xacro (robot description, xacro)
@@ -6,16 +6,19 @@
     <xacro:include filename="$(find i3e-d3_description)/urdf/wheel.urdf.xacro"/>
     <xacro:include filename="$(find i3e-d3_description)/urdf/accessories.urdf.xacro"/>
-    <!-- Base size -->
+    <xacro:include filename="$(find i3e-d3_description)/urdf/decorations.urdf.xacro"/>
+    <!-- Base and support sizes -->
+    <xacro:property name="support_x_size" value="0.31"/>
+    <xacro:property name="support_depth" value="0.009"/>
     <xacro:property name="base_x_size" value="0.35"/>
-    <xacro:property name="base_y_size" value="0.25"/>
+    <xacro:property name="base_y_size" value="0.22"/>
     <xacro:property name="base_z_size" value="0.085"/>
     <!-- Wheel Dimensions -->
-    <xacro:property name="wheel_length" value="0.035"/>
-    <xacro:property name="wheel_radius" value="0.04"/>
+    <xacro:property name="wheel_length" value="0.06"/>
+    <xacro:property name="wheel_radius" value="0.065"/>
     <!-- Wheel Mounting Positions -->
-    <!-- Need to adjust offsets -->
-    <xacro:property name="wheel_x_offset" value="0.11"/>
-    <xacro:property name="wheel_y_offset" value="${wheel_length/2 + 0.13}"/>
-    <xacro:property name="wheel_z_offset" value="-0.03"/>
+    <xacro:property name="wheel_xf_offset" value="0.09068514"/>
+    <xacro:property name="wheel_xr_offset" value="0.08931486"/>
+    <xacro:property name="wheel_y_offset" value="${wheel_length/2 + base_y_size/2 + 0.005}"/>
+    <xacro:property name="wheel_z_offset" value="-0.02805562"/>
     <!-- Base link is the center of the robot -->
     <link name="base_link">
@@ -23,5 +26,5 @@
             <origin xyz="0.0 0.0 0.0" rpy="0.0 0.0 0.0"/>
             <geometry>
-                <box size="${base_x_size} ${base_y_size} ${base_z_size}"/>
+                <mesh filename="package://i3e-d3_description/meshes/chassis.stl"/>
             </geometry>
             <material name="blue">
@@ -30,5 +33,4 @@
         </visual>
         <collision>
-            <!-- Need to adjust collision origin -->
             <origin xyz="0.0 0.0 0.0" rpy="0.0 0.0 0.0"/>
             <geometry>
@@ -44,15 +46,41 @@
         <child link="base_footprint"/>
     </joint>
+    <!-- Base support link -->
+    <link name="support_link">
+        <inertial>
+            <origin xyz="0.0 0.0 0.0" rpy="0.0 0.0 0.0"/>
+            <mass value="0.4358"/>
+            <inertia
+                ixx="1.7607e-3" ixy="0.0" ixz="0.0"
+                iyy="3.4930e-3" iyz="0.0"
+                izz="5.2477e-3"/>
+        </inertial>
+        <visual>
+            <origin xyz="0.0 0.0 0.0" rpy="0.0 0.0 0.0"/>
+            <geometry>
+                <box size="${support_x_size} ${base_y_size} ${support_depth}"/>
+            </geometry>
+        </visual>
+        <collision>
+            <origin xyz="0.0 0.0 0.0" rpy="0.0 0.0 0.0"/>
+            <geometry>
+                <box size="${support_x_size} ${base_y_size} ${support_depth}"/>
+            </geometry>
+        </collision>
+    </link>
+    <joint name="support_joint" type="fixed">
+        <origin xyz="-0.008 0.0 ${-base_z_size/2}" rpy="0.0 0.0 0.0"/>
+        <parent link="base_link"/>
+        <child link="support_link"/>
+    </joint>
     <!-- Base inertial link -->
     <link name="inertial_link">
         <inertial>
-            <!-- Center of mass -->
-            <origin xyz="0.012  0.002 0.067" rpy="0 0 0"/>
-            <mass value="16.523"/>
-            <!-- Need to adjust all inertia matrix -->
+            <origin xyz="0.0 0.0 0.0" rpy="0 0 0"/>
+            <mass value="1.086"/>
             <inertia
-              ixx="0.3136" ixy="-0.0008" ixz="0.0164"
-              iyy="0.3922" iyz="-0.0009"
-              izz="0.4485"/>
+              ixx="7.72416e-3" ixy="0.0" ixz="1.75758e-4"
+              iyy="1.39907e-2" iyz="0.0"
+              izz="1.92855e-2"/>
         </inertial>
     </link>
@@ -62,25 +90,27 @@
         <origin xyz="0.0 0.0 0.0" rpy="0.0 0.0 0.0"/>
     </joint>
+    <xacro:i3e-d3_decorate/>
     <!-- I3E-D3 wheel macros -->
     <xacro:i3e-d3_wheel prefix="front_left">
-        <origin xyz="${wheel_x_offset} ${wheel_y_offset} ${wheel_z_offset}" rpy="0.0 0.0 0.0"/>
+        <origin xyz="${wheel_xf_offset} ${wheel_y_offset} ${wheel_z_offset}" rpy="0.0 0.0 0.0"/>
     </xacro:i3e-d3_wheel>
     <xacro:i3e-d3_wheel prefix="front_right">
-        <origin xyz="${wheel_x_offset} ${-wheel_y_offset} ${wheel_z_offset}" rpy="0.0 0.0 0.0"/>
+        <origin xyz="${wheel_xf_offset} ${-wheel_y_offset} ${wheel_z_offset}" rpy="0.0 0.0 0.0"/>
     </xacro:i3e-d3_wheel>
     <xacro:i3e-d3_wheel prefix="rear_left">
-        <origin xyz="${-wheel_x_offset} ${wheel_y_offset} ${wheel_z_offset}" rpy="0.0 0.0 0.0"/>
+        <origin xyz="${-wheel_xr_offset} ${wheel_y_offset} ${wheel_z_offset}" rpy="0.0 0.0 0.0"/>
     </xacro:i3e-d3_wheel>
     <xacro:i3e-d3_wheel prefix="rear_right">
-        <origin xyz="${-wheel_x_offset} ${-wheel_y_offset} ${wheel_z_offset}" rpy="0.0 0.0 0.0"/>
+        <origin xyz="${-wheel_xr_offset} ${-wheel_y_offset} ${wheel_z_offset}" rpy="0.0 0.0 0.0"/>
     </xacro:i3e-d3_wheel>
     <!-- Sensors -->
     <xacro:i3e-d3_lidar>
-        <origin xyz="0.047 0.0 ${base_z_size/2 + lidar_length/2}" rpy="0.0 0.0 0.0"/>
+        <origin xyz="0.029 0.0 ${base_z_size/2}" rpy="0.0 0.0 0.0"/>
     </xacro:i3e-d3_lidar>
     <xacro:i3e-d3_camera>
-        <origin xyz="0.047 0.0 ${base_z_size/2 + lidar_length + camera_box_size/2}" rpy="0.0 0.0 0.0"/>
+        <origin xyz="-0.026 0.0 ${base_z_size/2 + camera_box_size + 0.025}" rpy="0.0 0.0 0.0"/>
     </xacro:i3e-d3_camera>
     <gazebo reference="base_link"><material>Gazebo/Yellow</material></gazebo>
+    <gazebo reference="support_link"><material>Gazebo/DarkYellow</material></gazebo>
     <!-- Gazebo ROS Control Plugin -->
     <gazebo>

File: i3e-d3_description/urdf/wheel.urdf.xacro (robot description, xacro)
@@ -6,14 +6,14 @@
                 <!-- Need to adjust inertia matrix -->
                 <origin xyz="0.0 0.0 0.0"/>
-                <mass value="0.16"/>
+                <mass value="0.160"/>
                 <inertia
-                  ixx="0.0013" ixy="0" ixz="0"
-                  iyy="0.0024" iyz="0"
-                  izz="0.0013"/>
+                  ixx="2.70474e-4" ixy="0.0" ixz="0.0"
+                  iyy="4.38099e-4" iyz="0.0"
+                  izz="2.70474e-4"/>
             </inertial>
             <visual>
-                <origin xyz="0.0 0.0 0.0" rpy="${PI/2} 0.0 0.0"/>
+                <origin xyz="0.0 0.0 0.0" rpy="0.0 0.0 0.0"/>
                 <geometry>
-                    <cylinder radius="${wheel_radius}" length="${wheel_length}"/>
+                    <mesh filename="package://i3e-d3_description/meshes/wheel_130x60.stl"/>
                 </geometry>
             </visual>

Commit message: implementing gmapping

File: i3e-d3_description/urdf/accessories.urdf.xacro (robot description, xacro)
@@ -12,5 +12,5 @@
             </inertial>
             <visual>
-                <origin xyz="0.0 0.0 0.0" rpy="0.0 0.0 0.0"/>
+                <origin xyz="0.0 0.0 -0.025" rpy="0.0 0.0 0.0"/>
                 <geometry>
                     <mesh filename="package://i3e-d3_description/meshes/lidar.stl"/>
@@ -41,5 +41,5 @@
                 <range>
                   <min>0.10</min>
-                  <max>4.0</max>
+                  <max>6.5</max>
                   <resolution>0.01</resolution>
                 </range>

File: i3e-d3_description/urdf/i3e-d3.urdf.xacro (robot description, xacro)
@@ -106,5 +106,5 @@
     <!-- Sensors -->
     <xacro:i3e-d3_lidar>
-        <origin xyz="0.029 0.0 ${base_z_size/2}" rpy="0.0 0.0 0.0"/>
+        <origin xyz="0.029 0.0 ${base_z_size/2 + 0.025}" rpy="0.0 0.0 0.0"/>
     </xacro:i3e-d3_lidar>
     <xacro:i3e-d3_camera>

File: i3e-d3_description/urdf/wheel.urdf.xacro (robot description, xacro)
@@ -17,5 +17,5 @@
                 <origin xyz="0.0 0.0 0.0" rpy="0.0 0.0 0.0"/>
                 <geometry>
-                    <mesh filename="package://i3e-d3_description/meshes/wheel_husky.stl"
+                    <mesh filename="package://i3e-d3_description/meshes/wheel_husky.dae"
                           scale="${wheel_radius/husky_wheel_radius} ${wheel_length/husky_wheel_length} ${wheel_radius/husky_wheel_radius}"/>
                 </geometry>

Commit message: finishing new urdf

File: i3e-d3_description/urdf/accessories.urdf.xacro (robot description, xacro)
@@ -1,5 +1,5 @@
 <?xml version="1.0"?>
 <robot xmlns:xacro="http://www.ros.org/wiki/xacro" name="i3e-d3_accessories">
-    <xacro:property name="camera_box_size" value="0.02"/>
+    <xacro:property name="camera_box_size" value="0.04"/>
     <arg name="robot_namespace" default="/"/>
     <!-- 3irobotix LIDAR -->
@@ -28,5 +28,5 @@
             <sensor type="ray" name="lidar_sensor">
               <pose>0 0 0 0 0 0</pose>
-              <visualize>false</visualize>
+              <visualize>true</visualize>
               <update_rate>40</update_rate>
               <ray>
@@ -41,5 +41,5 @@
                 <range>
                   <min>0.10</min>
-                  <max>6.5</max>
+                  <max>8.0</max>
                   <resolution>0.01</resolution>
                 </range>

File: i3e-d3_description/urdf/decorations.urdf.xacro (robot description, xacro)
@@ -19,6 +19,6 @@
         </link>
         <joint name="display_joint" type="fixed">
-            <origin xyz="0.16 0.0 0.019" rpy="0.0 ${40*PI/180} 0.0"/>
-            <parent link="base_link"/>
+            <origin xyz="0.062 0.0 0.054" rpy="0.0 ${53*PI/180} 0.0"/>
+            <parent link="head"/>
             <child link="display_link"/>
         </joint>

File: i3e-d3_description/urdf/i3e-d3.urdf.xacro (robot description, xacro)
@@ -17,11 +17,13 @@
     <xacro:property name="neck_y_size" value="0.08"/>
     <xacro:property name="neck_z_size" value="0.07"/>
+    <xacro:property name="cog_x" value="-0.013"/>
+    <xacro:property name="cog_z" value="-0.23825904"/>
     <!-- Wheel Dimensions -->
-    <xacro:property name="wheel_length" value="0.06"/>
-    <xacro:property name="wheel_radius" value="0.065"/>
+    <xacro:property name="wheel_length" value="0.0762"/>
+    <xacro:property name="wheel_radius" value="0.127"/>
     <!-- Wheel Mounting Positions -->
-    <xacro:property name="wheel_x_offset" value="-0.05"/>
+    <xacro:property name="wheel_x_offset" value="-0.075"/>
     <xacro:property name="wheel_y_offset" value="${wheel_length/2 + base_y_size/2 + 0.005}"/>
-    <xacro:property name="wheel_z_offset" value="-0.25"/>
+    <xacro:property name="wheel_z_offset" value="${cog_z + 0.05}"/>
     <!-- Base link is the center of the robot -->
     <link name="base_link">
@@ -124,5 +126,5 @@
             <origin xyz="0.0 0.0 0.0" rpy="0.0 0.0 0.0"/>
             <geometry>
-                <box size="0.05 0.05 0.05"/>
+                <sphere radius="0.035"/>
             </geometry>
         </visual>
@@ -130,5 +132,5 @@
             <origin xyz="0.0 0.0 0.0" rpy="0.0 0.0 0.0"/>
             <geometry>
-                <box size="0.05 0.05 0.05"/>
+                <box size="0.07 0.07 0.07"/>
             </geometry>
         </collision>
@@ -137,7 +139,7 @@
         <parent link="base_link"/>
         <child link="caster"/>
-        <origin xyz="0.1 0.0 ${wheel_z_offset - wheel_radius/2}" rpy="0.0 0.0 0.0"/>
+        <origin xyz="0.1 0.0 ${wheel_z_offset - wheel_radius + 0.035}" rpy="0.0 0.0 0.0"/>
     </joint>
-    <!--xacro:i3e-d3_decorate/-->
+    <xacro:i3e-d3_decorate/>
     <!-- I3E-D3 wheel macros -->
     <xacro:i3e-d3_wheel prefix="left">
@@ -149,10 +151,17 @@
     <!-- Sensors -->
     <xacro:i3e-d3_lidar>
-        <origin xyz="0.0469 0.0 ${base_z_size/2 + 0.025}" rpy="0.0 0.0 0.0"/>
+        <origin xyz="0.008 0.0 ${base_z_size + cog_z + 0.025}" rpy="0.0 0.0 0.0"/>
     </xacro:i3e-d3_lidar>
     <xacro:i3e-d3_camera>
-        <origin xyz="-0.005 0.0 ${base_z_size/2 + camera_box_size + 0.025}" rpy="0.0 0.0 0.0"/>
+        <origin xyz="0.1 0.0 0.22" rpy="0.0 0.0 0.0"/>
     </xacro:i3e-d3_camera>
     <gazebo reference="base_link"><material>Gazebo/Yellow</material></gazebo>
+    <gazebo reference="neck"><material>Gazebo/DarkGrey</material></gazebo>
+    <gazebo reference="head"><material>Gazebo/Yellow</material></gazebo>
+    <gazebo reference="caster">
+        <material>Gazebo/DarkGrey</material>
+        <mu1 value="0.0"/>
+        <mu2 value="0.0"/>
+    </gazebo>
     <!-- Gazebo ROS Control Plugin -->
     <gazebo>

File: i3e-d3_description/urdf/wheel.urdf.xacro (robot description, xacro)
@@ -8,5 +8,5 @@
                 <!-- Need to adjust inertia matrix -->
                 <origin xyz="0.0 0.0 0.0"/>
-                <mass value="0.160"/>
+                <mass value="1.1"/>
                 <inertia
                   ixx="2.70474e-4" ixy="0.0" ixz="0.0"
