Commit message: Odometry and IMU fused

File: i3e-d3_description/urdf/accessories.urdf.xacro (robot description, xacro)
@@ -28,5 +28,5 @@
             <sensor type="ray" name="lidar_sensor">
               <pose>0 0 0 0 0 0</pose>
-              <visualize>true</visualize>
+              <visualize>false</visualize>
               <update_rate>40</update_rate>
               <ray>
@@ -131,3 +131,33 @@
         </gazebo>
     </xacro:macro>
+    <!-- IMU -->
+    <xacro:macro name="i3e-d3_imu" params="*joint_pose">
+        <link name="imu_link"/>
+        <joint name="imu_joint" type="fixed">
+            <parent link="base_link"/>
+            <child link="imu_link"/>
+            <xacro:insert_block name="joint_pose"/>
+        </joint>
+        <!-- IMU plugin -->
+        <gazebo reference="imu_link">
+          <gravity>true</gravity>
+          <sensor name="imu_sensor" type="imu">
+            <always_on>true</always_on>
+            <update_rate>100</update_rate>
+            <visualize>true</visualize>
+            <topic>__default_topic__</topic>
+            <plugin filename="libgazebo_ros_imu_sensor.so" name="imu_plugin">
+              <topicName>imu/data</topicName>
+              <bodyName>imu_link</bodyName>
+              <updateRateHZ>10.0</updateRateHZ>
+              <gaussianNoise>0.0</gaussianNoise>
+              <xyzOffset>0 0 0</xyzOffset>
+              <rpyOffset>0 0 0</rpyOffset>
+              <frameName>imu_link</frameName>
+              <initialOrientationAsReference>false</initialOrientationAsReference>
+            </plugin>
+            <pose>0 0 0 0 0 0</pose>
+          </sensor>
+        </gazebo>
+    </xacro:macro>
 </robot>

File: i3e-d3_description/urdf/i3e-d3.urdf.xacro (robot description, xacro)
@@ -156,4 +156,7 @@
         <origin xyz="0.1 0.0 0.22" rpy="0.0 0.0 0.0"/>
     </xacro:i3e-d3_camera>
+    <xacro:i3e-d3_imu>
+        <origin xyz="0.0 0.0 0.0" rpy="0.0 0.0 0.0"/>
+    </xacro:i3e-d3_imu>
     <gazebo reference="base_link"><material>Gazebo/Yellow</material></gazebo>
     <gazebo reference="neck"><material>Gazebo/DarkGrey</material></gazebo>

File: i3e-d3_description/urdf/wheel.urdf.xacro (robot description, xacro)
@@ -31,6 +31,6 @@
         <gazebo reference="${prefix}_wheel_link">
             <material>Gazebo/DarkGrey</material>
-            <mu1 value="0.5"/>
-            <mu2 value="0.5"/>
+            <mu1 value="1.0"/>
+            <mu2 value="1.0"/>
             <kp value="10000000.0" />
             <kd value="1" />

Commit message: little changes

File: i3e-d3_description/urdf/accessories.urdf.xacro (robot description, xacro)
@@ -73,5 +73,5 @@
                 <origin xyz="0.0 0.0 0.0" rpy="0.0 0.0 0.0"/>
                 <geometry>
-                    <box size="${camera_box_size} ${camera_box_size} ${camera_box_size}"/>
+                    <box size="0.015 0.030 0.027"/>
                 </geometry>
             </visual>
@@ -79,5 +79,5 @@
                 <origin xyz="0.0 0.0 0.0" rpy="0.0 0.0 0.0"/>
                 <geometry>
-                    <box size="${camera_box_size} ${camera_box_size} ${camera_box_size}"/>
+                    <box size="0.015 0.030 0.027"/>
                 </geometry>
             </collision>
@@ -94,13 +94,13 @@
             <update_rate>30.0</update_rate>
             <camera name="head">
-              <horizontal_fov>1.3962634</horizontal_fov>
+              <horizontal_fov>1.085595</horizontal_fov>
               <image>
-                <width>800</width>
-                <height>800</height>
+                <width>640</width>
+                <height>480</height>
                 <format>R8G8B8</format>
               </image>
               <clip>
-                <near>0.02</near>
-                <far>300</far>
+                <near>0.03</near>
+                <far>100</far>
               </clip>
               <noise>

File: i3e-d3_description/urdf/i3e-d3.urdf.xacro (robot description, xacro)
@@ -32,4 +32,5 @@
             <geometry>
                 <mesh filename="package://i3e-d3_description/meshes/body.stl"/>
+                <!--cylinder radius="${base_x_size/2}" length="${base_z_size}"/-->
             </geometry>
             <material name="blue">
@@ -154,5 +155,5 @@
     </xacro:i3e-d3_lidar>
     <xacro:i3e-d3_camera>
-        <origin xyz="0.1 0.0 0.22" rpy="0.0 0.0 0.0"/>
+        <origin xyz="0.03 0.0 ${base_z_size + cog_z + neck_z_size + 0.04}" rpy="0.0 0.0 0.0"/>
     </xacro:i3e-d3_camera>
     <xacro:i3e-d3_imu>

File: i3e-d3_description/urdf/i3e-d3_open_manipulator.urdf.xacro (robot description, xacro)
@@ -10,5 +10,5 @@
     <parent link="base_link"/>
     <child link="link1"/>
-    <origin xyz="0.0 -0.2 0.25" rpy="0.0 ${PI} ${PI}"/>
+    <origin xyz="0.0 -0.2 0.25" rpy="${PI} 0.0 0.0"/>
   </joint>
 </robot>

Commit message: use_open_manipulator arg in urdf

File: i3e-d3_description/urdf/accessories.urdf.xacro (robot description, xacro)
@@ -1,163 +1,166 @@
 <?xml version="1.0"?>
 <robot xmlns:xacro="http://www.ros.org/wiki/xacro" name="i3e-d3_accessories">
-    <xacro:property name="camera_box_size" value="0.04"/>
-    <!-- 3irobotix LIDAR -->
-    <xacro:macro name="i3e-d3_lidar" params="*joint_pose">
-        <link name="3irobotix_lidar">
-            <inertial>
-                <origin xyz="0.0 0.0 0.0" rpy="0.0 0.0 0.0"/>
-                <mass value="0.185"/>
-                <inertia ixx="1e-6" ixy="0.0" ixz="0.0" iyy="1e-6" iyz="0.0" izz="1e-6"/>
-            </inertial>
-            <visual>
-                <origin xyz="0.0 0.0 -0.025" rpy="0.0 0.0 0.0"/>
-                <geometry>
-                    <mesh filename="package://i3e-d3_description/meshes/lidar.stl"/>
-                </geometry>
-            </visual>
-        </link>
-        <joint name="lidar_joint" type="fixed">
-            <parent link="base_link"/>
-            <child link="3irobotix_lidar"/>
-            <xacro:insert_block name="joint_pose"/>
-        </joint>
-        <gazebo reference="3irobotix_lidar"><material>Gazebo/Black</material></gazebo>
-         <!-- Laser Plugin -->
-        <gazebo reference="3irobotix_lidar">
-            <sensor type="ray" name="lidar_sensor">
-              <pose>0 0 0 0 0 0</pose>
-              <visualize>false</visualize>
-              <update_rate>40</update_rate>
-              <ray>
-                <scan>
-                  <horizontal>
-                    <samples>720</samples>
-                    <resolution>1</resolution>
-                    <min_angle>-2.35619</min_angle>
-                    <max_angle>2.35619</max_angle>
-                  </horizontal>
-                </scan>
-                <range>
-                  <min>0.10</min>
-                  <max>8.0</max>
-                  <resolution>0.01</resolution>
-                </range>
-                <noise>
-                  <type>gaussian</type>
-                  <!-- Noise parameters based on published spec for Hokuyo laser
-                       achieving "+-30mm" accuracy at range < 10m.  A mean of 0.0m and
-                       stddev of 0.01m will put 99.7% of samples within 0.03m of the true
-                       reading. -->
-                  <mean>0.0</mean>
-                  <stddev>0.01</stddev>
-                </noise>
-              </ray>
-              <plugin name="gazebo_ros_head_hokuyo_controller" filename="libgazebo_ros_laser.so">
-                <robotNamespace>$(arg robot_namespace)</robotNamespace>
-                <topicName>laser/scan</topicName>
-                <frameName>3irobotix_lidar</frameName>
-              </plugin>
-            </sensor>
-        </gazebo>
-    </xacro:macro>
-    <!-- Camera -->
-    <xacro:macro name="i3e-d3_camera" params="*joint_pose">
-        <link name="camera_link">
-            <inertial>
-                <origin xyz="0.0 0.0 0.0" rpy="0.0 0.0 0.0"/>
-                <mass value="0.05"/>
-                <inertia ixx="1e-6" ixy="0.0" ixz="0.0" iyy="1e-6" iyz="0.0" izz="1e-6"/>
-            </inertial>
-            <visual>
-                <origin xyz="0.0 0.0 0.0" rpy="0.0 0.0 0.0"/>
-                <geometry>
-                    <box size="0.015 0.030 0.027"/>
-                </geometry>
-            </visual>
-            <collision>
-                <origin xyz="0.0 0.0 0.0" rpy="0.0 0.0 0.0"/>
-                <geometry>
-                    <box size="0.015 0.030 0.027"/>
-                </geometry>
-            </collision>
-        </link>
-        <joint name="camera_joint" type="fixed">
-            <parent link="base_link"/>
-            <child link="camera_link"/>
-            <xacro:insert_block name="joint_pose"/>
-        </joint>
-        <gazebo reference="camera_link"><material>Gazebo/Red</material></gazebo>
-        <!-- Camera Plugin -->
-        <gazebo reference="camera_link">
-          <sensor type="camera" name="camera">
-            <update_rate>30.0</update_rate>
-            <camera name="head">
-              <horizontal_fov>1.085595</horizontal_fov>
-              <image>
-                <width>640</width>
-                <height>480</height>
-                <format>R8G8B8</format>
-              </image>
-              <clip>
-                <near>0.03</near>
-                <far>100</far>
-              </clip>
-              <noise>
-                <type>gaussian</type>
-                <!-- Noise is sampled independently per pixel on each frame.
-                     That pixel's noise value is added to each of its color
-                     channels, which at that point lie in the range [0,1]. -->
-                <mean>0.0</mean>
-                <stddev>0.007</stddev>
-              </noise>
-            </camera>
-            <plugin name="camera_controller" filename="libgazebo_ros_camera.so">
-              <robotNamespace>$(arg robot_namespace)</robotNamespace>
-              <alwaysOn>true</alwaysOn>
-              <updateRate>0.0</updateRate>
-              <cameraName>camera</cameraName>
-              <imageTopicName>image_raw</imageTopicName>
-              <cameraInfoTopicName>camera_info</cameraInfoTopicName>
-              <frameName>camera_link</frameName>
-              <hackBaseline>0.07</hackBaseline>
-              <distortionK1>0.0</distortionK1>
-              <distortionK2>0.0</distortionK2>
-              <distortionK3>0.0</distortionK3>
-              <distortionT1>0.0</distortionT1>
-              <distortionT2>0.0</distortionT2>
-            </plugin>
-          </sensor>
-        </gazebo>
-    </xacro:macro>
-    <!-- IMU -->
-    <xacro:macro name="i3e-d3_imu" params="*joint_pose">
-        <link name="imu_link"/>
-        <joint name="imu_joint" type="fixed">
-            <parent link="base_link"/>
-            <child link="imu_link"/>
-            <xacro:insert_block name="joint_pose"/>
-        </joint>
-        <!-- IMU plugin -->
-        <gazebo reference="imu_link">
-          <gravity>true</gravity>
-          <sensor name="imu_sensor" type="imu">
-            <always_on>true</always_on>
-            <update_rate>100</update_rate>
-            <visualize>true</visualize>
-            <topic>__default_topic__</topic>
-            <plugin filename="libgazebo_ros_imu_sensor.so" name="imu_plugin">
-              <!--robotNamespace>$(arg robot_namespace)</robotNamespace-->
-              <topicName>imu/data</topicName>
-              <bodyName>imu_link</bodyName>
-              <updateRateHZ>10.0</updateRateHZ>
-              <gaussianNoise>0.0</gaussianNoise>
-              <xyzOffset>0 0 0</xyzOffset>
-              <rpyOffset>0 0 0</rpyOffset>
-              <frameName>$(arg robot_namespace)/imu_link</frameName>
-              <initialOrientationAsReference>false</initialOrientationAsReference>
-            </plugin>
-            <pose>0 0 0 0 0 0</pose>
-          </sensor>
-        </gazebo>
-    </xacro:macro>
+  <xacro:if value="$(arg use_open_manipulator)">
+    <xacro:include filename="$(find i3e-d3_manipulation_description)/urdf/i3e-d3_manipulation_robot.urdf.xacro"/>
+  </xacro:if>
+  <xacro:property name="camera_box_size" value="0.04"/>
+  <!-- 3irobotix LIDAR -->
+  <xacro:macro name="i3e-d3_lidar" params="*joint_pose">
+    <link name="3irobotix_lidar">
+      <inertial>
+        <origin xyz="0.0 0.0 0.0" rpy="0.0 0.0 0.0"/>
+        <mass value="0.185"/>
+        <inertia ixx="1e-6" ixy="0.0" ixz="0.0" iyy="1e-6" iyz="0.0" izz="1e-6"/>
+      </inertial>
+      <visual>
+      <origin xyz="0.0 0.0 -0.025" rpy="0.0 0.0 0.0"/>
+      <geometry>
+        <mesh filename="package://i3e-d3_description/meshes/lidar.stl"/>
+      </geometry>
+      </visual>
+    </link>
+    <joint name="lidar_joint" type="fixed">
+      <parent link="base_link"/>
+      <child link="3irobotix_lidar"/>
+      <xacro:insert_block name="joint_pose"/>
+    </joint>
+    <gazebo reference="3irobotix_lidar"><material>Gazebo/Black</material></gazebo>
+      <!-- Laser Plugin -->
+    <gazebo reference="3irobotix_lidar">
+      <sensor type="ray" name="lidar_sensor">
+        <pose>0 0 0 0 0 0</pose>
+        <visualize>false</visualize>
+        <update_rate>40</update_rate>
+        <ray>
+          <scan>
+            <horizontal>
+              <samples>720</samples>
+              <resolution>1</resolution>
+              <min_angle>-2.35619</min_angle>
+              <max_angle>2.35619</max_angle>
+            </horizontal>
+          </scan>
+          <range>
+            <min>0.10</min>
+            <max>8.0</max>
+            <resolution>0.01</resolution>
+          </range>
+          <noise>
+            <type>gaussian</type>
+            <!-- Noise parameters based on published spec for Hokuyo laser
+                  achieving "+-30mm" accuracy at range < 10m.  A mean of 0.0m and
+                  stddev of 0.01m will put 99.7% of samples within 0.03m of the true
+                  reading. -->
+            <mean>0.0</mean>
+            <stddev>0.01</stddev>
+          </noise>
+        </ray>
+        <plugin name="gazebo_ros_head_hokuyo_controller" filename="libgazebo_ros_laser.so">
+          <robotNamespace>$(arg robot_namespace)</robotNamespace>
+          <topicName>laser/scan</topicName>
+          <frameName>3irobotix_lidar</frameName>
+        </plugin>
+      </sensor>
+    </gazebo>
+  </xacro:macro>
+  <!-- Camera -->
+  <xacro:macro name="i3e-d3_camera" params="*joint_pose">
+    <link name="camera_link">
+      <inertial>
+        <origin xyz="0.0 0.0 0.0" rpy="0.0 0.0 0.0"/>
+        <mass value="0.05"/>
+        <inertia ixx="1e-6" ixy="0.0" ixz="0.0" iyy="1e-6" iyz="0.0" izz="1e-6"/>
+      </inertial>
+      <visual>
+        <origin xyz="0.0 0.0 0.0" rpy="0.0 0.0 0.0"/>
+        <geometry>
+            <box size="0.015 0.030 0.027"/>
+        </geometry>
+      </visual>
+      <collision>
+        <origin xyz="0.0 0.0 0.0" rpy="0.0 0.0 0.0"/>
+        <geometry>
+            <box size="0.015 0.030 0.027"/>
+        </geometry>
+      </collision>
+    </link>
+    <joint name="camera_joint" type="fixed">
+      <parent link="base_link"/>
+      <child link="camera_link"/>
+      <xacro:insert_block name="joint_pose"/>
+    </joint>
+    <gazebo reference="camera_link"><material>Gazebo/Red</material></gazebo>
+    <!-- Camera Plugin -->
+    <gazebo reference="camera_link">
+      <sensor type="camera" name="camera">
+        <update_rate>30.0</update_rate>
+        <camera name="head">
+          <horizontal_fov>1.085595</horizontal_fov>
+          <image>
+            <width>640</width>
+            <height>480</height>
+            <format>R8G8B8</format>
+          </image>
+          <clip>
+            <near>0.03</near>
+            <far>100</far>
+          </clip>
+          <noise>
+            <type>gaussian</type>
+            <!-- Noise is sampled independently per pixel on each frame.
+                  That pixel's noise value is added to each of its color
+                  channels, which at that point lie in the range [0,1]. -->
+            <mean>0.0</mean>
+            <stddev>0.007</stddev>
+          </noise>
+        </camera>
+        <plugin name="camera_controller" filename="libgazebo_ros_camera.so">
+          <robotNamespace>$(arg robot_namespace)</robotNamespace>
+          <alwaysOn>true</alwaysOn>
+          <updateRate>0.0</updateRate>
+          <cameraName>camera</cameraName>
+          <imageTopicName>image_raw</imageTopicName>
+          <cameraInfoTopicName>camera_info</cameraInfoTopicName>
+          <frameName>camera_link</frameName>
+          <hackBaseline>0.07</hackBaseline>
+          <distortionK1>0.0</distortionK1>
+          <distortionK2>0.0</distortionK2>
+          <distortionK3>0.0</distortionK3>
+          <distortionT1>0.0</distortionT1>
+          <distortionT2>0.0</distortionT2>
+        </plugin>
+      </sensor>
+    </gazebo>
+  </xacro:macro>
+  <!-- IMU -->
+  <xacro:macro name="i3e-d3_imu" params="*joint_pose">
+    <link name="imu_link"/>
+    <joint name="imu_joint" type="fixed">
+      <parent link="base_link"/>
+      <child link="imu_link"/>
+      <xacro:insert_block name="joint_pose"/>
+    </joint>
+      <!-- IMU plugin -->
+      <gazebo reference="imu_link">
+        <gravity>true</gravity>
+        <sensor name="imu_sensor" type="imu">
+          <always_on>true</always_on>
+          <update_rate>100</update_rate>
+          <visualize>true</visualize>
+          <topic>__default_topic__</topic>
+          <plugin filename="libgazebo_ros_imu_sensor.so" name="imu_plugin">
+            <!--robotNamespace>$(arg robot_namespace)</robotNamespace-->
+            <topicName>imu/data</topicName>
+            <bodyName>imu_link</bodyName>
+            <updateRateHZ>10.0</updateRateHZ>
+            <gaussianNoise>0.0</gaussianNoise>
+            <xyzOffset>0 0 0</xyzOffset>
+            <rpyOffset>0 0 0</rpyOffset>
+            <frameName>$(arg robot_namespace)/imu_link</frameName>
+            <initialOrientationAsReference>false</initialOrientationAsReference>
+          </plugin>
+          <pose>0 0 0 0 0 0</pose>
+        </sensor>
+      </gazebo>
+  </xacro:macro>
 </robot>

File: i3e-d3_description/urdf/i3e-d3.urdf.xacro (robot description, xacro)
@@ -2,4 +2,5 @@
 <robot name="i3e-d3" xmlns:xacro="http://www.ros.org/wiki/xacro">
     <xacro:arg name="robot_namespace" default="i3e_d3"/>
+    <xacro:arg name="use_open_manipulator" default="true"/>
     <xacro:property name="PI" value="3.14159"/>
     <!-- Included URDF/XACRO Files -->
