Commit message: Implementing head joy controller

File: i3e-d3_description/urdf/accessories.urdf.xacro (robot description, xacro)
@@ -65,9 +65,9 @@
   </xacro:macro>
   <!-- Camera -->
-  <xacro:macro name="i3e-d3_camera" params="*joint_pose">
+  <xacro:macro name="i3e-d3_camera">
     <link name="camera_link">
       <inertial>
         <origin xyz="0.0 0.0 0.0" rpy="0.0 0.0 0.0"/>
-        <mass value="0.05"/>
+        <mass value="3.3e-3"/>
         <inertia ixx="1e-6" ixy="0.0" ixz="0.0" iyy="1e-6" iyz="0.0" izz="1e-6"/>
       </inertial>
@@ -75,5 +75,5 @@
         <origin xyz="0.0 0.0 0.0" rpy="0.0 0.0 0.0"/>
         <geometry>
-            <box size="0.015 0.030 0.027"/>
+          <box size="0.001 0.025 0.024"/>
         </geometry>
       </visual>
@@ -81,14 +81,14 @@
         <origin xyz="0.0 0.0 0.0" rpy="0.0 0.0 0.0"/>
         <geometry>
-            <box size="0.015 0.030 0.027"/>
+          <box size="0.025 0.024 0.001"/>
         </geometry>
       </collision>
     </link>
     <joint name="camera_joint" type="fixed">
-      <parent link="base_link"/>
+      <parent link="head_link"/>
       <child link="camera_link"/>
-      <xacro:insert_block name="joint_pose"/>
+      <origin xyz="0.0 -0.03 0.036" rpy="0.0 0.0 ${-PI/2}"/>
     </joint>
-    <gazebo reference="camera_link"><material>Gazebo/Red</material></gazebo>
+    <gazebo reference="camera_link"><material>Gazebo/Green</material></gazebo>
     <!-- Camera Plugin -->
     <gazebo reference="camera_link">

File: i3e-d3_description/urdf/head.urdf.xacro (robot description, xacro)
@@ -1,159 +1,167 @@
 <?xml version="1.0"?>
 <robot name="i3e-d3_head" xmlns:xacro="http://www.ros.org/wiki/xacro">
-  <xacro:property name="base_height" value="0.342"/>
-  <!-- Transmission macro -->
-  <xacro:macro name="SimpleTransmission" params="joint n">
-    <transmission name="tran_${n}">
-      <type>transmission_interface/SimpleTransmission</type>
-      <joint name="${joint}">
-        <hardwareInterface>hardware_interface/PositionJointInterface</hardwareInterface>
-      </joint>
-      <actuator name="servo_${n}">
-        <hardwareInterface>hardware_interface/PositionJointInterface</hardwareInterface>
-        <mechanicalReduction>1</mechanicalReduction>
-      </actuator>
-    </transmission>
+  <xacro:macro name="i3e-d3_head">
+    <xacro:macro name="TransmissionServo" params="joint n">
+        <transmission name="tran_${n}">
+        <type>transmission_interface/SimpleTransmission</type>
+        <joint name="${joint}">
+            <hardwareInterface>hardware_interface/PositionJointInterface</hardwareInterface>
+        </joint>
+        <actuator name="servo_${n}">
+            <hardwareInterface>hardware_interface/PositionJointInterface</hardwareInterface>
+            <mechanicalReduction>1</mechanicalReduction>
+        </actuator>
+        </transmission>
+    </xacro:macro>
+    <link name="motor_neck_link">
+        <visual>
+            <origin xyz="0.0 0.0 0.0" rpy="0.0 0.0 0.0"/>
+            <geometry>
+                <mesh filename="package://i3e-d3_description/meshes/servo.stl"/>
+            </geometry>
+        </visual>
+        <collision>
+            <origin xyz="0.0 0.0 0.0" rpy="0.0 0.0 0.0"/>
+            <geometry>
+                <box size="0.04 0.02 0.04"/>
+            </geometry>
+        </collision>
+        <inertial>
+            <origin xyz="0.0 0.0 0.0" rpy="0.0 0.0 0.0"/>
+                <mass value="0.001"/>
+                <inertia
+                    ixx="1e-6" ixy="0.0" ixz="0.0"
+                    iyy="1e-6" iyz="0.0"
+                    izz="1e-6"/>
+        </inertial>
+    </link>
+    <joint name="motor_neck_joint" type="fixed">
+        <parent link="base_link"/>
+        <child link="motor_neck_link"/>
+        <origin xyz="0.005 0.0 ${base_height/2}" rpy="0.0 0.0 ${PI/2}"/>
+    </joint>
+    <link name="neck_link">
+        <visual>
+            <origin xyz="0.0 0.0 0.0" rpy="0.0 0.0 0.0"/>
+            <geometry>
+                <box size="0.05 0.03 0.05"/>
+            </geometry>
+        </visual>
+        <collision>
+            <origin xyz="0.0 0.0 0.0" rpy="0.0 0.0 0.0"/>
+            <geometry>
+                <box size="0.05 0.03 0.05"/>
+            </geometry>
+        </collision>
+        <inertial>
+            <origin xyz="0.0 0.0 0.0" rpy="0.0 0.0 0.0"/>
+                <mass value="0.001"/>
+                <inertia
+                    ixx="1e-6" ixy="0.0" ixz="0.0"
+                    iyy="1e-6" iyz="0.0"
+                    izz="1e-6"/>
+        </inertial>
+    </link>
+    <joint name="neck_joint" type="revolute">
+        <parent link="motor_neck_link"/>
+        <child link="neck_link"/>
+        <axis xyz="0 0 1"/>
+        <limit lower="-1.5707" upper="1.5707" effort="0.8" velocity="0.5"/>
+        <origin xyz="0.0 0.0 0.038" rpy="0.0 0.0 0.0"/>
+    </joint>
+    <xacro:TransmissionServo n="neck" joint="neck_joint" />
+    <link name="motor_head_link">
+        <visual>
+            <origin xyz="0.0 0.0 0.0" rpy="0.0 0.0 0.0"/>
+            <geometry>
+                <mesh filename="package://i3e-d3_description/meshes/servo.stl"/>
+            </geometry>
+        </visual>
+        <collision>
+            <origin xyz="0.0 0.0 0.0" rpy="0.0 0.0 0.0"/>
+            <geometry>
+                <box size="0.04 0.02 0.04"/>
+            </geometry>
+        </collision>
+        <inertial>
+            <origin xyz="0.0 0.0 0.0" rpy="0.0 0.0 0.0"/>
+                <mass value="0.001"/>
+                <inertia
+                    ixx="1e-6" ixy="0.0" ixz="0.0"
+                    iyy="1e-6" iyz="0.0"
+                    izz="1e-6"/>
+        </inertial>
+    </link>
+    <joint name="motor_head_joint" type="revolute">
+        <origin xyz="0.0 -0.02 0.065" rpy="0.0 ${-PI/2} 0.0"/>
+        <parent link="neck_link"/>
+        <child link="motor_head_link"/>
+        <axis xyz="0 0 1"/>
+        <limit lower="-0.2618" upper="0.7854" effort="0.8" velocity="0.5"/>
+    </joint>
+    <xacro:TransmissionServo n="head" joint="motor_head_joint" />
+    <link name="head_link">
+        <visual>
+            <origin xyz="0.0 0.0 0.0" rpy="0.0 0.0 0.0"/>
+            <geometry>
+                <box size="0.13 0.06 0.1"/>
+            </geometry>
+        </visual>
+        <collision>
+            <origin xyz="0.0 0.0 0.0" rpy="0.0 0.0 0.0"/>
+            <geometry>
+                <box size="0.13 0.06 0.1"/>
+            </geometry>
+        </collision>
+        <inertial>
+            <origin xyz="0.0 0.0 0.0" rpy="0.0 0.0 0.0"/>
+                <mass value="0.001"/>
+                <inertia
+                    ixx="1e-6" ixy="0.0" ixz="0.0"
+                    iyy="1e-6" iyz="0.0"
+                    izz="1e-6"/>
+        </inertial>
+    </link>
+    <joint name="head_joint" type="fixed">
+        <origin xyz="0.0 -0.04 0.0" rpy="0.0 ${PI/2} 0.0"/>
+        <child link="head_link"/>
+        <parent link="motor_head_link"/>
+    </joint>
+    <link name="display">
+        <visual>
+            <origin xyz="0.0 0.0 0.0" rpy="0.0 0.0 0.0"/>
+            <geometry>
+                <box size="0.064 0.01 0.096"/>
+            </geometry>
+        </visual>
+        <collision>
+            <origin xyz="0.0 0.0 0.0" rpy="0.0 0.0 0.0"/>
+            <geometry>
+                <box size="0.064 0.01 0.096"/>
+            </geometry>
+        </collision>
+        <inertial>
+            <origin xyz="0.0 0.0 0.0" rpy="0.0 0.0 0.0"/>
+                <mass value="0.001"/>
+                <inertia
+                    ixx="1e-6" ixy="0.0" ixz="0.0"
+                    iyy="1e-6" iyz="0.0"
+                    izz="1e-6"/>
+        </inertial>
+    </link>
+    <joint name="display_joint" type="fixed">
+        <origin xyz="0.0 -0.033 -0.01" rpy="0.0 ${PI/2} 0.0"/>
+        <child link="display"/>
+        <parent link="head_link"/>
+    </joint>
+    <gazebo reference="motor_neck_link">
+        <material>Gazebo/DarkGrey</material>
+    </gazebo>
+    <gazebo reference="motor_head_link">
+        <material>Gazebo/DarkGrey</material>
+    </gazebo>
+    <gazebo reference="display">
+        <material>Gazebo/Red</material>
+    </gazebo>
   </xacro:macro>
-  <link name="motor_neck_link">
-      <visual>
-          <origin xyz="0.0 0.0 0.0" rpy="0.0 0.0 0.0"/>
-          <geometry>
-              <mesh filename="package://i3e-d3_description/meshes/servo.stl"/>
-          </geometry>
-      </visual>
-      <collision>
-          <origin xyz="0.0 0.0 0.0" rpy="0.0 0.0 0.0"/>
-          <geometry>
-              <box size="0.04 0.02 0.04"/>
-          </geometry>
-      </collision>
-      <inertial>
-          <origin xyz="0.0 0.0 0.0" rpy="0.0 0.0 0.0"/>
-              <mass value="0.001"/>
-              <inertia
-                  ixx="1e-6" ixy="0.0" ixz="0.0"
-                  iyy="1e-6" iyz="0.0"
-                  izz="1e-6"/>
-      </inertial>
-  </link>
-  <joint name="motor_neck_joint" type="fixed">
-      <parent link="base_link"/>
-      <child link="motor_neck_link"/>
-      <origin xyz="0.005 0.0 ${base_height/2}" rpy="0.0 0.0 ${PI/2}"/>
-  </joint>
-  <link name="neck_link">
-      <visual>
-          <origin xyz="0.0 0.0 0.0" rpy="0.0 0.0 0.0"/>
-          <geometry>
-              <box size="0.05 0.03 0.05"/>
-          </geometry>
-      </visual>
-      <collision>
-          <origin xyz="0.0 0.0 0.0" rpy="0.0 0.0 0.0"/>
-          <geometry>
-              <box size="0.05 0.03 0.05"/>
-          </geometry>
-      </collision>
-      <inertial>
-          <origin xyz="0.0 0.0 0.0" rpy="0.0 0.0 0.0"/>
-              <mass value="0.001"/>
-              <inertia
-                  ixx="1e-6" ixy="0.0" ixz="0.0"
-                  iyy="1e-6" iyz="0.0"
-                  izz="1e-6"/>
-      </inertial>
-  </link>
-  <joint name="neck_joint" type="revolute">
-      <parent link="motor_neck_link"/>
-      <child link="neck_link"/>
-      <axis xyz="0 0 1"/>
-      <limit lower="-1.5707" upper="1.5707" effort="0.8" velocity="0.2"/>
-      <origin xyz="0.0 0.0 0.038" rpy="0.0 0.0 0.0"/>
-  </joint>
-  <xacro:SimpleTransmission n="neck" joint="neck_joint" />
-  <link name="motor_head_link">
-      <visual>
-          <origin xyz="0.0 0.0 0.0" rpy="0.0 0.0 0.0"/>
-          <geometry>
-              <mesh filename="package://i3e-d3_description/meshes/servo.stl"/>
-          </geometry>
-      </visual>
-      <collision>
-          <origin xyz="0.0 0.0 0.0" rpy="0.0 0.0 0.0"/>
-          <geometry>
-              <box size="0.04 0.02 0.04"/>
-          </geometry>
-      </collision>
-      <inertial>
-          <origin xyz="0.0 0.0 0.0" rpy="0.0 0.0 0.0"/>
-              <mass value="0.001"/>
-              <inertia
-                  ixx="1e-6" ixy="0.0" ixz="0.0"
-                  iyy="1e-6" iyz="0.0"
-                  izz="1e-6"/>
-      </inertial>
-  </link>
-  <joint name="motor_head_joint" type="revolute">
-    <origin xyz="0.0 -0.02 0.065" rpy="0.0 ${-PI/2} 0.0"/>
-    <parent link="neck_link"/>
-    <child link="motor_head_link"/>
-    <axis xyz="0 0 1"/>
-    <limit lower="-0.2618" upper="0.7854" effort="0.8" velocity="0.2"/>
-    <origin xyz="0.0 0.0 0.038" rpy="0.0 0.0 0.0"/>
-  </joint>
-  <xacro:SimpleTransmission n="head" joint="motor_head_joint" />
-  <link name="head_link">
-      <visual>
-          <origin xyz="0.0 0.0 0.0" rpy="0.0 0.0 0.0"/>
-          <geometry>
-              <box size="0.13 0.06 0.1"/>
-          </geometry>
-      </visual>
-      <collision>
-          <origin xyz="0.0 0.0 0.0" rpy="0.0 0.0 0.0"/>
-          <geometry>
-              <box size="0.05 0.03 0.05"/>
-          </geometry>
-      </collision>
-      <inertial>
-          <origin xyz="0.0 0.0 0.0" rpy="0.0 0.0 0.0"/>
-              <mass value="0.001"/>
-              <inertia
-                  ixx="1e-6" ixy="0.0" ixz="0.0"
-                  iyy="1e-6" iyz="0.0"
-                  izz="1e-6"/>
-      </inertial>
-  </link>
-  <joint name="head_joint" type="fixed">
-      <origin xyz="0.0 -0.04 0.0" rpy="0.0 ${PI/2} 0.0"/>
-      <child link="head_link"/>
-      <parent link="motor_head_link"/>
-  </joint>
-  <link name="display">
-      <visual>
-          <origin xyz="0.0 0.0 0.0" rpy="0.0 0.0 0.0"/>
-          <geometry>
-              <box size="0.064 0.01 0.096"/>
-          </geometry>
-      </visual>
-      <collision>
-          <origin xyz="0.0 0.0 0.0" rpy="0.0 0.0 0.0"/>
-          <geometry>
-              <box size="0.064 0.01 0.096"/>
-          </geometry>
-      </collision>
-      <inertial>
-          <origin xyz="0.0 0.0 0.0" rpy="0.0 0.0 0.0"/>
-              <mass value="0.001"/>
-              <inertia
-                  ixx="1e-6" ixy="0.0" ixz="0.0"
-                  iyy="1e-6" iyz="0.0"
-                  izz="1e-6"/>
-      </inertial>
-  </link>
-  <joint name="display_joint" type="fixed">
-      <origin xyz="0.0 -0.033 -0.01" rpy="0.0 ${PI/2} 0.0"/>
-      <child link="display"/>
-      <parent link="head_link"/>
-  </joint>
 </robot>

File: i3e-d3_description/urdf/i3e-d3.urdf.xacro (robot description, xacro)
@@ -7,5 +7,4 @@
     <xacro:include filename="$(find i3e-d3_description)/urdf/wheel.urdf.xacro"/>
     <xacro:include filename="$(find i3e-d3_description)/urdf/accessories.urdf.xacro"/>
-    <xacro:include filename="$(find i3e-d3_description)/urdf/decorations.urdf.xacro"/>
     <xacro:include filename="$(find i3e-d3_description)/urdf/head.urdf.xacro"/>
     <!-- Base, head and neck sizes -->
@@ -61,5 +60,5 @@
         <origin xyz="0.0 0.0 0.0" rpy="0.0 0.0 0.0"/>
     </joint>
-    <!--xacro:i3e-d3_decorate/-->
+    <xacro:i3e-d3_head/>
     <!-- I3E-D3 wheel macros -->
     <xacro:i3e-d3_wheel prefix="left">
@@ -76,12 +75,8 @@
     </xacro:i3e-d3_caster>
     <!-- Sensors -->
+    <xacro:i3e-d3_camera/>
     <xacro:i3e-d3_lidar>
         <origin xyz="${base_radius/2} 0.0 ${base_height/2 + 0.025}" rpy="0.0 0.0 0.0"/>
     </xacro:i3e-d3_lidar>
-    <!--
-    <xacro:i3e-d3_camera>
-        <origin xyz="0.03 0.0 ${base_height/2 + neck_z_size + 0.04}" rpy="0.0 0.0 0.0"/>
-    </xacro:i3e-d3_camera>
-    -->
     <xacro:i3e-d3_imu>
         <origin xyz="0.0 0.0 0.0" rpy="0.0 0.0 0.0"/>

File: i3e-d3_description/urdf/wheel.urdf.xacro (robot description, xacro)
@@ -62,7 +62,7 @@
             </visual>
             <collision>
-                <origin xyz="0.0 0.0 0.0" rpy="0.0 0.0 0.0"/>
+                <origin xyz="-0.0 0.0 0.0" rpy="0.0 0.0 0.0"/>
                 <geometry>
-                    <box size="0.07 0.07 0.07"/>
+                    <sphere radius="0.035"/>
                 </geometry>
             </collision>

Commit message: update head and neck in URDF

File: i3e-d3_description/urdf/accessories.urdf.xacro (robot description, xacro)
@@ -4,5 +4,4 @@
     <xacro:include filename="$(find i3e-d3_manipulation_description)/urdf/i3e-d3_manipulation_robot.urdf.xacro"/>
   </xacro:if>
-  <xacro:property name="camera_box_size" value="0.04"/>
   <!-- 3irobotix LIDAR -->
   <xacro:macro name="i3e-d3_lidar" params="*joint_pose">
@@ -86,7 +85,7 @@
     </link>
     <joint name="camera_joint" type="fixed">
-      <parent link="head_link"/>
+      <parent link="face_link"/>
       <child link="camera_link"/>
-      <origin xyz="0.0 -0.03 0.036" rpy="0.0 0.0 ${-PI/2}"/>
+      <origin xyz="0.05 -0.026 0.0" rpy="${-PI/2} 0.0 ${-PI/2}"/>
     </joint>
     <gazebo reference="camera_link"><material>Gazebo/Green</material></gazebo>

File: i3e-d3_description/urdf/head.urdf.xacro (robot description, xacro)
@@ -45,11 +45,11 @@
             <origin xyz="0.0 0.0 0.0" rpy="0.0 0.0 0.0"/>
             <geometry>
-                <box size="0.05 0.03 0.05"/>
-            </geometry>
-        </visual>
-        <collision>
-            <origin xyz="0.0 0.0 0.0" rpy="0.0 0.0 0.0"/>
-            <geometry>
-                <box size="0.05 0.03 0.05"/>
+                <mesh filename="package://i3e-d3_description/meshes/neck.stl"/>
+            </geometry>
+        </visual>
+        <collision>
+            <origin xyz="0.0 0.0 0.0" rpy="0.0 0.0 0.0"/>
+            <geometry>
+                <mesh filename="package://i3e-d3_description/meshes/neck.stl"/>
             </geometry>
         </collision>
@@ -68,5 +68,5 @@
         <axis xyz="0 0 1"/>
         <limit lower="-1.5707" upper="1.5707" effort="0.8" velocity="0.5"/>
-        <origin xyz="0.0 0.0 0.038" rpy="0.0 0.0 0.0"/>
+        <origin xyz="0.0 0.0 0.016" rpy="0.0 0.0 0.0"/>
     </joint>
     <xacro:TransmissionServo n="neck" joint="neck_joint" />
@@ -94,22 +94,22 @@
     </link>
     <joint name="head_joint" type="revolute">
-        <origin xyz="0.0 -0.02 0.065" rpy="0.0 ${-PI/2} 0.0"/>
+        <origin xyz="-0.0085 -0.117 0.142" rpy="0.0 ${-PI/2} 0.0"/>
         <parent link="neck_link"/>
         <child link="motor_head_link"/>
         <axis xyz="0 0 1"/>
-        <limit lower="-0.2618" upper="0.7854" effort="0.8" velocity="0.5"/>
+        <limit lower="-0.2618" upper="0.2618" effort="0.8" velocity="0.5"/>
     </joint>
     <xacro:TransmissionServo n="head" joint="head_joint" />
-    <link name="head_link">
-        <visual>
-            <origin xyz="0.0 0.0 0.0" rpy="0.0 0.0 0.0"/>
-            <geometry>
-                <box size="0.13 0.06 0.1"/>
-            </geometry>
-        </visual>
-        <collision>
-            <origin xyz="0.0 0.0 0.0" rpy="0.0 0.0 0.0"/>
-            <geometry>
-                <box size="0.13 0.06 0.1"/>
+    <link name="face_link">
+        <visual>
+            <origin xyz="0.0 0.0 0.0" rpy="0.0 ${-PI/2} ${PI}"/>
+            <geometry>
+                <mesh filename="package://i3e-d3_description/meshes/face.stl"/>
+            </geometry>
+        </visual>
+        <collision>
+            <origin xyz="0.0 0.0 0.0" rpy="0.0 ${-PI/2} ${PI}"/>
+            <geometry>
+                <mesh filename="package://i3e-d3_description/meshes/face.stl"/>
             </geometry>
         </collision>
@@ -124,19 +124,19 @@
     </link>
     <joint name="motor_head_joint" type="fixed">
-        <origin xyz="0.0 -0.04 0.0" rpy="0.0 ${PI/2} 0.0"/>
-        <child link="head_link"/>
+        <origin xyz="-0.0115 -0.0435 -0.012" rpy="0.0 0.0 0.0"/>
+        <child link="face_link"/>
         <parent link="motor_head_link"/>
     </joint>
-    <link name="display">
-        <visual>
-            <origin xyz="0.0 0.0 0.0" rpy="0.0 0.0 0.0"/>
-            <geometry>
-                <box size="0.064 0.01 0.096"/>
-            </geometry>
-        </visual>
-        <collision>
-            <origin xyz="0.0 0.0 0.0" rpy="0.0 0.0 0.0"/>
-            <geometry>
-                <box size="0.064 0.01 0.096"/>
+    <link name="display_link">
+        <visual>
+            <origin xyz="0.0 0.0 0.0" rpy="0.0 0.0 0.0"/>
+            <geometry>
+                <mesh filename="package://i3e-d3_description/meshes/LEDs_face.stl"/>
+            </geometry>
+        </visual>
+        <collision>
+            <origin xyz="0.0 0.0 0.0" rpy="0.0 0.0 0.0"/>
+            <geometry>
+                <mesh filename="package://i3e-d3_description/meshes/LEDs_face.stl"/>
             </geometry>
         </collision>
@@ -151,8 +151,41 @@
     </link>
     <joint name="display_joint" type="fixed">
-        <origin xyz="0.0 -0.033 -0.01" rpy="0.0 ${PI/2} 0.0"/>
-        <child link="display"/>
-        <parent link="head_link"/>
-    </joint>
+        <origin xyz="-0.005 -0.02 0.0" rpy="${PI/2} ${PI/2} 0.0"/>
+        <child link="display_link"/>
+        <parent link="face_link"/>
+    </joint>
+    <link name="head_cover_link">
+        <visual>
+            <origin xyz="0.0 0.0 0.0" rpy="${-PI/2} ${PI/2} ${PI/2}"/>
+            <geometry>
+                <mesh filename="package://i3e-d3_description/meshes/head_cover.stl"/>
+            </geometry>
+        </visual>
+        <collision>
+            <origin xyz="0.0 0.0 0.0" rpy="0.0 0.0 0.0"/>
+            <geometry>
+                <mesh filename="package://i3e-d3_description/meshes/head_cover.stl"/>
+            </geometry>
+        </collision>
+        <inertial>
+            <origin xyz="0.0 0.0 0.0" rpy="0.0 0.0 0.0"/>
+                <mass value="0.001"/>
+                <inertia
+                    ixx="1e-6" ixy="0.0" ixz="0.0"
+                    iyy="1e-6" iyz="0.0"
+                    izz="1e-6"/>
+        </inertial>
+    </link>
+    <joint name="head_cover_joint" type="fixed">
+        <origin xyz="0.011 0.009 0.0" rpy="0.0 ${PI} 0.0"/>
+        <child link="head_cover_link"/>
+        <parent link="face_link"/>
+    </joint>
+    <gazebo reference="neck_link">
+        <material>Gazebo/White</material>
+    </gazebo>
+    <gazebo reference="face_link">
+        <material>Gazebo/Whire</material>
+    </gazebo>
     <gazebo reference="motor_neck_link">
         <material>Gazebo/DarkGrey</material>
@@ -161,6 +194,9 @@
         <material>Gazebo/DarkGrey</material>
     </gazebo>
-    <gazebo reference="display">
-        <material>Gazebo/Red</material>
+    <gazebo reference="display_link">
+        <material>Gazebo/Gray</material>
+    </gazebo>
+    <gazebo reference="head_cover_link">
+        <material>Gazebo/Blue</material>
     </gazebo>
   </xacro:macro>

File: i3e-d3_description/urdf/i3e-d3.urdf.xacro (robot description, xacro)
@@ -82,5 +82,5 @@
         <origin xyz="0.0 0.0 0.0" rpy="0.0 0.0 0.0"/>
     </xacro:i3e-d3_imu>
-    <gazebo reference="base_link"><material>Gazebo/Yellow</material></gazebo>
+    <gazebo reference="base_link"><material>Gazebo/Blue</material></gazebo>
     <!--
     <gazebo reference="neck"><material>Gazebo/DarkGrey</material></gazebo>
