Commit message: materials.urdf.xacro created

File: i3e-d3_description/urdf/accessories.urdf.xacro (robot description, xacro)
@@ -89,5 +89,4 @@
       <origin xyz="0.05 -0.026 0.0" rpy="${-PI/2} 0.0 ${-PI/2}"/>
     </joint>
-    <gazebo reference="camera_link"><material>Gazebo/Green</material></gazebo>
     <!-- Camera Plugin -->
     <gazebo reference="camera_link">

File: i3e-d3_description/urdf/head.urdf.xacro (robot description, xacro)
@@ -20,4 +20,5 @@
                 <mesh filename="package://i3e-d3_description/meshes/servo.stl"/>
             </geometry>
+            <material name="darkgray"/>
         </visual>
         <collision>
@@ -47,4 +48,5 @@
                 <mesh filename="package://i3e-d3_description/meshes/neck.stl"/>
             </geometry>
+            <material name="gray"/>
         </visual>
         <collision>
@@ -77,4 +79,5 @@
                 <mesh filename="package://i3e-d3_description/meshes/servo.stl"/>
             </geometry>
+            <material name="darkgray"/>
         </visual>
         <collision>
@@ -107,4 +110,5 @@
                 <mesh filename="package://i3e-d3_description/meshes/face.stl"/>
             </geometry>
+            <material name="gray"/>
         </visual>
         <collision>
@@ -134,4 +138,5 @@
                 <mesh filename="package://i3e-d3_description/meshes/LEDs_face.stl"/>
             </geometry>
+            <material name="white"/>
         </visual>
         <collision>
@@ -161,4 +166,5 @@
                 <mesh filename="package://i3e-d3_description/meshes/head_cover.stl"/>
             </geometry>
+            <material name="blue"/>
         </visual>
         <collision>
@@ -166,5 +172,5 @@
             <geometry>
                 <mesh filename="package://i3e-d3_description/meshes/head_cover.stl"/>
-            </geometry>
+            </geometry>cover
         </collision>
         <inertial>
@@ -182,22 +188,4 @@
         <parent link="face_link"/>
     </joint>
-    <gazebo reference="neck_link">
-        <material>Gazebo/White</material>
-    </gazebo>
-    <gazebo reference="face_link">
-        <material>Gazebo/Whire</material>
-    </gazebo>
-    <gazebo reference="motor_neck_link">
-        <material>Gazebo/DarkGrey</material>
-    </gazebo>
-    <gazebo reference="motor_head_link">
-        <material>Gazebo/DarkGrey</material>
-    </gazebo>
-    <gazebo reference="display_link">
-        <material>Gazebo/Gray</material>
-    </gazebo>
-    <gazebo reference="head_cover_link">
-        <material>Gazebo/Blue</material>
-    </gazebo>
   </xacro:macro>
 </robot>

File: i3e-d3_description/urdf/i3e-d3.urdf.xacro (robot description, xacro)
@@ -8,4 +8,5 @@
     <xacro:include filename="$(find i3e-d3_description)/urdf/accessories.urdf.xacro"/>
     <xacro:include filename="$(find i3e-d3_description)/urdf/head.urdf.xacro"/>
+    <xacro:include filename="$(find i3e-d3_description)/urdf/materials.urdf.xacro"/>
     <!-- Base, head and neck sizes -->
     <xacro:property name="base_radius" value="0.155"/>
@@ -26,7 +27,5 @@
                 <cylinder radius="${base_radius}" length="${base_height}"/>
             </geometry>
-            <material name="blue">
-                <color rgba="0.0 0.0 1.0 1.0"/>
-            </material>
+            <material name="blue"/>"
         </visual>
         <collision>

File: i3e-d3_description/urdf/wheel.urdf.xacro (robot description, xacro)
@@ -30,5 +30,4 @@
         <!-- Need to adjust gazebo properties -->
         <gazebo reference="${prefix}_wheel_link">
-            <material>Gazebo/DarkGrey</material>
             <mu1 value="1.0"/>
             <mu2 value="1.0"/>

Commit message: update meshes orientation

File: i3e-d3_description/urdf/accessories.urdf.xacro (robot description, xacro)
@@ -13,9 +13,16 @@
       </inertial>
       <visual>
-      <origin xyz="0.0 0.0 -0.025" rpy="0.0 0.0 0.0"/>
-      <geometry>
-        <mesh filename="package://i3e-d3_description/meshes/lidar.stl"/>
-      </geometry>
+        <origin xyz="0.0 0.0 -0.025" rpy="0.0 0.0 0.0"/>
+        <geometry>
+          <mesh filename="package://i3e-d3_description/meshes/lidar.stl"/>
+        </geometry>
+        <material name="black"/>
       </visual>
+      <collision>
+        <origin xyz="0.0 0.0 0.0" rpy="0.0 0.0 0.0"/>
+        <geometry>
+          <mesh filename="package://i3e-d3_description/meshes/lidar.stl"/>
+        </geometry>
+      </collision>
     </link>
     <joint name="lidar_joint" type="fixed">
@@ -64,5 +71,5 @@
   </xacro:macro>
   <!-- Camera -->
-  <xacro:macro name="i3e-d3_camera">
+  <xacro:macro name="i3e-d3_camera" params="*joint_pose">
     <link name="camera_link">
       <inertial>
@@ -87,5 +94,5 @@
       <parent link="face_link"/>
       <child link="camera_link"/>
-      <origin xyz="0.05 -0.026 0.0" rpy="${-PI/2} 0.0 ${-PI/2}"/>
+      <xacro:insert_block name="joint_pose"/>
     </joint>
     <!-- Camera Plugin -->

File: i3e-d3_description/urdf/head.urdf.xacro (robot description, xacro)
@@ -16,5 +16,5 @@
     <link name="motor_neck_link">
         <visual>
-            <origin xyz="0.0 0.0 0.0" rpy="0.0 0.0 0.0"/>
+            <origin xyz="0.0 0.0 0.0" rpy="0.0 0.0 ${PI/2}"/>
             <geometry>
                 <mesh filename="package://i3e-d3_description/meshes/servo.stl"/>
@@ -23,11 +23,11 @@
         </visual>
         <collision>
-            <origin xyz="0.0 0.0 0.0" rpy="0.0 0.0 0.0"/>
+            <origin xyz="0.0 0.0 0.0" rpy="0.0 0.0 ${PI/2}"/>
             <geometry>
-                <box size="0.04 0.02 0.04"/>
+                <mesh filename="package://i3e-d3_description/meshes/servo.stl"/>
             </geometry>
         </collision>
         <inertial>
-            <origin xyz="0.0 0.0 0.0" rpy="0.0 0.0 0.0"/>
+            <origin xyz="0.0 0.0 0.0" rpy="0.0 0.0 ${PI/2}"/>
                 <mass value="0.001"/>
                 <inertia
@@ -40,5 +40,5 @@
         <parent link="base_link"/>
         <child link="motor_neck_link"/>
-        <origin xyz="0.005 0.0 ${base_height/2}" rpy="0.0 0.0 ${PI/2}"/>
+        <origin xyz="0.005 0.0 ${base_height/2}" rpy="0.0 0.0 0.0"/>
     </joint>
     <link name="neck_link">
@@ -57,10 +57,10 @@
         </collision>
         <inertial>
-            <origin xyz="0.0 0.0 0.0" rpy="0.0 0.0 0.0"/>
-                <mass value="0.001"/>
+            <origin xyz="0.045 0.0 0.1" rpy="0.0 0.0 0.0"/>
+                <mass value="0.165"/>
                 <inertia
-                    ixx="1e-6" ixy="0.0" ixz="0.0"
-                    iyy="1e-6" iyz="0.0"
-                    izz="1e-6"/>
+                    ixx="4.755e-4" ixy="1.448e-7" ixz="-2.282e-4"
+                    iyy="6.841e-4" iyz="8.589e-8"
+                    izz="3.525e-4"/>
         </inertial>
     </link>
@@ -75,5 +75,5 @@
     <link name="motor_head_link">
         <visual>
-            <origin xyz="0.0 0.0 0.0" rpy="0.0 0.0 0.0"/>
+            <origin xyz="0.0 0.0 0.0" rpy="${PI/2} ${-PI/2} 0.0"/>
             <geometry>
                 <mesh filename="package://i3e-d3_description/meshes/servo.stl"/>
@@ -82,11 +82,11 @@
         </visual>
         <collision>
-            <origin xyz="0.0 0.0 0.0" rpy="0.0 0.0 0.0"/>
+            <origin xyz="0.0 0.0 0.0" rpy="${PI/2} ${-PI/2} 0.0"/>
             <geometry>
-                <box size="0.04 0.02 0.04"/>
+                <mesh filename="package://i3e-d3_description/meshes/servo.stl"/>
             </geometry>
         </collision>
         <inertial>
-            <origin xyz="0.0 0.0 0.0" rpy="0.0 0.0 0.0"/>
+            <origin xyz="0.0 0.0 0.0" rpy="${PI/2} ${-PI/2} 0.0"/>
                 <mass value="0.001"/>
                 <inertia
@@ -97,8 +97,8 @@
     </link>
     <joint name="head_joint" type="revolute">
-        <origin xyz="-0.0085 -0.117 0.142" rpy="0.0 ${-PI/2} 0.0"/>
+        <origin xyz="0.117 -0.0085 0.142" rpy="0.0 0.0 0.0"/>
         <parent link="neck_link"/>
         <child link="motor_head_link"/>
-        <axis xyz="0 0 1"/>
+        <axis xyz="0 -1 0"/>
         <limit lower="-0.2618" upper="0.2618" effort="0.8" velocity="0.5"/>
     </joint>
@@ -106,5 +106,5 @@
     <link name="face_link">
         <visual>
-            <origin xyz="0.0 0.0 0.0" rpy="0.0 ${-PI/2} ${PI}"/>
+            <origin xyz="0.0 0.0 0.0" rpy="0.0 0.0 0.0"/>
             <geometry>
                 <mesh filename="package://i3e-d3_description/meshes/face.stl"/>
@@ -113,5 +113,5 @@
         </visual>
         <collision>
-            <origin xyz="0.0 0.0 0.0" rpy="0.0 ${-PI/2} ${PI}"/>
+            <origin xyz="0.0 0.0 0.0" rpy="0.0 0.0 0.0"/>
             <geometry>
                 <mesh filename="package://i3e-d3_description/meshes/face.stl"/>
@@ -128,5 +128,5 @@
     </link>
     <joint name="motor_head_joint" type="fixed">
-        <origin xyz="-0.0115 -0.0435 -0.012" rpy="0.0 0.0 0.0"/>
+        <origin xyz="0.0475 0.005 -0.012" rpy="0.0 0.0 0.0"/>
         <child link="face_link"/>
         <parent link="motor_head_link"/>
@@ -134,5 +134,5 @@
     <link name="display_link">
         <visual>
-            <origin xyz="0.0 0.0 0.0" rpy="0.0 0.0 0.0"/>
+            <origin xyz="0.0 0.0 0.0" rpy="0.0 0.0 ${PI}"/>
             <geometry>
                 <mesh filename="package://i3e-d3_description/meshes/LEDs_face.stl"/>
@@ -141,7 +141,35 @@
         </visual>
         <collision>
+            <origin xyz="0.0 0.0 0.0" rpy="0.0 0.0 ${PI}"/>
+            <geometry>
+                <mesh filename="package://i3e-d3_description/meshes/LEDs_face.stl"/>
+            </geometry>
+        </collision>
+        <inertial>
+            <origin xyz="0.0 0.0 0.0" rpy="0.0 0.0 ${PI}"/>
+                <mass value="0.001"/>
+                <inertia
+                    ixx="1e-6" ixy="0.0" ixz="0.0"
+                    iyy="1e-6" iyz="0.0"
+                    izz="1e-6"/>
+        </inertial>
+    </link>
+    <joint name="display_joint" type="fixed">
+        <origin xyz="0.018 0.004 -0.0046" rpy="0.0 0.0 0.0"/>
+        <child link="display_link"/>
+        <parent link="face_link"/>
+    </joint>
+    <link name="head_cover_link">
+        <visual>
             <origin xyz="0.0 0.0 0.0" rpy="0.0 0.0 0.0"/>
             <geometry>
-                <mesh filename="package://i3e-d3_description/meshes/LEDs_face.stl"/>
+                <mesh filename="package://i3e-d3_description/meshes/head_cover.stl"/>
+            </geometry>
+            <material name="blue"/>
+        </visual>
+        <collision>
+            <origin xyz="0.0 0.0 0.0" rpy="0.0 0.0 0.0"/>
+            <geometry>
+                <mesh filename="package://i3e-d3_description/meshes/head_cover.stl"/>
             </geometry>
         </collision>
@@ -155,34 +183,6 @@
         </inertial>
     </link>
-    <joint name="display_joint" type="fixed">
-        <origin xyz="-0.005 -0.02 0.0" rpy="${PI/2} ${PI/2} 0.0"/>
-        <child link="display_link"/>
-        <parent link="face_link"/>
-    </joint>
-    <link name="head_cover_link">
-        <visual>
-            <origin xyz="0.0 0.0 0.0" rpy="${-PI/2} ${PI/2} ${PI/2}"/>
-            <geometry>
-                <mesh filename="package://i3e-d3_description/meshes/head_cover.stl"/>
-            </geometry>
-            <material name="blue"/>
-        </visual>
-        <collision>
-            <origin xyz="0.0 0.0 0.0" rpy="0.0 0.0 0.0"/>
-            <geometry>
-                <mesh filename="package://i3e-d3_description/meshes/head_cover.stl"/>
-            </geometry>cover
-        </collision>
-        <inertial>
-            <origin xyz="0.0 0.0 0.0" rpy="0.0 0.0 0.0"/>
-                <mass value="0.001"/>
-                <inertia
-                    ixx="1e-6" ixy="0.0" ixz="0.0"
-                    iyy="1e-6" iyz="0.0"
-                    izz="1e-6"/>
-        </inertial>
-    </link>
     <joint name="head_cover_joint" type="fixed">
-        <origin xyz="0.011 0.009 0.0" rpy="0.0 ${PI} 0.0"/>
+        <origin xyz="-0.011 0.004 0.009" rpy="0.0 0.0 0.0"/>
         <child link="head_cover_link"/>
         <parent link="face_link"/>

File: i3e-d3_description/urdf/i3e-d3.urdf.xacro (robot description, xacro)
@@ -74,5 +74,7 @@
     </xacro:i3e-d3_caster>
     <!-- Sensors -->
-    <xacro:i3e-d3_camera/>
+    <xacro:i3e-d3_camera>
+      <origin xyz="0.026 0.004 0.05" rpy="0.0 0.0 0.0"/>
+    </xacro:i3e-d3_camera>
     <xacro:i3e-d3_lidar>
         <origin xyz="${base_radius/2} 0.0 ${base_height/2 + 0.025}" rpy="0.0 0.0 0.0"/>
@@ -81,9 +83,4 @@
         <origin xyz="0.0 0.0 0.0" rpy="0.0 0.0 0.0"/>
     </xacro:i3e-d3_imu>
-    <gazebo reference="base_link"><material>Gazebo/Blue</material></gazebo>
-    <!--
-    <gazebo reference="neck"><material>Gazebo/DarkGrey</material></gazebo>
-    <gazebo reference="head"><material>Gazebo/Yellow</material></gazebo>
-    -->
     <!-- Gazebo ROS Control Plugin -->
     <!--gazebo>

File: i3e-d3_description/urdf/materials.urdf.xacro (robot description, xacro)
@@ -16,4 +16,7 @@
     <color rgba="1.0 1.0 1.0 1.0"/>
   </material>
+  <gazebo reference="base_link">
+    <material>Gazebo/Blue</material>
+  </gazebo>
   <gazebo reference="neck_link">
     <material>Gazebo/White</material>

File: i3e-d3_description/urdf/wheel.urdf.xacro (robot description, xacro)
@@ -20,4 +20,5 @@
                           scale="${wheel_radius/husky_wheel_radius} ${wheel_length/husky_wheel_length} ${wheel_radius/husky_wheel_radius}"/>
                 </geometry>
+                <material name="dark_grey"/>
             </visual>
             <collision>

Commit message: update colisions in urdf

File: i3e-d3_description/urdf/accessories.urdf.xacro (robot description, xacro)
@@ -84,10 +84,4 @@
         </geometry>
       </visual>
-      <collision>
-        <origin xyz="0.0 0.0 0.0" rpy="0.0 0.0 0.0"/>
-        <geometry>
-          <box size="0.025 0.024 0.001"/>
-        </geometry>
-      </collision>
     </link>
     <joint name="camera_joint" type="fixed">

File: i3e-d3_description/urdf/head.urdf.xacro (robot description, xacro)
@@ -112,17 +112,11 @@
             <material name="gray"/>
         </visual>
-        <collision>
-            <origin xyz="0.0 0.0 0.0" rpy="0.0 0.0 0.0"/>
-            <geometry>
-                <mesh filename="package://i3e-d3_description/meshes/face.stl"/>
-            </geometry>
-        </collision>
         <inertial>
-            <origin xyz="0.0 0.0 0.0" rpy="0.0 0.0 0.0"/>
-                <mass value="0.001"/>
+            <origin xyz="0.01 0.004 -0.004" rpy="0.0 0.0 0.0"/>
+                <mass value="0.259"/>
                 <inertia
-                    ixx="1e-6" ixy="0.0" ixz="0.0"
-                    iyy="1e-6" iyz="0.0"
-                    izz="1e-6"/>
+                    ixx="7.966e-4" ixy="-1.019e-7" ixz="9.196e-6"
+                    iyy="5.993e-4" iyz="7.634e-8"
+                    izz="3.527e-4"/>
         </inertial>
     </link>
@@ -140,10 +134,4 @@
             <material name="white"/>
         </visual>
-        <collision>
-            <origin xyz="0.0 0.0 0.0" rpy="0.0 0.0 ${PI}"/>
-            <geometry>
-                <mesh filename="package://i3e-d3_description/meshes/LEDs_face.stl"/>
-            </geometry>
-        </collision>
         <inertial>
             <origin xyz="0.0 0.0 0.0" rpy="0.0 0.0 ${PI}"/>
@@ -169,16 +157,16 @@
         </visual>
         <collision>
-            <origin xyz="0.0 0.0 0.0" rpy="0.0 0.0 0.0"/>
+            <origin xyz="-0.012 0.0 -0.008" rpy="0.0 0.0 0.0"/>
             <geometry>
-                <mesh filename="package://i3e-d3_description/meshes/head_cover.stl"/>
+                <box size="0.105 0.130 0.170"/>
             </geometry>
         </collision>
         <inertial>
             <origin xyz="0.0 0.0 0.0" rpy="0.0 0.0 0.0"/>
-                <mass value="0.001"/>
+                <mass value="0.252"/>
                 <inertia
-                    ixx="1e-6" ixy="0.0" ixz="0.0"
-                    iyy="1e-6" iyz="0.0"
-                    izz="1e-6"/>
+                    ixx="1.463e-3" ixy="0.0" ixz="1.598e-4"
+                    iyy="1.046e-3" iyz="0.0"
+                    izz="8.181e-4"/>
         </inertial>
     </link>

File: i3e-d3_description/urdf/i3e-d3.urdf.xacro (robot description, xacro)
@@ -59,4 +59,5 @@
         <origin xyz="0.0 0.0 0.0" rpy="0.0 0.0 0.0"/>
     </joint>
+    <!-- I3E-D3 head and neck -->
     <xacro:i3e-d3_head/>
     <!-- I3E-D3 wheel macros -->
@@ -67,4 +68,5 @@
         <origin xyz="${wheel_x_offset} ${-wheel_y_offset} ${wheel_z_offset}" rpy="0.0 0.0 0.0"/>
     </xacro:i3e-d3_wheel>
+    <!-- I3E-D3 caster macros -->
     <xacro:i3e-d3_caster prefix="front">
         <origin xyz="${2*base_radius/3} 0.0 ${-base_height/2}" rpy="0.0 0.0 0.0"/>

Commit message: Remove tf_prefix

File: i3e-d3_description/urdf/accessories.urdf.xacro (robot description, xacro)
@@ -63,5 +63,5 @@
         </ray>
         <plugin name="gazebo_ros_head_hokuyo_controller" filename="libgazebo_ros_laser.so">
-          <robotNamespace>$(arg robot_namespace)</robotNamespace>
+          <!--robotNamespace>$(arg robot_namespace)</robotNamespace-->
           <topicName>laser/scan</topicName>
           <frameName>3irobotix_lidar</frameName>
@@ -115,5 +115,5 @@
         </camera>
         <plugin name="camera_controller" filename="libgazebo_ros_camera.so">
-          <robotNamespace>$(arg robot_namespace)</robotNamespace>
+          <!--robotNamespace>$(arg robot_namespace)</robotNamespace-->
           <alwaysOn>true</alwaysOn>
           <updateRate>0.0</updateRate>
@@ -156,5 +156,5 @@
             <xyzOffset>0 0 0</xyzOffset>
             <rpyOffset>0 0 0</rpyOffset>
-            <frameName>$(arg robot_namespace)/imu_link</frameName>
+            <frameName>imu_link</frameName>
             <initialOrientationAsReference>false</initialOrientationAsReference>
           </plugin>

File: i3e-d3_description/urdf/caster.urdf.xacro (robot description, xacro)
@@ -13,5 +13,5 @@
 					<mesh filename="package://i3e-d3_description/meshes/caster_base.stl" scale="1 1 1"/>
 				</geometry>
-				<material name="Grey"/>
+				<material name="gray"/>
 			</visual>
 			<collision>
@@ -48,5 +48,5 @@
 					<mesh filename="package://i3e-d3_description/meshes/caster_rot.stl" scale="1 1 1"/>
 				</geometry>
-				<material name="Grey"/>
+				<material name="gray"/>
 			</visual>
 			<collision>
@@ -83,5 +83,5 @@
 					<sphere radius="${35/2000}"/>
 				</geometry>
-				<material name="Yellow"/>
+				<material name="yellow"/>
 			</visual>
 			<collision>

File: i3e-d3_description/urdf/head.urdf.xacro (robot description, xacro)
@@ -20,5 +20,5 @@
                 <mesh filename="package://i3e-d3_description/meshes/servo.stl"/>
             </geometry>
-            <material name="darkgray"/>
+            <material name="dark_gray"/>
         </visual>
         <collision>
@@ -79,5 +79,5 @@
                 <mesh filename="package://i3e-d3_description/meshes/servo.stl"/>
             </geometry>
-            <material name="darkgray"/>
+            <material name="dark_gray"/>
         </visual>
         <collision>

File: i3e-d3_description/urdf/i3e-d3.urdf.xacro (robot description, xacro)
@@ -5,9 +5,9 @@
     <xacro:property name="PI" value="3.14159"/>
     <!-- Included URDF/XACRO Files -->
+    <xacro:include filename="$(find i3e-d3_description)/urdf/materials.urdf.xacro"/>
     <xacro:include filename="$(find i3e-d3_description)/urdf/wheel.urdf.xacro"/>
     <xacro:include filename="$(find i3e-d3_description)/urdf/caster.urdf.xacro"/>
     <xacro:include filename="$(find i3e-d3_description)/urdf/accessories.urdf.xacro"/>
     <xacro:include filename="$(find i3e-d3_description)/urdf/head.urdf.xacro"/>
-    <xacro:include filename="$(find i3e-d3_description)/urdf/materials.urdf.xacro"/>
     <!-- Base, head and neck sizes -->
     <xacro:property name="base_radius" value="0.155"/>
@@ -113,5 +113,5 @@
   <gazebo>
     <plugin name="gazebo_ros_control" filename="libgazebo_ros_control.so">
-      <robotNamespace>$(arg robot_namespace)</robotNamespace>
+      <!--robotNamespace>$(arg robot_namespace)</robotNamespace-->
       <controlPeriod>0.001</controlPeriod>
       <robotSimType>gazebo_ros_control/DefaultRobotHWSim</robotSimType>

File: i3e-d3_description/urdf/materials.urdf.xacro (robot description, xacro)
@@ -7,8 +7,11 @@
     <color rgba="0.0 0.0 0.8 1.0"/>
   </material>
+  <material name="yellow">
+    <color rgba="1.0 1.0 0.0 1.0"/>
+  </material>
   <material name="gray">
     <color rgba="0.7 0.7 0.7 1.0"/>
   </material>
-  <material name="darkgray">
+  <material name="dark_gray">
     <color rgba="0.3 0.3 0.3 1.0"/>
   </material>

File: i3e-d3_description/urdf/wheel.urdf.xacro (robot description, xacro)
@@ -20,5 +20,5 @@
                           scale="${wheel_radius/husky_wheel_radius} ${wheel_length/husky_wheel_length} ${wheel_radius/husky_wheel_radius}"/>
                 </geometry>
-                <material name="dark_grey"/>
+                <material name="dark_gray"/>
             </visual>
             <collision>
