Commit message: Finish i3e-d3_bringup

File: i3e-d3_description/urdf/accessories.urdf.xacro (robot description, xacro)
@@ -6,5 +6,5 @@
   <!-- 3irobotix LIDAR -->
   <xacro:macro name="i3e-d3_lidar" params="*joint_pose">
-    <link name="3irobotix_lidar">
+    <link name="lidar">
       <inertial>
         <origin xyz="0.0 0.0 0.0" rpy="0.0 0.0 0.0"/>
@@ -28,10 +28,10 @@
     <joint name="lidar_joint" type="fixed">
       <parent link="base_link"/>
-      <child link="3irobotix_lidar"/>
+      <child link="lidar"/>
       <xacro:insert_block name="joint_pose"/>
     </joint>
-    <gazebo reference="3irobotix_lidar"><material>Gazebo/Black</material></gazebo>
+    <gazebo reference="lidar"><material>Gazebo/Black</material></gazebo>
       <!-- Laser Plugin -->
-    <gazebo reference="3irobotix_lidar">
+    <gazebo reference="lidar">
       <sensor type="ray" name="lidar_sensor">
         <pose>0 0 0 0 0 0</pose>
@@ -65,5 +65,5 @@
           <!--robotNamespace>$(arg robot_namespace)</robotNamespace-->
           <topicName>laser/scan</topicName>
-          <frameName>3irobotix_lidar</frameName>
+          <frameName>lidar</frameName>
         </plugin>
       </sensor>
@@ -72,5 +72,5 @@
   <!-- Camera -->
   <xacro:macro name="i3e-d3_camera" params="*joint_pose">
-    <link name="camera_link">
+    <link name="camera">
       <inertial>
         <origin xyz="0.0 0.0 0.0" rpy="0.0 0.0 0.0"/>
@@ -87,9 +87,9 @@
     <joint name="camera_joint" type="fixed">
       <parent link="face_link"/>
-      <child link="camera_link"/>
+      <child link="camera"/>
       <xacro:insert_block name="joint_pose"/>
     </joint>
     <!-- Camera Plugin -->
-    <gazebo reference="camera_link">
+    <gazebo reference="camera">
       <sensor type="camera" name="camera">
         <update_rate>30.0</update_rate>
@@ -121,5 +121,5 @@
           <imageTopicName>image_raw</imageTopicName>
           <cameraInfoTopicName>camera_info</cameraInfoTopicName>
-          <frameName>camera_link</frameName>
+          <frameName>camera</frameName>
           <hackBaseline>0.07</hackBaseline>
           <distortionK1>0.0</distortionK1>
@@ -134,12 +134,12 @@
   <!-- IMU -->
   <xacro:macro name="i3e-d3_imu" params="*joint_pose">
-    <link name="imu_link"/>
+    <link name="imu"/>
     <joint name="imu_joint" type="fixed">
       <parent link="base_link"/>
-      <child link="imu_link"/>
+      <child link="imu_"/>
       <xacro:insert_block name="joint_pose"/>
     </joint>
       <!-- IMU plugin -->
-      <gazebo reference="imu_link">
+      <gazebo reference="imu">
         <gravity>true</gravity>
         <sensor name="imu_sensor" type="imu">
@@ -150,11 +150,11 @@
           <plugin filename="libgazebo_ros_imu_sensor.so" name="imu_plugin">
             <!--robotNamespace>$(arg robot_namespace)</robotNamespace-->
-            <topicName>imu/data</topicName>
-            <bodyName>imu_link</bodyName>
+            <topicName>imu/data/filtered</topicName>
+            <bodyName>imu</bodyName>
             <updateRateHZ>10.0</updateRateHZ>
             <gaussianNoise>0.0</gaussianNoise>
             <xyzOffset>0 0 0</xyzOffset>
             <rpyOffset>0 0 0</rpyOffset>
-            <frameName>imu_link</frameName>
+            <frameName>imu</frameName>
             <initialOrientationAsReference>false</initialOrientationAsReference>
           </plugin>

File: i3e-d3_description/urdf/materials.urdf.xacro (robot description, xacro)
@@ -46,5 +46,5 @@
     <material>Gazebo/DarkGray</material>
   </gazebo>
-  <gazebo reference="camera_link">
+  <gazebo reference="camera">
     <material>Gazebo/Green</material>
   </gazebo>

Commit message: Create odometry publisher in i3e-d3_bringup

File: i3e-d3_description/urdf/accessories.urdf.xacro (robot description, xacro)
@@ -137,5 +137,5 @@
     <joint name="imu_joint" type="fixed">
       <parent link="base_link"/>
-      <child link="imu_"/>
+      <child link="imu"/>
       <xacro:insert_block name="joint_pose"/>
     </joint>

Commit message: Update meshes and URDF

File: i3e-d3_description/urdf/accessories.urdf.xacro (robot description, xacro)
@@ -13,5 +13,5 @@
       </inertial>
       <visual>
-        <origin xyz="0.0 0.0 -0.025" rpy="0.0 0.0 0.0"/>
+        <origin xyz="0.0 0.0 -0.024" rpy="0.0 0.0 0.0"/>
         <geometry>
           <mesh filename="package://i3e-d3_description/meshes/lidar.stl"/>
@@ -20,5 +20,5 @@
       </visual>
       <collision>
-        <origin xyz="0.0 0.0 0.0" rpy="0.0 0.0 0.0"/>
+        <origin xyz="0.0 0.0 -0.024" rpy="0.0 0.0 0.0"/>
         <geometry>
           <mesh filename="package://i3e-d3_description/meshes/lidar.stl"/>
@@ -36,5 +36,5 @@
       <sensor type="ray" name="lidar_sensor">
         <pose>0 0 0 0 0 0</pose>
-        <visualize>false</visualize>
+        <visualize>true</visualize>
         <update_rate>40</update_rate>
         <ray>

File: i3e-d3_description/urdf/head.urdf.xacro (robot description, xacro)
@@ -1,5 +1,5 @@
 <?xml version="1.0"?>
 <robot name="i3e-d3_head" xmlns:xacro="http://www.ros.org/wiki/xacro">
-  <xacro:macro name="i3e-d3_head">
+  <xacro:macro name="i3e-d3_head" params="*joint_pose">
     <xacro:macro name="TransmissionServo" params="joint n">
         <transmission name="tran_${n}">
@@ -40,5 +40,5 @@
         <parent link="base_link"/>
         <child link="motor_neck_link"/>
-        <origin xyz="0.005 0.0 ${base_height/2}" rpy="0.0 0.0 0.0"/>
+        <xacro:insert_block name="joint_pose"/>
     </joint>
     <link name="neck_link">

File: i3e-d3_description/urdf/i3e-d3.urdf.xacro (robot description, xacro)
@@ -10,7 +10,8 @@
     <xacro:include filename="$(find i3e-d3_description)/urdf/accessories.urdf.xacro"/>
     <xacro:include filename="$(find i3e-d3_description)/urdf/head.urdf.xacro"/>
+    <xacro:include filename="$(find i3e-d3_description)/urdf/arm.urdf.xacro"/>
     <!-- Base, head and neck sizes -->
     <xacro:property name="base_radius" value="0.155"/>
-    <xacro:property name="base_height" value="0.342"/>
+    <xacro:property name="base_height" value="0.34568"/>
     <xacro:property name="base_weight" value="0.515"/>
     <!-- Wheel Dimensions -->
@@ -20,5 +21,5 @@
     <xacro:property name="wheel_x_offset" value="0"/>
     <xacro:property name="wheel_y_offset" value="${wheel_length/2 + base_radius + 0.005}"/>
-    <xacro:property name="wheel_z_offset" value="${-base_height/2 + 0.05}"/>
+    <xacro:property name="wheel_z_offset" value="0.0312"/>
     <!-- Base link is the center of the robot -->
     <link name="base_link">
@@ -26,10 +27,9 @@
             <origin xyz="0.0 0.0 0.0" rpy="0.0 0.0 0.0"/>
             <geometry>
-                <cylinder radius="${base_radius}" length="${base_height}"/>
+                <mesh filename="package://i3e-d3_description/meshes/base_link.dae"/>
             </geometry>
-            <material name="blue"/>"
         </visual>
         <collision>
-            <origin xyz="0.0 0.0 0.0" rpy="0.0 0.0 0.0"/>
+            <origin xyz="0.0 0.0 ${base_height/2 - 0.0007}" rpy="0.0 0.0 0.0"/>
             <geometry>
                 <cylinder radius="${base_radius}" length="${base_height}"/>
@@ -60,151 +60,15 @@
         <origin xyz="0.0 0.0 0.0" rpy="0.0 0.0 0.0"/>
     </joint>
-    <!-- I3E-D3 Arm -->
-    <link name="left_arm">
-        <inertial>
-            <origin xyz="0.04 0.0 0.0" rpy="0.0 ${-PI/2} ${PI/6}"/>
-            <mass value="0.05"/>
-            <inertia ixx="1e-6" ixy="0.0" ixz="0.0" iyy="1e-6" iyz="0.0" izz="1e-6"/>
-        </inertial>
-        <visual>
-            <origin xyz="0.04 0.0 0.0" rpy="0.0 ${-PI/2} ${PI/6}"/>
-            <geometry>
-                <mesh filename="package://i3e-d3_description/meshes/arm.stl" scale="1e-3 1e-3 1e-3"/>
-            </geometry>
-        </visual>
-        <collision>
-            <origin xyz="0.04 0.0 0.0" rpy="0.0 ${-PI/2} ${PI/6}"/>
-            <geometry>
-                <mesh filename="package://i3e-d3_description/meshes/arm.stl" scale="1e-3 1e-3 1e-3"/>
-            </geometry>
-        </collision>
-    </link>
-    <link name="right_arm">
-        <inertial>
-            <origin xyz="0.04 0.0 0.0" rpy="0.0 ${-PI/2} ${PI/6}"/>
-            <mass value="0.05"/>
-            <inertia ixx="1e-6" ixy="0.0" ixz="0.0" iyy="1e-6" iyz="0.0" izz="1e-6"/>
-        </inertial>
-        <visual>
-            <origin xyz="0.04 0.0 0.0" rpy="0.0 ${-PI/2} ${PI/6}"/>
-            <geometry>
-                <mesh filename="package://i3e-d3_description/meshes/arm.stl" scale="1e-3 1e-3 1e-3"/>
-            </geometry>
-        </visual>
-        <collision>
-            <origin xyz="0.04 0.0 0.0" rpy="0.0 ${-PI/2} ${PI/6}"/>
-            <geometry>
-                <mesh filename="package://i3e-d3_description/meshes/arm.stl" scale="1e-3 1e-3 1e-3"/>
-            </geometry>
-        </collision>
-    </link>
-    <joint name="left_arm_joint" type="fixed">
-        <parent link="base_link"/>
-        <child link="left_arm"/>
-        <origin xyz="0.0 0.18 -0.03" rpy="0.0 0.0 0.0"/>
-    </joint>
-    <joint name="right_arm_joint" type="fixed">
-        <parent link="base_link"/>
-        <child link="right_arm"/>
-        <origin xyz="0.0 -0.20 -0.03" rpy="0.0 0.0 0.0"/>
-    </joint>
-    <link name="left_forearm">
-        <inertial>
-            <origin xyz="0.04 0.0 0.0" rpy="0.0 ${-PI/2} ${PI/6}"/>
-            <mass value="0.05"/>
-            <inertia ixx="1e-6" ixy="0.0" ixz="0.0" iyy="1e-6" iyz="0.0" izz="1e-6"/>
-        </inertial>
-        <visual>
-            <origin xyz="0.04 0.0 0.0" rpy="0.0 ${-PI/2} ${PI/6}"/>
-            <geometry>
-                <mesh filename="package://i3e-d3_description/meshes/forearm.stl" scale="1e-3 1e-3 1e-3"/>
-            </geometry>
-        </visual>
-        <collision>
-            <origin xyz="0.04 0.0 0.0" rpy="0.0 ${-PI/2} ${PI/6}"/>
-            <geometry>
-                <mesh filename="package://i3e-d3_description/meshes/forearm.stl" scale="1e-3 1e-3 1e-3"/>
-            </geometry>
-        </collision>
-    </link>
-    <link name="right_forearm">
-        <inertial>
-            <origin xyz="0.04 0.0 0.0" rpy="0.0 ${-PI/2} ${PI/6}"/>
-            <mass value="0.05"/>
-            <inertia ixx="1e-6" ixy="0.0" ixz="0.0" iyy="1e-6" iyz="0.0" izz="1e-6"/>
-        </inertial>
-        <visual>
-            <origin xyz="0.04 0.0 0.0" rpy="0.0 ${-PI/2} ${PI/6}"/>
-            <geometry>
-                <mesh filename="package://i3e-d3_description/meshes/forearm.stl" scale="1e-3 1e-3 1e-3"/>
-            </geometry>
-        </visual>
-        <collision>
-            <origin xyz="0.04 0.0 0.0" rpy="0.0 ${-PI/2} ${PI/6}"/>
-            <geometry>
-                <mesh filename="package://i3e-d3_description/meshes/forearm.stl" scale="1e-3 1e-3 1e-3"/>
-            </geometry>
-        </collision>
-    </link>
-    <joint name="left_forearm_joint" type="fixed">
-        <parent link="left_arm"/>
-        <child link="left_forearm"/>
-        <origin xyz="0.0 0.0 0.08" rpy="0.0 ${PI} 0.0"/>
-    </joint>
-    <joint name="right_forearm_joint" type="fixed">
-        <parent link="right_arm"/>
-        <child link="right_forearm"/>
-        <origin xyz="0.0 0.0 0.08" rpy="0.0 ${PI} 0.0"/>
-    </joint>
-    <link name="left_hand">
-        <inertial>
-            <origin xyz="0.04 0.0 0.0" rpy="0.0 ${-PI/2} ${PI/6}"/>
-            <mass value="0.05"/>
-            <inertia ixx="1e-6" ixy="0.0" ixz="0.0" iyy="1e-6" iyz="0.0" izz="1e-6"/>
-        </inertial>
-        <visual>
-            <origin xyz="0.04 0.0 0.0" rpy="0.0 ${-PI/2} ${PI/6}"/>
-            <geometry>
-                <mesh filename="package://i3e-d3_description/meshes/hand.stl" scale="1e-3 1e-3 1e-3"/>
-            </geometry>
-        </visual>
-        <collision>
-            <origin xyz="0.04 0.0 0.0" rpy="0.0 ${-PI/2} ${PI/6}"/>
-            <geometry>
-                <mesh filename="package://i3e-d3_description/meshes/hand.stl" scale="1e-3 1e-3 1e-3"/>
-            </geometry>
-        </collision>
-    </link>
-    <link name="right_hand">
-        <inertial>
-            <origin xyz="0.04 0.0 0.0" rpy="0.0 ${-PI/2} ${PI/6}"/>
-            <mass value="0.05"/>
-            <inertia ixx="1e-6" ixy="0.0" ixz="0.0" iyy="1e-6" iyz="0.0" izz="1e-6"/>
-        </inertial>
-        <visual>
-            <origin xyz="0.04 0.0 0.0" rpy="0.0 ${-PI/2} ${PI/6}"/>
-            <geometry>
-                <mesh filename="package://i3e-d3_description/meshes/hand.stl" scale="1e-3 1e-3 1e-3"/>
-            </geometry>
-        </visual>
-        <collision>
-            <origin xyz="0.04 0.0 0.0" rpy="0.0 ${-PI/2} ${PI/6}"/>
-            <geometry>
-                <mesh filename="package://i3e-d3_description/meshes/hand.stl" scale="1e-3 1e-3 1e-3"/>
-            </geometry>
-        </collision>
-    </link>
-    <joint name="left_hand_joint" type="fixed">
-        <parent link="left_forearm"/>
-        <child link="left_hand"/>
-        <origin xyz="0.0 -0.022 0.04" rpy="${-PI/2} 0.0 ${PI/16}"/>
-    </joint>
-    <joint name="right_hand_joint" type="fixed">
-        <parent link="right_forearm"/>
-        <child link="right_hand"/>
-        <origin xyz="0.0 -0.028 0.04" rpy="${-PI/2} 0.0 ${-PI/24}"/>
-    </joint>
+    <!-- I3E-D3 arms, forearms and hands -->
+    <xacro:i3e-d3_arm prefix="left">
+        <origin xyz="0.0 0.100 0.294" rpy="0.0 0.0 0.0"/>
+    </xacro:i3e-d3_arm>
+    <!-- <xacro:i3e-d3_arm prefix="right">
+        <origin xyz="0.0 -0.100 0.294" rpy="0.0 0.0 0.0"/>
+    <xacro:i3e-d3_arm/> -->
     <!-- I3E-D3 head and neck -->
-    <xacro:i3e-d3_head/>
+    <xacro:i3e-d3_head>
+        <origin xyz="-0.01 0.0 ${base_height - 0.0014}" rpy="0.0 0.0 0.0"/>
+    </xacro:i3e-d3_head>
     <!-- I3E-D3 wheel macros -->
     <xacro:i3e-d3_wheel prefix="left">
@@ -219,5 +83,5 @@
 						 x="${2*base_radius/3}"
 						 y="0.0"
-						 z="${-base_height/2 + 0.008}"
+						 z="-0.01"
 						 roll="0.0"
 						 pitch="0.0"
@@ -231,5 +95,5 @@
 						 x="${-2*base_radius/3}"
 						 y="0.0"
-						 z="${-base_height/2 + 0.008}"
+						 z="-0.01"
 						 roll="0.0"
 						 pitch="0.0"
@@ -244,5 +108,5 @@
     </xacro:i3e-d3_camera>
     <xacro:i3e-d3_lidar>
-        <origin xyz="${base_radius/2} 0.0 ${base_height/2 + 0.025}" rpy="0.0 0.0 0.0"/>
+        <origin xyz="${base_radius/2 - 0.012} 0.0 ${base_height - 0.0014 + 0.036 + 0.024}" rpy="0.0 0.0 0.0"/>
     </xacro:i3e-d3_lidar>
     <xacro:i3e-d3_imu>

File: i3e-d3_description/urdf/materials.urdf.xacro (robot description, xacro)
@@ -19,7 +19,4 @@
     <color rgba="1.0 1.0 1.0 1.0"/>
   </material>
-  <gazebo reference="base_link">
-    <material>Gazebo/Blue</material>
-  </gazebo>
   <gazebo reference="neck_link">
     <material>Gazebo/White</material>

Commit message: Update URDF

File: i3e-d3_description/urdf/accessories.urdf.xacro (robot description, xacro)
@@ -13,5 +13,5 @@
       </inertial>
       <visual>
-        <origin xyz="0.0 0.0 -0.024" rpy="0.0 0.0 0.0"/>
+        <origin xyz="0.0 0.0 -0.02" rpy="0.0 0.0 0.0"/>
         <geometry>
           <mesh filename="package://i3e-d3_description/meshes/lidar.stl"/>
@@ -20,5 +20,5 @@
       </visual>
       <collision>
-        <origin xyz="0.0 0.0 -0.024" rpy="0.0 0.0 0.0"/>
+        <origin xyz="0.0 0.0 -0.02" rpy="0.0 0.0 0.0"/>
         <geometry>
           <mesh filename="package://i3e-d3_description/meshes/lidar.stl"/>
@@ -36,5 +36,5 @@
       <sensor type="ray" name="lidar_sensor">
         <pose>0 0 0 0 0 0</pose>
-        <visualize>true</visualize>
+        <visualize>false</visualize>
         <update_rate>40</update_rate>
         <ray>

File: i3e-d3_description/urdf/i3e-d3.urdf.xacro (robot description, xacro)
@@ -64,7 +64,7 @@
         <origin xyz="0.0 0.100 0.294" rpy="0.0 0.0 0.0"/>
     </xacro:i3e-d3_arm>
-    <!-- <xacro:i3e-d3_arm prefix="right">
+    <xacro:i3e-d3_arm prefix="right">
         <origin xyz="0.0 -0.100 0.294" rpy="0.0 0.0 0.0"/>
-    <xacro:i3e-d3_arm/> -->
+    </xacro:i3e-d3_arm>
     <!-- I3E-D3 head and neck -->
     <xacro:i3e-d3_head>
@@ -108,20 +108,13 @@
     </xacro:i3e-d3_camera>
     <xacro:i3e-d3_lidar>
-        <origin xyz="${base_radius/2 - 0.012} 0.0 ${base_height - 0.0014 + 0.036 + 0.024}" rpy="0.0 0.0 0.0"/>
+        <origin xyz="${base_radius/2 - 0.012} 0.0 ${base_height - 0.0014 + 0.036 + 0.024 - 0.01}" rpy="0.0 0.0 0.0"/>
     </xacro:i3e-d3_lidar>
     <xacro:i3e-d3_imu>
         <origin xyz="0.0 0.0 0.0" rpy="0.0 0.0 0.0"/>
     </xacro:i3e-d3_imu>
-    <!-- Gazebo ROS Control Plugin -->
-    <!--gazebo>
-        <plugin name="gazebo_ros_control" filename="libgazebo_ros_control.so">
-            <robotNamespace>$(arg robot_namespace)</robotNamespace>
-            <legacyModeNS>true</legacyModeNS>
-        </plugin>
-    </gazebo-->
   <gazebo>
     <plugin name="gazebo_ros_control" filename="libgazebo_ros_control.so">
       <!--robotNamespace>$(arg robot_namespace)</robotNamespace-->
-      <controlPeriod>0.001</controlPeriod>
+      <controlPeriod>0.002</controlPeriod>
       <robotSimType>gazebo_ros_control/DefaultRobotHWSim</robotSimType>
       <legacyModeNS>true</legacyModeNS>

File: i3e-d3_description/urdf/wheel.urdf.xacro (robot description, xacro)
@@ -31,6 +31,6 @@
         <!-- Need to adjust gazebo properties -->
         <gazebo reference="${prefix}_wheel_link">
-            <mu1 value="1.0"/>
-            <mu2 value="1.0"/>
+            <mu1 value="2.0"/>
+            <mu2 value="2.0"/>
             <kp value="10000000.0" />
             <kd value="1" />
